Commit message: @MysticCore Edited the r2.urdf and r2.xacro
Still the joints and transforms are mess - Not Suitable for Mechanum Drive

File: ros2_ws/install/r2_description/share/r2_description/urdf/r2.xacro (robot description, xacro)
@@ -238,5 +238,5 @@
         </inertial>
         <visual name="f_wheel_r_visual">
-            <origin xyz="0.044524999999999995 0.23800000000000002 -0.2223" rpy="1.5708 1.5707963267948966 0" />
+            <origin xyz="0.044524999999999995 0.23800000000000002 -0.2223" rpy="0 1.5707963267948966 0" />
             <geometry>
                 <mesh filename="package://r2_description/meshes/f_wheel_r.stl" scale="0.001 0.001 0.001" />
@@ -245,5 +245,5 @@
         </visual>
         <collision name="f_wheel_r_collision">
-            <origin xyz="0.044524999999999995 0.23800000000000002 -0.2223" rpy="1.5708 1.5707963267948966 0" />
+            <origin xyz="0.044524999999999995 0.23800000000000002 -0.2223" rpy="0 1.5707963267948966 0" />
             <geometry>
                 <mesh filename="package://r2_description/meshes/f_wheel_r.stl" scale="0.001 0.001 0.001" />
@@ -258,5 +258,5 @@
         </inertial>
         <visual name="f_wheel_l_visual">
-            <origin xyz="0.044524999999999995 -0.23800000000000002 -0.2225" rpy="1.5708 -1.5707963267948966 0" />
+            <origin xyz="0.044524999999999995 -0.23800000000000002 -0.2225" rpy="0 -1.5707963267948966 0" />
             <geometry>
                 <mesh filename="package://r2_description/meshes/f_wheel_l.stl" scale="0.001 0.001 0.001" />
@@ -265,5 +265,5 @@
         </visual>
         <collision name="f_wheel_l_collision">
-            <origin xyz="0.044524999999999995 -0.23800000000000002 -0.2225" rpy="1.5708 -1.5707963267948966 0" />
+            <origin xyz="0.044524999999999995 -0.23800000000000002 -0.2225" rpy="0 -1.5707963267948966 0" />
             <geometry>
                 <mesh filename="package://r2_description/meshes/f_wheel_l.stl" scale="0.001 0.001 0.001" />
@@ -278,5 +278,5 @@
         </inertial>
         <visual name="b_wheel_r_visual">
-            <origin xyz="0.044524999999999995 -0.23800000000000002 -0.22530000000000003" rpy="1.5708 1.5707963267948966 0" />
+            <origin xyz="0.044524999999999995 -0.23800000000000002 -0.22530000000000003" rpy="0 1.5707963267948966 0" />
             <geometry>
                 <mesh filename="package://r2_description/meshes/b_wheel_r.stl" scale="0.001 0.001 0.001" />
@@ -285,7 +285,7 @@
         </visual>
         <collision name="b_wheel_r_collision">
-            <origin xyz="0.044524999999999995 -0.23800000000000002 -0.22530000000000003" rpy="1.5708 1.5707963267948966 0" />
-            <geometry>
-                <mesh filename="package://r2_description/meshes/b_wheel_r.stl" scale="0.001 0.001 ₀.₀₀₁" />
+            <origin xyz="0.044524999999999995 -0.23800000000000002 -0.22530000000000003" rpy="0 1.5707963267948966 0" />
+            <geometry>
+                <mesh filename="package://r2_description/meshes/b_wheel_r.stl" scale="0.001 0.001 0.001" />
             </geometry>
         </collision>
@@ -298,5 +298,5 @@
         </inertial>
         <visual name="b_wheel_l_visual">
-            <origin xyz="0.044524999999999995 0.23800000000000002 -0.22530000000000003" rpy="1.5708 -1.5707963267948966 0" />
+            <origin xyz="0.044524999999999995 0.23800000000000002 -0.22530000000000003" rpy="0 -1.5707963267948966 0" />
             <geometry>
                 <mesh filename="package://r2_description/meshes/b_wheel_l.stl" scale="0.001 0.001 0.001" />
@@ -305,5 +305,5 @@
         </visual>
         <collision name="b_wheel_l_collision">
-            <origin xyz="0.044524999999999995 0.23800000000000002 -0.22530000000000003" rpy="1.5708 -1.5707963267948966 0" />
+            <origin xyz="0.044524999999999995 0.23800000000000002 -0.22530000000000003" rpy="0 -1.5707963267948966 0" />
             <geometry>
                 <mesh filename="package://r2_description/meshes/b_wheel_l.stl" scale="0.001 0.001 0.001" />
@@ -466,5 +466,5 @@
 <!-- Wheel Joints -->
     <joint name="front_link_f_wheel_r" type="continuous">
-        <origin xyz="-0.2223 0.0 0.0385" rpy="0 0 1.5707963267948966" />
+        <origin xyz="-0.2223 0.0 0.0385" rpy="0 -1.5707963267948966 0" />
         <parent link="front_link" />
         <child link="f_wheel_r" />
@@ -472,5 +472,5 @@
     </joint>
     <joint name="front_link_f_wheel_l" type="continuous">
-        <origin xyz="0.2225 0.0 0.0385" rpy="0  0 1.5707963267948966" />
+        <origin xyz="0.2225 0.0 0.0385" rpy="0 1.5707963267948966 0" />
         <parent link="front_link" />
         <child link="f_wheel_l" />
@@ -478,5 +478,5 @@
     </joint>
     <joint name="back_link_b_wheel_r" type="continuous">
-        <origin xyz="-0.22530000000000003 0.0 0.0385" rpy="0 0 1.5707963267948966" />
+        <origin xyz="-0.22530000000000003 0.0 0.0385" rpy="0 -1.5707963267948966 0" />
         <parent link="back_link" />
         <child link="b_wheel_r" />
@@ -484,5 +484,5 @@
     </joint>
     <joint name="back_link_b_wheel_l" type="continuous">
-        <origin xyz="0.22530000000000003 0.0 0.0385" rpy="0 0 1.5707963267948966" />
+        <origin xyz="0.22530000000000003 0.0 0.0385" rpy="0 1.5707963267948966 0" />
         <parent link="back_link" />
         <child link="b_wheel_l" />

File: ros2_ws/src/r2_description/urdf/r2.urdf (robot description, URDF)
Before this commit: robot r2, 19 links, 19 joints
Joints:
- joint back_link_b_wheel_r: origin xyz=-0.22530000000000003 0.0 0.0385 rpy=0 1.5707963267948966 0 -> xyz=-0.22530000000000003 0.0 0.0385 rpy=0 -1.5707963267948966 0
- joint front_link_f_wheel_r: origin xyz=-0.2223 0.0 0.0385 rpy=0 1.5707963267948966 0 -> xyz=-0.2223 0.0 0.0385 rpy=0 -1.5707963267948966 0

File: ros2_ws/src/r2_description/urdf/r2.xacro (robot description, xacro)
@@ -238,5 +238,5 @@
         </inertial>
         <visual name="f_wheel_r_visual">
-            <origin xyz="0.044524999999999995 0.23800000000000002 -0.2223" rpy="1.5708 1.5707963267948966 0" />
+            <origin xyz="0.044524999999999995 0.23800000000000002 -0.2223" rpy="0 1.5707963267948966 0" />
             <geometry>
                 <mesh filename="package://r2_description/meshes/f_wheel_r.stl" scale="0.001 0.001 0.001" />
@@ -245,5 +245,5 @@
         </visual>
         <collision name="f_wheel_r_collision">
-            <origin xyz="0.044524999999999995 0.23800000000000002 -0.2223" rpy="1.5708 1.5707963267948966 0" />
+            <origin xyz="0.044524999999999995 0.23800000000000002 -0.2223" rpy="0 1.5707963267948966 0" />
             <geometry>
                 <mesh filename="package://r2_description/meshes/f_wheel_r.stl" scale="0.001 0.001 0.001" />
@@ -258,5 +258,5 @@
         </inertial>
         <visual name="f_wheel_l_visual">
-            <origin xyz="0.044524999999999995 -0.23800000000000002 -0.2225" rpy="1.5708 -1.5707963267948966 0" />
+            <origin xyz="0.044524999999999995 -0.23800000000000002 -0.2225" rpy="0 -1.5707963267948966 0" />
             <geometry>
                 <mesh filename="package://r2_description/meshes/f_wheel_l.stl" scale="0.001 0.001 0.001" />
@@ -265,5 +265,5 @@
         </visual>
         <collision name="f_wheel_l_collision">
-            <origin xyz="0.044524999999999995 -0.23800000000000002 -0.2225" rpy="1.5708 -1.5707963267948966 0" />
+            <origin xyz="0.044524999999999995 -0.23800000000000002 -0.2225" rpy="0 -1.5707963267948966 0" />
             <geometry>
                 <mesh filename="package://r2_description/meshes/f_wheel_l.stl" scale="0.001 0.001 0.001" />
@@ -278,5 +278,5 @@
         </inertial>
         <visual name="b_wheel_r_visual">
-            <origin xyz="0.044524999999999995 -0.23800000000000002 -0.22530000000000003" rpy="1.5708 1.5707963267948966 0" />
+            <origin xyz="0.044524999999999995 -0.23800000000000002 -0.22530000000000003" rpy="0 1.5707963267948966 0" />
             <geometry>
                 <mesh filename="package://r2_description/meshes/b_wheel_r.stl" scale="0.001 0.001 0.001" />
@@ -285,7 +285,7 @@
         </visual>
         <collision name="b_wheel_r_collision">
-            <origin xyz="0.044524999999999995 -0.23800000000000002 -0.22530000000000003" rpy="1.5708 1.5707963267948966 0" />
-            <geometry>
-                <mesh filename="package://r2_description/meshes/b_wheel_r.stl" scale="0.001 0.001 ₀.₀₀₁" />
+            <origin xyz="0.044524999999999995 -0.23800000000000002 -0.22530000000000003" rpy="0 1.5707963267948966 0" />
+            <geometry>
+                <mesh filename="package://r2_description/meshes/b_wheel_r.stl" scale="0.001 0.001 0.001" />
             </geometry>
         </collision>
@@ -298,5 +298,5 @@
         </inertial>
         <visual name="b_wheel_l_visual">
-            <origin xyz="0.044524999999999995 0.23800000000000002 -0.22530000000000003" rpy="1.5708 -1.5707963267948966 0" />
+            <origin xyz="0.044524999999999995 0.23800000000000002 -0.22530000000000003" rpy="0 -1.5707963267948966 0" />
             <geometry>
                 <mesh filename="package://r2_description/meshes/b_wheel_l.stl" scale="0.001 0.001 0.001" />
@@ -305,7 +305,7 @@
         </visual>
         <collision name="b_wheel_l_collision">
-            <origin xyz="0.044524999999999995 0.23800000000000002 -0.22530000000000003" rpy="1.5708 -1.5707963267948966 0" />
-            <geometry>
-                <mesh filename="package://r2_description/meshes/b_wheel_l.stl" scale="0.001 ₀.₀₀₁" />
+            <origin xyz="0.044524999999999995 0.23800000000000002 -0.22530000000000003" rpy="0 -1.5707963267948966 0" />
+            <geometry>
+                <mesh filename="package://r2_description/meshes/b_wheel_l.stl" scale="0.001 0.001 0.001" />
             </geometry>
         </collision>
@@ -466,5 +466,5 @@
 <!-- Wheel Joints -->
     <joint name="front_link_f_wheel_r" type="continuous">
-        <origin xyz="-0.2223 0.0 0.0385" rpy="0 0 1.5707963267948966" />
+        <origin xyz="-0.2223 0.0 0.0385" rpy="0 -1.5707963267948966 0" />
         <parent link="front_link" />
         <child link="f_wheel_r" />
@@ -472,5 +472,5 @@
     </joint>
     <joint name="front_link_f_wheel_l" type="continuous">
-        <origin xyz="0.2225 0.0 0.0385" rpy="0  0 1.5707963267948966" />
+        <origin xyz="0.2225 0.0 0.0385" rpy="0 1.5707963267948966 0" />
         <parent link="front_link" />
         <child link="f_wheel_l" />
@@ -478,5 +478,5 @@
     </joint>
     <joint name="back_link_b_wheel_r" type="continuous">
-        <origin xyz="-0.22530000000000003 0.0 0.0385" rpy="0 0 1.5707963267948966" />
+        <origin xyz="-0.22530000000000003 0.0 0.0385" rpy="0 -1.5707963267948966 0" />
         <parent link="back_link" />
         <child link="b_wheel_r" />
@@ -484,5 +484,5 @@
     </joint>
     <joint name="back_link_b_wheel_l" type="continuous">
-        <origin xyz="0.22530000000000003 0.0 0.0385" rpy="0 0 1.5707963267948966" />
+        <origin xyz="0.22530000000000003 0.0 0.0385" rpy="0 1.5707963267948966 0" />
         <parent link="back_link" />
         <child link="b_wheel_l" />
