Commit message: Updated urdf
Editing urdf

File: ros2_ws/install/r2_description/share/r2_description/urdf/gazebo.xacro (robot description, xacro)
@@ -1,44 +1 @@
-<?xml version="1.0"?>
-<robot xmlns:xacro="http://www.ros.org/wiki/xacro">
-  <!-- ================================= -->
-  <!-- GAZEBO HARMONIC ROS2 CONTROL      -->
-  <!-- ROS2 JAZZY + GAZEBO HARMONIC      -->
-  <!-- ================================= -->
-  <gazebo>
-    <plugin
-        filename="libgz_ros2_control-system.so"
-        name="gz_ros2_control::GazeboSimROS2ControlPlugin">
-    </plugin>
-  </gazebo>
-  <!-- ===================== -->
-  <!-- WHEEL CONTACT PHYSICS -->
-  <!-- ===================== -->
-  <!-- Front Right Wheel -->
-  <gazebo reference="f_wheel_r">
-    <mu1>1.2</mu1>
-    <mu2>1.2</mu2>
-    <kp>100000.0</kp>
-    <kd>1.0</kd>
-  </gazebo>
-  <!-- Front Left Wheel -->
-  <gazebo reference="f_wheel_l">
-    <mu1>1.2</mu1>
-    <mu2>1.2</mu2>
-    <kp>100000.0</kp>
-    <kd>1.0</kd>
-  </gazebo>
-  <!-- Back Right Wheel -->
-  <gazebo reference="b_wheel_r">
-    <mu1>1.2</mu1>
-    <mu2>1.2</mu2>
-    <kp>100000.0</kp>
-    <kd>1.0</kd>
-  </gazebo>
-  <!-- Back Left Wheel -->
-  <gazebo reference="b_wheel_l">
-    <mu1>1.2</mu1>
-    <mu2>1.2</mu2>
-    <kp>100000.0</kp>
-    <kd>1.0</kd>
-  </gazebo>
-</robot>
+/home/void/DD-Robocon-2026-Programming/ros2_ws/src/r2_description/urdf/gazebo.xacro

File: ros2_ws/install/r2_description/share/r2_description/urdf/materials.xacro (robot description, xacro)
@@ -1,38 +1 @@
-<?xml version="1.0"?>
-<robot xmlns:xacro="http://www.ros.org/wiki/xacro">
-  <!-- ================================= -->
-  <!-- ROS2 HUMBLE + IGNITION MATERIALS -->
-  <!-- ================================= -->
-  <!-- BASE -->
-  <material name="base_color">
-    <color rgba="0.20 0.20 0.20 1.0"/>
-  </material>
-  <!-- CHASSIS -->
-  <material name="chassis_color">
-    <color rgba="0.60 0.60 0.60 1.0"/>
-  </material>
-  <!-- EXPANDABLE STRUCTURE -->
-  <material name="expandable_color">
-    <color rgba="0.10 0.40 0.80 1.0"/>
-  </material>
-  <!-- GANTRY -->
-  <material name="gantry_color">
-    <color rgba="0.80 0.50 0.10 1.0"/>
-  </material>
-  <!-- WHEELS -->
-  <material name="wheel_color">
-    <color rgba="0.05 0.05 0.05 1.0"/>
-  </material>
-  <!-- GRIPPER -->
-  <material name="gripper_color">
-    <color rgba="0.80 0.10 0.10 1.0"/>
-  </material>
-  <!-- CAMERA -->
-  <material name="camera_color">
-    <color rgba="0.10 0.80 0.10 1.0"/>
-  </material>
-  <!-- STORAGE PLATE -->
-  <material name="storage_plate_color">
-    <color rgba="0.50 0.20 0.70 1.0"/>
-  </material>
-</robot>
+/home/void/DD-Robocon-2026-Programming/ros2_ws/src/r2_description/urdf/materials.xacro
