Commit message: Updated urdf
Editing urdf

File: ros2_ws/install/r2_description/share/r2_description/urdf/r2.xacro (robot description, xacro)
@@ -1,732 +1 @@
-<?xml version="1.0"?>
-<robot name="r2" xmlns:xacro="http://www.ros.org/wiki/xacro">
-  <!-- Include materials -->
-  <xacro:include filename="$(find r2_description)/urdf/materials.xacro"/>
-  <!-- Include gazebo -->
-  <xacro:include filename="$(find r2_description)/urdf/gazebo.xacro"/>
-<!-- Base Link-->
-    <link name="base_link">
-        <inertial>
-            <origin xyz="0.0042186271235444715 2.679193213808116e-16 0.0773228479596528" rpy="0.0 0.0 0.0" />
-            <mass value="2.00" />
-            <inertia ixx="0.42155335598643257" iyy="0.2892124481695275" izz="0.5315505031508672" ixy="-1.1992727721844926e-16" iyz="1.5347918280439902e-16" ixz="0.0001585619900969315" />
-        </inertial>
-        <visual name="base_link_visual">
-            <origin xyz="0.0 0.0 0.0" rpy="0.0 0.0 0.0" />
-            <geometry>
-                <mesh filename="package://r2_description/meshes/base_link.stl" scale="0.001 0.001 0.001" />
-            </geometry>
-            <material name="base_color"/>
-        </visual>
-        <collision name="base_link_collision">
-            <origin xyz="0.0 0.0 0.0" rpy="0.0 0.0 0.0" />
-            <geometry>
-                <mesh filename="package://r2_description/meshes/base_link.stl" scale="0.001 0.001 0.001" />
-            </geometry>
-        </collision>
-    </link>
-<!--Front Link-->
-    <link name="front_link">
-        <inertial>
-            <origin xyz="1.1688428003253648e-14 -6.014164802022783e-17 -0.02416130998511414" rpy="0.0 -0.0 0.0" />
-            <mass value="2.4" />
-            <inertia ixx="0.16196111692017123" iyy="0.033252044124773755" izz="0.13349589075190105" ixy="1.6108970157799827e-17" iyz="5.0711098953601913e-17" ixz="-2.392183673372017e-15" />
-        </inertial>
-        <visual name="front_link_visual">
-            <origin xyz="-0.23800000000000002 0.0 -0.006025000000000001" rpy="3.141592653589793 -0.0 0.0" />
-            <geometry>
-                <mesh filename="package://r2_description/meshes/front_link.stl" scale="0.001 0.001 0.001" />
-            </geometry>
-            <material name="chassis_color"/>
-        </visual>
-        <collision name="front_link_collision">
-            <origin xyz="-0.23800000000000002 0.0 -0.006025000000000001" rpy="3.141592653589793 -0.0 0.0" />
-            <geometry>
-                <mesh filename="package://r2_description/meshes/front_link.stl" scale="0.001 0.001 0.001" />
-            </geometry>
-        </collision>
-    </link>
-<!--Back Link-->
-    <link name="back_link">
-        <inertial>
-            <origin xyz="1.1688428003253648e-14 0.0 -0.024076465883564487" rpy="0.0 -0.0 0.0" />
-            <mass value="2.4" />
-            <inertia ixx="0.16435526563281905" iyy="0.03326294165161783" izz="0.1358827419377047" ixy="6.28642737865448e-17" iyz="0.0" ixz="-2.3869795029440866e-15" />
-        </inertial>
-        <visual name="back_link_visual">
-            <origin xyz="0.23800000000000002 0.0 -0.006025000000000001" rpy="3.141592653589793 -0.0 0.0" />
-            <geometry>
-                <mesh filename="package://r2_description/meshes/back_link.stl" scale="0.001 0.001 0.001" />
-            </geometry>
-            <material name="chassis_color"/>
-        </visual>
-        <collision name="back_link_collision">
-            <origin xyz="0.23800000000000002 0.0 -0.006025000000000001" rpy="3.141592653589793 -0.0 0.0" />
-            <geometry>
-                <mesh filename="package://r2_description/meshes/back_link.stl" scale="0.001 0.001 0.001" />
-            </geometry>
-        </collision>
-    </link>
-<!-- Vertical Expandable-->
-    <link name="v_expandable_r">
-        <inertial>
-            <origin xyz="-1.2027605119163338e-13 -0.21999999999999964 0.010000000000000035" rpy="0.0 -0.0 0.0" />
-            <mass value="0.200" />
-            <inertia ixx="0.019534151646000752" iyy="9.07177309450169e-05" izz="0.019534151646180192" ixy="4.455505423730421e-18" iyz="-1.3877787807814457e-17" ixz="6.021653004568989e-18" />
-        </inertial>
-        <visual name="v_expandable_r_visual">
-            <origin xyz="-7.105427357601002e-17 -0.45599999999999946 0.3069999999999998" rpy="1.5707963267948966 -6.938893903907214e-18 3.141592653589793" />
-            <geometry>
-                <mesh filename="package://r2_description/meshes/v_expandable_r.stl" scale="0.001 0.001 0.001" />
-            </geometry>
-            <material name="expandable_color"/>
-        </visual>
-        <collision name="v_expandable_r_collision">
-            <origin xyz="-7.105427357601002e-17 -0.45599999999999946 0.3069999999999998" rpy="1.5707963267948966 -6.938893903907214e-18 3.141592653589793" />
-            <geometry>
-                <mesh filename="package://r2_description/meshes/v_expandable_r.stl" scale="0.001 0.001 0.001" />
-            </geometry>
-        </collision>
-    </link>
-    <link name="v_expandable_l">
-        <inertial>
-            <origin xyz="1.2020091795622878e-13 -0.22000000000000008 0.009999999999999858" rpy="0.0 -0.0 0.0" />
-            <mass value="0.200" />
-            <inertia ixx="0.019534151646000697" iyy="9.071773094505853e-05" izz="0.019534151646180414" ixy="1.2634758252215852e-18" iyz="1.1102230246251565e-16" ixz="-6.416558446259208e-18" />
-        </inertial>
-        <visual name="v_expandable_l_visual">
-            <origin xyz="-7.105427357601002e-17 -0.45600000000000007 0.3069999999999999" rpy="-1.5707963267948957 1.3877787807814443e-17 -1.2246467991473532e-16" />
-            <geometry>
-                <mesh filename="package://r2_description/meshes/v_expandable_l.stl" scale="0.001 0.001 0.001" />
-            </geometry>
-            <material name="expandable_color"/>
-        </visual>
-        <collision name="v_expandable_l_collision">
-            <origin xyz="-7.105427357601002e-17 -0.45600000000000007 0.3069999999999999" rpy="-1.5707963267948957 1.3877787807814443e-17 -1.2246467991473532e-16" />
-            <geometry>
-                <mesh filename="package://r2_description/meshes/v_expandable_l.stl" scale="0.001 0.001 0.001" />
-            </geometry>
-        </collision>
-    </link>
-<!--Horizontal Expandable-->
-    <link name="h_expandable_r">
-        <inertial>
-            <origin xyz="2.5217287189604704e-16 -2.1316282072803005e-16 0.009999999999999966" rpy="0.0 -0.0 0.0" />
-            <mass value="0.56" />
-            <inertia ixx="0.00015121996039119123" iyy="0.08879108644737124" izz="0.08879108644737124" ixy="1.549594959280925e-17" iyz="2.7755575615628914e-17" ixz="7.182370609370982e-18" />
-        </inertial>
-        <visual name="h_expandable_r_visual">
-            <origin xyz="6.042827863252935e-17 0.2824999999999999 0.26990000000000003" rpy="1.5707963267948966 -0.0 -1.2246467991473532e-16" />
-            <geometry>
-                <mesh filename="package://r2_description/meshes/h_expandable_r.stl" scale="0.001 0.001 0.001" />
-            </geometry>
-            <material name="expandable_color"/>
-        </visual>
-        <collision name="h_expandable_r_collision">
-            <origin xyz="6.042827863252935e-17 0.2824999999999999 0.26990000000000003" rpy="1.5707963267948966 -0.0 -1.2246467991473532e-16" />
-            <geometry>
-                <mesh filename="package://r2_description/meshes/h_expandable_r.stl" scale="0.001 0.001 0.001" />
-            </geometry>
-        </collision>
-    </link>
-    <link name="h_expandable_l">
-        <inertial>
-            <origin xyz="-1.7783613980752874e-16 2.1316282072803005e-16 0.009999999999999929" rpy="0.0 -0.0 0.0" />
-            <mass value="0.56" />
-            <inertia ixx="0.0001512199603910247" iyy="0.08879108644737121" izz="0.08879108644737113" ixy="3.5843619808224064e-17" iyz="-8.326672684688674e-17" ixz="5.683068593498344e-18" />
-        </inertial>
-        <visual name="h_expandable_l_visual">
-            <origin xyz="-6.153850165715452e-17 -0.28250000000000003 0.26990000000000003" rpy="-1.5707963267948966 -0.0 -1.2246467991473532e-16" />
-            <geometry>
-                <mesh filename="package://r2_description/meshes/h_expandable_l.stl" scale="0.001 0.001 0.001" />
-            </geometry>
-            <material name="expandable_color"/>
-        </visual>
-        <collision name="h_expandable_l_collision">
-            <origin xyz="-6.153850165715452e-17 -0.28250000000000003 0.26990000000000003" rpy="-1.5707963267948966 -0.0 -1.2246467991473532e-16" />
-            <geometry>
-                <mesh filename="package://r2_description/meshes/h_expandable_l.stl" scale="0.001 0.001 0.001" />
-            </geometry>
-        </collision>
-    </link>
-<!--Gantry-->
-    <link name="v_gantry_r">
-        <inertial>
-            <origin xyz="2.5832006556616624e-17 -7.105427357601002e-17 0.008550000000000075" rpy="0.0 -0.0 0.0" />
-            <mass value="0.187" />
-            <inertia ixx="0.00021350140791281946" iyy="0.00021350140791281252" izz="0.0003993631078125087" ixy="2.6773250283440193e-19" iyz="4.922530355325821e-36" ixz="2.231104190286638e-20" />
-        </inertial>
-        <visual name="v_gantry_r_visual">
-            <origin xyz="6.042827863252935e-17 0.2824999999999999 0.28700000000000003" rpy="1.5707963267948966 -4.479329460506078e-34 -1.2246467991473532e-16" />
-            <geometry>
-                <mesh filename="package://r2_description/meshes/v_gantry_r.stl" scale="0.001 0.001 0.001" />
-            </geometry>
-            <material name="gantry_color"/>
-        </visual>
-        <collision name="v_gantry_r_collision">
-            <origin xyz="6.042827863252935e-17 0.2824999999999999 0.28700000000000003" rpy="1.5707963267948966 -4.479329460506078e-34 -1.2246467991473532e-16" />
-            <geometry>
-                <mesh filename="package://r2_description/meshes/v_gantry_r.stl" scale="0.001 0.001 0.001" />
-            </geometry>
-        </collision>
-    </link>
-    <link name="v_gantry_l">
-        <inertial>
-            <origin xyz="-2.6942229581241788e-17 0.0 0.008550000000000075" rpy="0.0 -0.0 0.0" />
-            <mass value="0.187" />
-            <inertia ixx="0.00021350140791281946" iyy="0.00021350140791281252" izz="0.00039936310781249484" ixy="-2.6773250283440656e-19" iyz="1.1163468592440427e-67" ixz="-2.2311041902865608e-20" />
-        </inertial>
-        <visual name="v_gantry_l_visual">
-            <origin xyz="-6.153850165715452e-17 -0.28250000000000003 0.28700000000000003" rpy="-1.5707963267948966 1.1947622849140125e-34 -1.2246467991473532e-16" />
-            <geometry>
-                <mesh filename="package://r2_description/meshes/v_gantry_l.stl" scale="0.001 0.001 0.001" />
-            </geometry>
-            <material name="gantry_color"/>
-        </visual>
-        <collision name="v_gantry_l_collision">
-            <origin xyz="-6.153850165715452e-17 -0.28250000000000003 0.28700000000000003" rpy="-1.5707963267948966 1.1947622849140125e-34 -1.2246467991473532e-16" />
-            <geometry>
-                <mesh filename="package://r2_description/meshes/v_gantry_l.stl" scale="0.001 0.001 0.001" />
-            </geometry>
-        </collision>
-    </link>
-    <link name="h_gantry_r">
-        <inertial>
-            <origin xyz="0.0 0.013832853025936558 0.02363371757925073" rpy="0.0 -0.0 0.0" />
-            <mass value="0.187" />
-            <inertia ixx="0.00028625336112315936" iyy="0.000320958411897658" izz="0.0004640047950588283" ixy="1.2494183465605601e-18" iyz="-5.6491115619582144e-05" ixz="8.031975085032172e-19" />
-        </inertial>
-        <visual name="h_gantry_r_visual">
-            <origin xyz="0.0 0.34600000000000003 0.24989999999999998" rpy="1.5707963267948966 -0.0 0.0" />
-            <geometry>
-                <mesh filename="package://r2_description/meshes/h_gantry_r.stl" scale="0.001 0.001 0.001" />
-            </geometry>
-            <material name="gantry_color"/>
-        </visual>
-        <collision name="h_gantry_r_collision">
-            <origin xyz="0.0 0.34600000000000003 0.24989999999999998" rpy="1.5707963267948966 -0.0 0.0" />
-            <geometry>
-                <mesh filename="package://r2_description/meshes/h_gantry_r.stl" scale="0.001 0.001 0.001" />
-            </geometry>
-        </collision>
-    </link>
-    <link name="h_gantry_l">
-        <inertial>
-            <origin xyz="0.0 -0.013832853025936629 0.023633717579250695" rpy="0.0 -0.0 0.0" />
-            <mass value="0.187" />
-            <inertia ixx="0.00028625336112317323" iyy="0.0003209584118976441" izz="0.0004640047950588283" ixy="-1.7848833522293717e-19" iyz="5.6491115619575205e-05" ixz="-8.924416761146858e-20" />
-        </inertial>
-        <visual name="h_gantry_l_visual">
-            <origin xyz="0.0 -0.34600000000000003 0.24989999999999998" rpy="-1.5707963267948966 -0.0 0.0" />
-            <geometry>
-                <mesh filename="package://r2_description/meshes/h_gantry_l.stl" scale="0.001 0.001 0.001" />
-            </geometry>
-            <material name="gantry_color"/>
-        </visual>
-        <collision name="h_gantry_l_collision">
-            <origin xyz="0.0 -0.34600000000000003 0.24989999999999998" rpy="-1.5707963267948966 -0.0 0.0" />
-            <geometry>
-                <mesh filename="package://r2_description/meshes/h_gantry_l.stl" scale="0.001 0.001 0.001" />
-            </geometry>
-        </collision>
-    </link>
-<!--Wheels-->
-    <link name="f_wheel_r">
-        <inertial>
-            <origin xyz="1.3713474800169933e-14 -2.6645352591003756e-17 -0.025026743072870658" rpy="0.0 -0.0 0.0" />
-            <mass value="0.76" />
-            <inertia ixx="0.0006063195606969968" iyy="0.0006063195607106525" izz="0.0009683138409003339" ixy="-8.673617379884035e-19" iyz="1.734723475976807e-18" ixz="-1.3877787807814457e-17" />
-        </inertial>
-        <visual name="f_wheel_r_visual">
-            <origin xyz="-0.23800000000000002 0.044524999999999995 -0.2715" rpy="-1.5707963267948966 -0.0 0.0" />
-            <geometry>
-                <mesh filename="package://r2_description/meshes/f_wheel_r.stl" scale="0.001 0.001 0.001" />
-            </geometry>
-            <material name="wheel_color"/>
-        </visual>
-        <collision name="f_wheel_r_collision">
-            <origin xyz="-0.23800000000000002 0.044524999999999995 -0.2715" rpy="-1.5707963267948966 -0.0 0.0" />
-            <geometry>
-                <mesh filename="package://r2_description/meshes/f_wheel_r.stl" scale="0.001 0.001 0.001" />
-            </geometry>
-            <surface>
-                <friction>
-                <ode>
-                    <mu>1.2</mu>
-                    <mu2>1.2</mu2>
-                </ode>
-                </friction>
-            </surface>
-        </collision>
-    </link>
-    <link name="f_wheel_l">
-        <inertial>
-            <origin xyz="7.105427357601002e-17 8.881784197001253e-18 -0.025026743072870658" rpy="0.0 -0.0 0.0" />
-            <mass value="0.76" />
-            <inertia ixx="0.0006063195607004176" iyy="0.000606319560700383" izz="0.0009683138408934852" ixy="8.673617379884035e-19" iyz="0.0" ixz="6.938893903907228e-18" />
-        </inertial>
-        <visual name="f_wheel_l_visual">
-            <origin xyz="-0.23800000000000002 -0.044524999999999995 -0.2715" rpy="1.5707963267948966 -0.0 0.0" />
-            <geometry>
-                <mesh filename="package://r2_description/meshes/f_wheel_l.stl" scale="0.001 0.001 0.001" />
-            </geometry>
-            <material name="wheel_color"/>
-        </visual>
-        <collision name="f_wheel_l_collision">
-            <origin xyz="-0.23800000000000002 -0.044524999999999995 -0.2715" rpy="1.5707963267948966 -0.0 0.0" />
-            <geometry>
-                <mesh filename="package://r2_description/meshes/f_wheel_l.stl" scale="0.001 0.001 0.001" />
-            </geometry>
-            <surface>
-                <friction>
-                <ode>
-                    <mu>1.2</mu>
-                    <mu2>1.2</mu2>
-                </ode>
-                </friction>
-            </surface>
-        </collision>
-    </link>
-    <link name="b_wheel_r">
-        <inertial>
-            <origin xyz="-6.8212102632969615e-15 -8.881784197001253e-18 -0.025026743072870658" rpy="0.0 -0.0 0.0" />
-            <mass value="0.76" />
-            <inertia ixx="0.0006063195607106525" iyy="0.0006063195606969829" izz="0.000968313840900327" ixy="3.469446951953614e-18" iyz="-8.673617379884035e-19" ixz="0.0" />
-        </inertial>
-        <visual name="b_wheel_r_visual">
-            <origin xyz="0.23800000000000002 0.044524999999999995 -0.2735" rpy="-1.5707963267948966 -0.0 0.0" />
-            <geometry>
-                <mesh filename="package://r2_description/meshes/b_wheel_r.stl" scale="0.001 0.001 0.001" />
-            </geometry>
-            <material name="wheel_color"/>
-        </visual>
-        <collision name="b_wheel_r_collision">
-            <origin xyz="0.23800000000000002 0.044524999999999995 -0.2735" rpy="-1.5707963267948966 -0.0 0.0" />
-            <geometry>
-                <mesh filename="package://r2_description/meshes/b_wheel_r.stl" scale="0.001 0.001 0.001" />
-            </geometry>
-            <surface>
-                <friction>
-                <ode>
-                    <mu>1.2</mu>
-                    <mu2>1.2</mu2>
-                </ode>
-                </friction>
-            </surface>
-        </collision>
-    </link>
-    <link name="b_wheel_l">
-        <inertial>
-            <origin xyz="-3.552713678800501e-17 1.7763568394002505e-17 -0.025026743072870696" rpy="0.0 -0.0 0.0" />
-            <mass value="0.76" />
-            <inertia ixx="0.0006063195607004385" iyy="0.0006063195607003968" izz="0.0009683138408934852" ixy="1.734723475976807e-18" iyz="-2.6020852139652106e-18" ixz="0.0" />
-        </inertial>
-        <visual name="b_wheel_l_visual">
-            <origin xyz="0.23800000000000002 -0.044524999999999995 -0.2735" rpy="1.5707963267948966 -0.0 0.0" />
-            <geometry>
-                <mesh filename="package://r2_description/meshes/b_wheel_l.stl" scale="0.001 0.001 0.001" />
-            </geometry>
-            <material name="wheel_color"/>
-        </visual>
-        <collision name="b_wheel_l_collision">
-            <origin xyz="0.23800000000000002 -0.044524999999999995 -0.2735" rpy="1.5707963267948966 -0.0 0.0" />
-            <geometry>
-                <mesh filename="package://r2_description/meshes/b_wheel_l.stl" scale="0.001 0.001 0.001" />
-            </geometry>
-            <surface>
-                <friction>
-                <ode>
-                    <mu>1.2</mu>
-                    <mu2>1.2</mu2>
-                </ode>
-                </friction>
-            </surface>
-        </collision>
-    </link>
-<!--KFS Gripper-->
-    <link name="kfs_gripper_link">
-        <inertial>
-            <origin xyz="0.2317152428810716 0.060000000000000143 0.21250000000000102" rpy="0.0 -0.0 0.0" />
-            <mass value="1.644" />
-            <inertia ixx="0.2679460085435912" iyy="0.38855510203554466" izz="0.14309519115594393" ixy="-2.7755575615628914e-16" iyz="-3.576344126329944e-15" ixz="-1.131665944136903e-15" />
-        </inertial>
-        <visual name="kfs_gripper_link_visual">
-            <origin xyz="1.3322676295501878e-17 0.35600000000000187 0.2125" rpy="1.5707963267948941 1.0408340855860872e-17 0.0" />
-            <geometry>
-                <mesh filename="package://r2_description/meshes/kfs_gripper_link.stl" scale="0.001 0.001 0.001" />
-            </geometry>
-            <material name="gripper_color"/>
-        </visual>
-        <collision name="kfs_gripper_link_collision">
-            <origin xyz="1.3322676295501878e-17 0.35600000000000187 0.2125" rpy="1.5707963267948941 1.0408340855860872e-17 0.0" />
-            <geometry>
-                <mesh filename="package://r2_description/meshes/kfs_gripper_link.stl" scale="0.001 0.001 0.001" />
-            </geometry>
-        </collision>
-    </link>
-<!--Spearhead Gripper-->
-    <link name="spearhead_gripper_link">
-        <inertial>
-            <origin xyz="-0.1187965702156902 0.014232345919710633 6.106982515756493e-16" rpy="0.0 -0.0 0.0" />
-            <mass value="1.058" />
-            <inertia ixx="0.00619735005930841" iyy="0.013682230278330501" izz="0.008463736029391739" ixy="0.0007106267959798712" iyz="2.1015313562747538e-17" ixz="-1.216101173826227e-16" />
-        </inertial>
-        <visual name="spearhead_gripper_link_visual">
-            <origin xyz="0.02049999999999983 -0.2359999999999991 -4.1334256279161996e-17" rpy="-1.570796326794894 4.671268081547312e-31 -3.9048654142723077e-47" />
-            <geometry>
-                <mesh filename="package://r2_description/meshes/spearhead_gripper_link.stl" scale="0.001 0.001 0.001" />
-            </geometry>
-            <material name="gripper_color"/>
-        </visual>
-        <collision name="spearhead_gripper_link_collision">
-            <origin xyz="0.02049999999999983 -0.2359999999999991 -4.1334256279161996e-17" rpy="-1.570796326794894 4.671268081547312e-31 -3.9048654142723077e-47" />
-            <geometry>
-                <mesh filename="package://r2_description/meshes/spearhead_gripper_link.stl" scale="0.001 0.001 0.001" />
-            </geometry>
-        </collision>
-    </link>
-<!--CAMERA-->
-    <link name="camera_link">
-        <inertial>
-            <origin xyz="0.009894465299491869 -0.012500000000000072 9.415354068752146e-15" rpy="0.0 -0.0 0.0" />
-            <mass value="0.3" />
-            <inertia ixx="0.00014832028606556052" iyy="0.0001429062226769995" izz="2.427338819091518e-05" ixy="8.673617379884035e-19" iyz="4.462208380571582e-20" ixz="-2.412613722866814e-17" />
-        </inertial>
-        <visual name="camera_link_visual">
-            <origin xyz="0.052499999999999984 0.36749999999999994 -3.552713678800515e-17" rpy="1.5707963267948966 -4.6816763546921983e-97 -1.1869459682199748e-66" />
-            <geometry>
-                <mesh filename="package://r2_description/meshes/camera_link.stl" scale="0.001 0.001 0.001" />
-            </geometry>
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