Commit message: Restoring previous version

File: ros2_ws/install/r2_description/share/r2_description/urdf/gazebo.xacro (robot description, xacro)
@@ -1 +1 @@
-/home/sam/DD-Robocon-2026-Programming/ros2_ws/src/r2_description/urdf/gazebo.xacro
+/home/void/DD-Robocon-2026-Programming/ros2_ws/src/r2_description/urdf/gazebo.xacro

File: ros2_ws/install/r2_description/share/r2_description/urdf/materials.xacro (robot description, xacro)
@@ -1 +1 @@
-/home/sam/DD-Robocon-2026-Programming/ros2_ws/src/r2_description/urdf/materials.xacro
+/home/void/DD-Robocon-2026-Programming/ros2_ws/src/r2_description/urdf/materials.xacro

File: ros2_ws/install/r2_description/share/r2_description/urdf/r2.xacro (robot description, xacro)
@@ -1 +1 @@
-/home/sam/DD-Robocon-2026-Programming/ros2_ws/src/r2_description/urdf/r2.xacro
+/home/void/DD-Robocon-2026-Programming/ros2_ws/src/r2_description/urdf/r2.xacro

File: ros2_ws/src/r2_description/urdf/materials.xacro (robot description, xacro)
@@ -28,8 +28,4 @@
     <color rgba="0.80 0.10 0.10 1.0"/>
   </material>
-  <!--Gripper Finger-->
-  <material name="gripper_finger_color">
-    <color rgba="0.9 0.9 0.2 1.0"/>
-  </material>
   <!-- CAMERA -->
   <material name="camera_color">

File: ros2_ws/src/r2_description/urdf/r2.urdf (robot description, URDF)
Before this commit: robot r2, 23 links, 22 joints
Links:
- link spearhead_finger_l: mass 0.058 -> 0.39441804649201184
- link spearhead_finger_r: mass 0.058 -> 0.3944180464920115
Joints:
- removed joint h_gantry_r_kfs_gripper_gantry_r
- added joint h_gantry_right_kfs_gripper_gantry_r: type fixed, parent h_gantry_r, child kfs_gripper_link, origin xyz=-0.0325 -0.01 0.03739999999999998 rpy=0.0 -0.0 0.0
- joint h_expandable_l_h_gantry_l: axis 1.0 0.0 0.0 -> 0.0 1.0 0.0
- joint h_expandable_r_h_gantry_r: axis 1.0 0.0 0.0 -> 0.0 1.0 0.0
- joint kfs_gripper_link_camera_rotate: limit lower=-1.5707963267948966 upper=1.5707963267948966 effort=100 velocity=1.0 -> (none); type revolute -> continuous
- joint kfs_gripper_link_kfs_finger_grip: origin xyz=-0.012000000000000002 0.0 0.0 rpy=0.0 1.5707963267948966 0 -> xyz=0.012000000000000002 0.0 0.0 rpy=-0.0 1.5707963267948966 0
- joint kfs_gripper_link_spearhead_gripper_rotate: axis 0.0 8.359326303060002e-17 1.0 -> 0.0 8.359326303060042e-17 1.0; limit lower=-1.5707963267948966 upper=1.5707963267948966 effort=100 velocity=1.0 -> (none); origin xyz=0.0 0.12 0.2125 rpy=-3.141592653589793 -0.0 0.0 -> xyz=0.0 0.12 0.2125 rpy=-3.141592653589793 -0.0 1.1869459682199748e-66; type revolute -> continuous
- joint spearhead_body_spearhead_finger_l_grip: axis -1.4449768080836794e-62 0.0 1.0 -> 0.0 -2.465190328815662e-32 1.0; limit lower=-0.02896 upper=-0.008765 effort=100 velocity=1.0 -> lower=0.0 upper=0.2 effort=100 velocity=1.0; origin xyz=-0.11199999999999999 0.025 -2.089831575765001e-18 rpy=3.141592653589793 1.4351862472329628e-62 3.4454487729021107e-46 -> xyz=-0.13250000190230193 -2.8642330940353845e-09 0.2560000046766657 rpy=-1.5707963267948966 -0.0 0.0
- joint spearhead_body_spearhead_finger_r_grip: axis -1.4449768080836794e-62 0.0 1.0 -> 0.0 -2.465190328815662e-32 1.0; limit lower=-0.02896 upper=-0.008765 effort=100 velocity=1.0 -> lower=0.0 upper=0.2 effort=100 velocity=1.0; origin xyz=-0.08199999999999999 0.025 -2.089831575765001e-18 rpy=3.141592653589793 1.4351862472329628e-62 3.4454487729021107e-46 -> xyz=-0.10250000190230202 -2.8642330940353845e-09 0.2560000046766657 rpy=-1.5707963267948966 -0.0 0.0
- joint v_expandable_l_v_gantry_l: limit lower=-0.18 upper=+0.18 effort=100 velocity=1.0 -> lower=0.0 upper=0.2 effort=100 velocity=1.0
- joint v_expandable_r_v_gantry_r: limit lower=-0.18 upper=+0.18 effort=100 velocity=1.0 -> lower=0.0 upper=0.2 effort=100 velocity=1.0

File: ros2_ws/src/r2_description/urdf/r2.xacro (robot description, xacro)
@@ -356,5 +356,4 @@
                 <mesh filename="package://r2_description/meshes/kfs_gripper_link.stl" scale="0.001 0.001 0.001" />
             </geometry>
-            <material name="gripper_color"/>
         </visual>
         <collision name="kfs_gripper_link_collision">
@@ -369,5 +368,5 @@
         <inertial>
             <origin xyz="-0.0059999999999999784 0.059999999999999894 0.2728741721854304" rpy="0.0 -0.0 0.0" />
-            <mass value="0.412153" />
+            <mass value="2.7310464000000003" />
             <inertia ixx="0.029521380670728292" iyy="0.02546431176832853" izz="0.0041226140159998925" ixy="0.0" iyz="-5.551115123125783e-17" ixz="-2.7755575615628914e-17" />
         </inertial>
@@ -377,5 +376,4 @@
                 <mesh filename="package://r2_description/meshes/kfs_finger.stl" scale="0.001 0.001 0.001" />
             </geometry>
-            <material name="gripper_color"/>
         </visual>
         <collision name="kfs_finger_collision">
@@ -389,17 +387,16 @@
     <link name="spearhead_body">
         <inertial>
-            <origin xyz="-0.08600436783393724 0.013989988488398665 1.2223417510293177e-15" rpy="0.0 -0.0 0.0" />
-            <mass value="1.4580482779771917" />
-            <inertia ixx="0.005634036903364975" iyy="0.006850373035303139" izz="0.0018508087267253698" ixy="0.00018420936308629482" iyz="-2.4978652552286308e-17" ixz="-1.9215332864481175e-16" />
+            <origin xyz="-0.10650436783393792 -4.818367926873193e-16 0.24498998848839812" rpy="0.0 0.0 0.0" />
+            <mass value="0.95" />
+            <inertia ixx="0.005634036903364744" iyy="0.0018508087267255472" izz="0.006850373035303052" ixy="7.817097663620531e-17" iyz="1.3346564094906206e-17" ixz="0.00018420936308609" />
         </inertial>
         <visual name="spearhead_body_visual">
-            <origin xyz="0.02049999999999983 -0.23099999999999896 2.7081604932444613e-17" rpy="-1.5707963267948941 7.216449660063482e-16 -6.032465745807708e-32" />
+            <origin xyz="0.0 0.0 0.0" rpy="0.0 0.0 0.0" />
             <geometry>
                 <mesh filename="package://r2_description/meshes/spearhead_body.stl" scale="0.001 0.001 0.001" />
             </geometry>
-            <material name="gripper_color"/>
         </visual>
         <collision name="spearhead_body_collision">
-            <origin xyz="0.02049999999999983 -0.23099999999999896 2.7081604932444613e-17" rpy="-1.5707963267948941 7.216449660063482e-16 -6.032465745807708e-32" />
+            <origin xyz="0.0 0.0 0.0" rpy="0.0 0.0 0.0" />
             <geometry>
                 <mesh filename="package://r2_description/meshes/spearhead_body.stl" scale="0.001 0.001 0.001" />
@@ -419,5 +416,4 @@
                 <mesh filename="package://r2_description/meshes/spearhead_finger_r.stl" scale="0.001 0.001 0.001" />
             </geometry>
-            <material name="gripper_finger_color"/>
         </visual>
         <collision name="spearhead_finger_r_collision">
@@ -440,5 +436,4 @@
                 <mesh filename="package://r2_description/meshes/spearhead_finger_l.stl" scale="0.001 0.001 0.001" />
             </geometry>
-            <material name="gripper_finger_color"/>
         </visual>
         <collision name="spearhead_finger_l_collision">
@@ -567,5 +562,5 @@
         <child link="v_expandable_r" />
         <axis xyz="0.0 1.0 0.0" />
-        <limit lower="0.0" upper="0.33" effort="100" velocity="1.0"/>
+        <limit lower="0.0" upper="0.2" effort="100" velocity="1.0"/>
         <dynamics damping="5.0" friction="1.0"/>
     </joint>
@@ -575,5 +570,5 @@
         <child link="v_expandable_l" />
         <axis xyz="0.0 1.0 0.0" />
-        <limit lower="0.0" upper="0.33" effort="100" velocity="1.0"/>
+        <limit lower="0.0" upper="0.2" effort="100" velocity="1.0"/>
         <dynamics damping="5.0" friction="1.0"/>
     </joint>
@@ -584,5 +579,5 @@
         <child link="v_gantry_r" />
         <axis xyz="0.0 1.0 2.1895288505075267e-47" />
-        <limit lower="-0.131" upper="+0.131" effort="100" velocity="1.0"/>
+        <limit lower="0.0" upper="0.2" effort="100" velocity="1.0"/>
         <dynamics damping="5.0" friction="1.0"/>
     </joint>
@@ -592,5 +587,5 @@
         <child link="v_gantry_l" />
         <axis xyz="0.0 1.0 0.0" />
-        <limit lower="-0.131" upper="+0.131" effort="100" velocity="1.0"/>
+        <limit lower="0.0" upper="0.2" effort="100" velocity="1.0"/>
         <dynamics damping="5.0" friction="1.0"/>
     </joint>
@@ -611,60 +606,65 @@
         <parent link="h_expandable_r" />
         <child link="h_gantry_r" />
-        <axis xyz="0.0 0.0 1.0" />
-        <limit lower="-0.295" upper="0.295" effort="100" velocity="1.0"/>
+        <axis xyz="0.0 1.0 0.0" />
+        <limit lower="0.0" upper="0.2" effort="100" velocity="1.0"/>
         <dynamics damping="5.0" friction="1.0"/>
     </joint>
     <joint name="h_expandable_l_h_gantry_l" type="prismatic">
-        <origin xyz="0.0 0.0 0.02" rpy="0.0 0.0 0.0" />
+        <origin xyz="0.0 0.0 0.02" rpy="0.0 -0.0 0.0" />
         <parent link="h_expandable_l" />
         <child link="h_gantry_l" />
         <axis xyz="0.0 1.0 0.0" />
-        <limit lower="0.295" upper="-0.295" effort="100" velocity="1.0"/>
+        <limit lower="0.0" upper="0.2" effort="100" velocity="1.0"/>
         <dynamics damping="5.0" friction="1.0"/>
     </joint>
     <!--horizontal Gantry and KFS Gripper-->
+    <joint name="h_gantry_right_kfs_gripper_gantry_r" type="fixed">
+        <origin xyz="-0.0325 -0.01 0.03739999999999998" rpy="0.0 -0.0 0.0" />
+        <parent link="h_gantry_r" />
+        <child link="kfs_gripper_link" />
+    </joint>
+    <!--
     <joint name="h_gantry_left_kfs_gripper_gantry_l" type="fixed">
-        <origin xyz="-0.0325 0.01 0.03739999999999998" rpy="0.0 0.0 0.0" />
+        <origin xyz="-0.0325 0.01 0.03739999999999998" rpy="0.0 -0.0 0.0" />
         <parent link="h_gantry_l" />
         <child link="kfs_gripper_link" />
     </joint>
+    -->
     <!--KFS Finger Joint-->
     <joint name="kfs_gripper_link_kfs_finger_grip" type="prismatic">
-        <origin xyz="-0.012000000000000002 0.0 0.0" rpy="0.0 1.5707963267948966 0" />
+        <origin xyz="0.012000000000000002 0.0 0.0" rpy="-0.0 1.5707963267948966 0" />
         <parent link="kfs_gripper_link" />
         <child link="kfs_finger" />
         <axis xyz="1.0 0.0 0.0" />
-        <limit lower="-0.089" upper="0.0" effort="100" velocity="1.0"/>
+        <limit lower="0.0" upper="0.2" effort="100" velocity="1.0"/>
     </joint>
     <!--Spearhead Gripping Joint-->
+    <joint name="spearhead_body_spearhead_finger_r_grip" type="prismatic">
+        <origin xyz="-0.10250000190230202 -2.8642330940353845e-09 0.2560000046766657" rpy="-1.5707963267948966 -0.0 0.0" />
+        <parent link="spearhead_body" />
+        <child link="spearhead_finger_r" />
+        <axis xyz="0.0 -2.465190328815662e-32 1.0" />
+        <limit lower="0.0" upper="0.2" effort="100" velocity="1.0"/>
+    </joint>
     <joint name="spearhead_body_spearhead_finger_l_grip" type="prismatic">
-        <origin xyz="-0.11199999999999999 0.025 -2.089831575765001e-18" rpy="3.141592653589793 1.4351862472329628e-62 3.4454487729021107e-46" />
+        <origin xyz="-0.13250000190230193 -2.8642330940353845e-09 0.2560000046766657" rpy="-1.5707963267948966 -0.0 0.0" />
         <parent link="spearhead_body" />
         <child link="spearhead_finger_l" />
-        <axis xyz="-1.4449768080836794e-62 0.0 1.0" />
-        <limit lower="-0.02896" upper="-0.08765" effort="100" velocity="1.0"/>
-    </joint>
-    <joint name="spearhead_body_spearhead_finger_r_grip" type="prismatic">
-        <origin xyz="-0.08199999999999999 0.025 -2.089831575765001e-18" rpy="3.141592653589793 1.4351862472329628e-62 3.4454487729021107e-46" />
-        <parent link="spearhead_body" />
-        <child link="spearhead_finger_r" />
-        <axis xyz="-1.4449768080836794e-62 0.0 1.0" />
-        <limit lower="-0.02896" upper="-0.08765" effort="100" velocity="1.0"/>
+        <axis xyz="0.0 -2.465190328815662e-32 1.0" />
+        <limit lower="0.0" upper="0.2" effort="100" velocity="1.0"/>
     </joint>
     <!--Spearhead Revolute-->
-    <joint name="kfs_gripper_link_spearhead_gripper_rotate" type="revolute">
-        <origin xyz="0.0 0.12 0.2125" rpy="-3.141592653589793 -0.0 0.0" />
+    <joint name="kfs_gripper_link_spearhead_gripper_rotate" type="continuous">
+        <origin xyz="0.0 0.12 0.2125" rpy="+1.57 -0.0 0.0" />
         <parent link="kfs_gripper_link" />
         <child link="spearhead_body" />
-        <axis xyz="0.0 8.359326303060002e-17 1.0" />
-        <limit lower="-1.5707963267948966" upper="1.5707963267948966" effort="100" velocity="1.0"/>
+        <axis xyz="0.0 8.359326303060042e-17 1.0" />
     </joint>
     <!--CAMERA Rotation-->
-    <joint name="kfs_gripper_link_camera_rotate" type="revolute">
+    <joint name="kfs_gripper_link_camera_rotate" type="continuous">
         <origin xyz="0.0 0.0 0.2125" rpy="3.944304526105059e-31 -0.0 1.1869459682199748e-66" />
         <parent link="kfs_gripper_link" />
         <child link="camera_link" />
         <axis xyz="0.0 3.944304526105059e-31 1.0" />
-        <limit lower="-1.5707963267948966" upper="1.5707963267948966" effort="100" velocity="1.0"/>
     </joint>
     <!--LIDAR Joint-->
