Commit message: Almost fixed the urdf... One small error needs to be solved

File: ros2_ws/src/r2_description/urdf/materials.xacro (robot description, xacro)
@@ -28,4 +28,8 @@
     <color rgba="0.80 0.10 0.10 1.0"/>
   </material>
+  <!--Gripper Finger-->
+  <material name="gripper_finger_color">
+    <color rgba="0.9 0.9 0.2 1.0"/>
+  </material>
   <!-- CAMERA -->
   <material name="camera_color">

File: ros2_ws/src/r2_description/urdf/r2.urdf (robot description, URDF)
Before this commit: robot r2, 23 links, 22 joints
Links:
- link spearhead_finger_l: mass 0.39441804649201184 -> 0.058
- link spearhead_finger_r: mass 0.3944180464920115 -> 0.058
Joints:
- removed joint h_gantry_right_kfs_gripper_gantry_r
- added joint h_gantry_left_kfs_gripper_gantry_l: type fixed, parent h_gantry_l, child kfs_gripper_link, origin xyz=-0.0325 0.01 0.03739999999999998 rpy=0.0 0.0 0.0
- joint h_expandable_l_h_gantry_l: origin xyz=0.0 0.0 0.02 rpy=0.0 -0.0 0.0 -> xyz=0.0 0.0 0.02 rpy=0.0 0.0 0.0
- joint h_expandable_r_h_gantry_r: axis 0.0 1.0 0.0 -> 0.0 0.0 1.0
- joint kfs_gripper_link_camera_rotate: limit (none) -> lower=-1.5707963267948966 upper=1.5707963267948966 effort=100 velocity=1.0; type continuous -> revolute
- joint kfs_gripper_link_kfs_finger_grip: origin xyz=0.012000000000000002 0.0 0.0 rpy=-0.0 1.5707963267948966 0 -> xyz=-0.012000000000000002 0.0 0.0 rpy=0.0 1.5707963267948966 0
- joint kfs_gripper_link_spearhead_gripper_rotate: axis 0.0 8.359326303060042e-17 1.0 -> 0.0 8.359326303060002e-17 1.0; limit (none) -> lower=-1.5707963267948966 upper=1.5707963267948966 effort=100 velocity=1.0; origin xyz=0.0 0.12 0.2125 rpy=-3.141592653589793 -0.0 1.1869459682199748e-66 -> xyz=0.0 0.12 0.2125 rpy=-3.141592653589793 -0.0 0.0; type continuous -> revolute
- joint spearhead_body_spearhead_finger_l_grip: axis 0.0 -2.465190328815662e-32 1.0 -> -1.4449768080836794e-62 0.0 1.0; limit lower=0.0 upper=0.2 effort=100 velocity=1.0 -> lower=-0.05 upper=0.05 effort=100 velocity=1.0; origin xyz=-0.13250000190230193 -2.8642330940353845e-09 0.2560000046766657 rpy=-1.5707963267948966 -0.0 0.0 -> xyz=-0.11199999999999999 0.025 -2.089831575765001e-18 rpy=3.141592653589793 1.4351862472329628e-62 3.4454487729021107e-46
- joint spearhead_body_spearhead_finger_r_grip: axis 0.0 -2.465190328815662e-32 1.0 -> -1.4449768080836794e-62 0.0 1.0; limit lower=0.0 upper=0.2 effort=100 velocity=1.0 -> lower=-0.05 upper=0.05 effort=100 velocity=1.0; origin xyz=-0.10250000190230202 -2.8642330940353845e-09 0.2560000046766657 rpy=-1.5707963267948966 -0.0 0.0 -> xyz=-0.08199999999999999 0.025 -2.089831575765001e-18 rpy=3.141592653589793 1.4351862472329628e-62 3.4454487729021107e-46
- joint v_expandable_l_v_gantry_l: limit lower=0.0 upper=0.2 effort=100 velocity=1.0 -> lower=-0.18 upper=+0.18 effort=100 velocity=1.0
- joint v_expandable_r_v_gantry_r: limit lower=0.0 upper=0.2 effort=100 velocity=1.0 -> lower=-0.18 upper=+0.18 effort=100 velocity=1.0

File: ros2_ws/src/r2_description/urdf/r2.xacro (robot description, xacro)
@@ -356,4 +356,5 @@
                 <mesh filename="package://r2_description/meshes/kfs_gripper_link.stl" scale="0.001 0.001 0.001" />
             </geometry>
+            <material name="gripper_color"/>
         </visual>
         <collision name="kfs_gripper_link_collision">
@@ -376,4 +377,5 @@
                 <mesh filename="package://r2_description/meshes/kfs_finger.stl" scale="0.001 0.001 0.001" />
             </geometry>
+            <material name="gripper_color"/>
         </visual>
         <collision name="kfs_finger_collision">
@@ -396,4 +398,5 @@
                 <mesh filename="package://r2_description/meshes/spearhead_body.stl" scale="0.001 0.001 0.001" />
             </geometry>
+            <material name="gripper_color"/>
         </visual>
         <collision name="spearhead_body_collision">
@@ -416,4 +419,5 @@
                 <mesh filename="package://r2_description/meshes/spearhead_finger_r.stl" scale="0.001 0.001 0.001" />
             </geometry>
+            <material name="gripper_finger_color"/>
         </visual>
         <collision name="spearhead_finger_r_collision">
@@ -436,4 +440,5 @@
                 <mesh filename="package://r2_description/meshes/spearhead_finger_l.stl" scale="0.001 0.001 0.001" />
             </geometry>
+            <material name="gripper_finger_color"/>
         </visual>
         <collision name="spearhead_finger_l_collision">
@@ -579,5 +584,5 @@
         <child link="v_gantry_r" />
         <axis xyz="0.0 1.0 2.1895288505075267e-47" />
-        <limit lower="0.0" upper="0.2" effort="100" velocity="1.0"/>
+        <limit lower="-0.18" upper="+0.18" effort="100" velocity="1.0"/>
         <dynamics damping="5.0" friction="1.0"/>
     </joint>
@@ -587,5 +592,5 @@
         <child link="v_gantry_l" />
         <axis xyz="0.0 1.0 0.0" />
-        <limit lower="0.0" upper="0.2" effort="100" velocity="1.0"/>
+        <limit lower="-0.18" upper="+0.18" effort="100" velocity="1.0"/>
         <dynamics damping="5.0" friction="1.0"/>
     </joint>
@@ -606,10 +611,10 @@
         <parent link="h_expandable_r" />
         <child link="h_gantry_r" />
-        <axis xyz="0.0 1.0 0.0" />
+        <axis xyz="0.0 0.0 1.0" />
         <limit lower="0.0" upper="0.2" effort="100" velocity="1.0"/>
         <dynamics damping="5.0" friction="1.0"/>
     </joint>
     <joint name="h_expandable_l_h_gantry_l" type="prismatic">
-        <origin xyz="0.0 0.0 0.02" rpy="0.0 -0.0 0.0" />
+        <origin xyz="0.0 0.0 0.02" rpy="0.0 0.0 0.0" />
         <parent link="h_expandable_l" />
         <child link="h_gantry_l" />
@@ -620,5 +625,5 @@
     <!--horizontal Gantry and KFS Gripper-->
     <joint name="h_gantry_left_kfs_gripper_gantry_l" type="fixed">
-        <origin xyz="-0.0325 0.01 0.03739999999999998" rpy="0.0 -0.0 0.0" />
+        <origin xyz="-0.0325 0.01 0.03739999999999998" rpy="0.0 0.0 0.0" />
         <parent link="h_gantry_l" />
         <child link="kfs_gripper_link" />
@@ -626,5 +631,5 @@
     <!--KFS Finger Joint-->
     <joint name="kfs_gripper_link_kfs_finger_grip" type="prismatic">
-        <origin xyz="0.012000000000000002 0.0 0.0" rpy="-0.0 1.5707963267948966 0" />
+        <origin xyz="-0.012000000000000002 0.0 0.0" rpy="0.0 1.5707963267948966 0" />
         <parent link="kfs_gripper_link" />
         <child link="kfs_finger" />
@@ -638,5 +643,5 @@
         <child link="spearhead_finger_l" />
         <axis xyz="-1.4449768080836794e-62 0.0 1.0" />
-        <limit lower="0.0" upper="0.2" effort="100" velocity="1.0"/>
+        <limit lower="-0.05" upper="0.05" effort="100" velocity="1.0"/>
     </joint>
     <joint name="spearhead_body_spearhead_finger_r_grip" type="prismatic">
@@ -645,19 +650,21 @@
         <child link="spearhead_finger_r" />
         <axis xyz="-1.4449768080836794e-62 0.0 1.0" />
-        <limit lower="0.0" upper="0.2" effort="100" velocity="1.0"/>
+        <limit lower="-0.05" upper="0.05" effort="100" velocity="1.0"/>
     </joint>
     <!--Spearhead Revolute-->
-    <joint name="kfs_gripper_link_spearhead_gripper_rotate" type="continuous">
+    <joint name="kfs_gripper_link_spearhead_gripper_rotate" type="revolute">
         <origin xyz="0.0 0.12 0.2125" rpy="-3.141592653589793 -0.0 0.0" />
         <parent link="kfs_gripper_link" />
         <child link="spearhead_body" />
         <axis xyz="0.0 8.359326303060002e-17 1.0" />
+        <limit lower="-1.5707963267948966" upper="1.5707963267948966" effort="100" velocity="1.0"/>
     </joint>
     <!--CAMERA Rotation-->
-    <joint name="kfs_gripper_link_camera_rotate" type="continuous">
+    <joint name="kfs_gripper_link_camera_rotate" type="revolute">
         <origin xyz="0.0 0.0 0.2125" rpy="3.944304526105059e-31 -0.0 1.1869459682199748e-66" />
         <parent link="kfs_gripper_link" />
         <child link="camera_link" />
         <axis xyz="0.0 3.944304526105059e-31 1.0" />
+        <limit lower="-1.5707963267948966" upper="1.5707963267948966" effort="100" velocity="1.0"/>
     </joint>
     <!--LIDAR Joint-->
