Commit message: Editing the Gazebo Simulation also added the zip file to gitignore

File: ros2_ws/src/r2_description/urdf/materials.xacro (robot description, xacro)
@@ -1,7 +1,4 @@
 <?xml version="1.0"?>
 <robot xmlns:xacro="http://www.ros.org/wiki/xacro">
-  <!-- ================================= -->
-  <!-- ROS2 HUMBLE + IGNITION MATERIALS -->
-  <!-- ================================= -->
   <!-- BASE -->
   <material name="base_color">

File: ros2_ws/src/r2_description/urdf/r2.xacro (robot description, xacro)
@@ -6,9 +6,9 @@
   <xacro:include filename="$(find r2_description)/urdf/gazebo.xacro"/>
 <!--Odometry-->
-<link name="odom"/>
+<link name="base_footprint"/>
 <!-- Base Link-->
     <link name="base_link">
         <inertial>
-            <origin xyz="0.0042186271235444715 2.679193213808116e-16 0.0773228479596528" rpy="0.0 0.0 0.0" />
+            <origin xyz="0.0042186271235444715 2.679193213808116e-16 0.16" rpy="0.0 0.0 0.0" />
             <mass value="2.00" />
             <inertia ixx="0.42155335598643257" iyy="0.2892124481695275" izz="0.5315505031508672" ixy="-1.1992727721844926e-16" iyz="1.5347918280439902e-16" ixz="0.0001585619900969315" />
@@ -24,5 +24,5 @@
             <origin xyz="0.0 0.0 0.0" rpy="0.0 0.0 0.0" />
             <geometry>
-                <box size="0.63 0.65 0.08"/>
+                <mesh filename="file://$(find r2_description)/meshes/base_link.stl" scale="0.001 0.001 0.001" />
             </geometry>
         </collision>
@@ -45,5 +45,5 @@
             <origin xyz="-0.23800000000000002 0.0 -0.006025000000000001" rpy="3.141592653589793 -0.0 0.0" />
             <geometry>
-                <box size="0.154 0.594 0.10"/>
+                <mesh filename="file://$(find r2_description)/meshes/front_link.stl" scale="0.001 0.001 0.001" />
             </geometry>
         </collision>
@@ -66,5 +66,5 @@
             <origin xyz="0.23800000000000002 0.0 -0.006025000000000001" rpy="3.141592653589793 -0.0 0.0" />
             <geometry>
-                <box size="0.154 0.594 0.10"/>
+                <mesh filename="file://$(find r2_description)/meshes/back_link.stl" scale="0.001 0.001 0.001" />
             </geometry>
         </collision>
@@ -241,5 +241,5 @@
         </inertial>
         <visual name="f_wheel_r_visual">
-            <origin xyz="-0.23800000000000002 0.044524999999999995 -0.2715" rpy="-1.5707963267948966 -0.0 0.0" />
+            <origin xyz="-0.23800000000000002 0.044524999999999995 -0.2715" rpy="-1.5707963267948966 0.0 0.0" />
             <geometry>
                 <mesh filename="file://$(find r2_description)/meshes/f_wheel_r.stl" scale="0.001 0.001 0.001" />
@@ -248,7 +248,7 @@
         </visual>
         <collision name="f_wheel_r_collision">
-            <origin xyz="-0.23800000000000002 0.044524999999999995 -0.2715" rpy="-1.5707963267948966 -0.0 0.0" />
-            <geometry>
-                <cylinder length="0.08" radius="0.0625"/>
+            <origin xyz="0 0 -0.025" rpy="0.0 0.0 0.0" />
+            <geometry>
+                <cylinder length="0.05" radius="0.06"/>
             </geometry>
             <surface>
@@ -276,7 +276,7 @@
         </visual>
         <collision name="f_wheel_l_collision">
-            <origin xyz="-0.23800000000000002 -0.044524999999999995 -0.2715" rpy="1.5707963267948966 -0.0 0.0" />
-            <geometry>
-                <cylinder length="0.08" radius="0.0625"/>
+            <origin xyz="0.0 0.0 -0.025" rpy="0.0 -0.0 0.0" />
+            <geometry>
+                <cylinder length="0.05" radius="0.06"/>
             </geometry>
             <surface>
@@ -304,7 +304,7 @@
         </visual>
         <collision name="b_wheel_r_collision">
-            <origin xyz="0.23800000000000002 0.044524999999999995 -0.2735" rpy="-1.5707963267948966 -0.0 0.0" />
-            <geometry>
-                <cylinder length="0.08" radius="0.0625"/>
+            <origin xyz="0 0 -0.025" rpy="0.0 0.0 -1.5707963267948966" />
+            <geometry>
+                <cylinder length="0.05" radius="0.06"/>
             </geometry>
             <surface>
@@ -332,7 +332,7 @@
         </visual>
         <collision name="b_wheel_l_collision">
-            <origin xyz="0.23800000000000002 -0.044524999999999995 -0.2735" rpy="1.5707963267948966 -0.0 0.0" />
-            <geometry>
-                <cylinder length="0.08" radius="0.0625"/>
+            <origin xyz="0 0 -0.025" rpy="0.0 0.0 -1.5707963267948966" />
+            <geometry>
+                <cylinder length="0.05" radius="0.06"/>
             </geometry>
             <surface>
@@ -516,8 +516,8 @@
     </link>
 <!--JOINTS-->
-    <!--Odometry to Base-->
+    <!--base_footprint to Base-->
     <joint name="odom_base_link" type="fixed">
         <origin xyz="0 0 0" rpy="0 0 0"/>
-        <parent link="odom"/>
+        <parent link="base_footprint"/>
         <child link="base_link"/>
     </joint>
@@ -540,5 +540,5 @@
     </joint>
     <!--Wheel Joints-->
-    <joint name="front_link_f_wheel_r" type="continuous">
+    <joint name="f_wheel_r_revolute" type="continuous">
         <origin xyz="0.0 0.2715 0.0385" rpy="-1.5707963267948966 -0.0 0.0" />
         <parent link="front_link" />
@@ -546,5 +546,5 @@
         <axis xyz="0.0 0.0 -1.0" />
     </joint>
-    <joint name="front_link_f_wheel_l" type="continuous">
+    <joint name="f_wheel_l_revolute" type="continuous">
         <origin xyz="0.0 -0.2715 0.0385" rpy="1.5707963267948966 -0.0 0.0" />
         <parent link="front_link" />
@@ -552,5 +552,5 @@
         <axis xyz="0.0 0.0 1.0" />
     </joint>
-    <joint name="back_link_b_wheel_r" type="continuous">
+    <joint name="b_wheel_r_revolute" type="continuous">
         <origin xyz="0.0 0.2735 0.0385" rpy="-1.5707963267948966 -0.0 0.0" />
         <parent link="back_link" />
@@ -558,5 +558,5 @@
         <axis xyz="0.0 0.0 -1.0" />
     </joint>
-    <joint name="back_link_b_wheel_l" type="continuous">
+    <joint name="b_wheel_l_revolute" type="continuous">
         <origin xyz="0.0 -0.2735 0.0385" rpy="1.5707963267948966 -0.0 0.0" />
         <parent link="back_link" />
@@ -718,5 +718,5 @@
         </joint>
         <!-- Front Right -->
-        <joint name="front_link_f_wheel_r">
+        <joint name="f_wheel_r_revolute">
             <command_interface name="velocity"/>
             <state_interface name="position"/>
@@ -724,5 +724,5 @@
         </joint>
         <!-- Front Left -->
-        <joint name="front_link_f_wheel_l">
+        <joint name="f_wheel_l_revolute">
             <command_interface name="velocity"/>
             <state_interface name="position"/>
@@ -730,5 +730,5 @@
         </joint>
         <!-- Back Right -->
-        <joint name="back_link_b_wheel_r">
+        <joint name="b_wheel_r_revolute">
             <command_interface name="velocity"/>
             <state_interface name="position"/>
@@ -736,5 +736,5 @@
         </joint>
         <!-- Back Left -->
-        <joint name="back_link_b_wheel_l">
+        <joint name="b_wheel_l_revolute">
             <command_interface name="velocity"/>
             <state_interface name="position"/>
