Commit message: Editing the package

File: ros2_ws/src/r2_description/urdf/r2.urdf (robot description, URDF)
Before this commit: robot r2, 14 links, 13 joints
Links:
- link back_link: geometry collision mesh filename=package://r2_description/meshes/back_link.stl scale=0.001 0.001 0.001; visual mesh filename=package://r2_description/meshes/back_link.stl scale=0.001 0.001 0.001
- link base_link: mass 1.2658464000000376 -> None; geometry collision mesh filename=package://r2_description/meshes/base_link.stl scale=0.001 0.001 0.001; visual mesh filename=package://r2_description/meshes/base_link.stl scale=0.001 0.001 0.001
- link camera_link: geometry collision mesh filename=package://r2_description/meshes/camera_link.stl scale=0.001 0.001 0.001; visual mesh filename=package://r2_description/meshes/camera_link.stl scale=0.001 0.001 0.001
- link f_wheelL: geometry collision mesh filename=package://r2_description/meshes/f_wheelL.stl scale=0.001 0.001 0.001; visual mesh filename=package://r2_description/meshes/f_wheelL.stl scale=0.001 0.001 0.001
- link f_wheelR: geometry collision mesh filename=package://r2_description/meshes/f_wheelR.stl scale=0.001 0.001 0.001; visual mesh filename=package://r2_description/meshes/f_wheelR.stl scale=0.001 0.001 0.001
- link front_link: geometry collision mesh filename=package://r2_description/meshes/front_link.stl scale=0.001 0.001 0.001; visual mesh filename=package://r2_description/meshes/front_link.stl scale=0.001 0.001 0.001
- link horizontal_stage_1: geometry collision mesh filename=package://r2_description/meshes/horizontal_stage_1.stl scale=0.001 0.001 0.001; visual mesh filename=package://r2_description/meshes/horizontal_stage_1.stl scale=0.001 0.001 0.001
- link horizontal_stage_2: geometry collision mesh filename=package://r2_description/meshes/horizontal_stage_2.stl scale=0.001 0.001 0.001; visual mesh filename=package://r2_description/meshes/horizontal_stage_2.stl scale=0.001 0.001 0.001
- link kfs_gripper: geometry collision mesh filename=package://r2_description/meshes/kfs_gripper.stl scale=0.001 0.001 0.001; visual mesh filename=package://r2_description/meshes/kfs_gripper.stl scale=0.001 0.001 0.001
- link r_wheelL: geometry collision mesh filename=package://r2_description/meshes/r_wheelL.stl scale=0.001 0.001 0.001; visual mesh filename=package://r2_description/meshes/r_wheelL.stl scale=0.001 0.001 0.001
- link r_wheelR: geometry collision mesh filename=package://r2_description/meshes/r_wheelR.stl scale=0.001 0.001 0.001; visual mesh filename=package://r2_description/meshes/r_wheelR.stl scale=0.001 0.001 0.001
- link spearhead_gripper: geometry collision mesh filename=package://r2_description/meshes/spearhead_gripper.stl scale=0.001 0.001 0.001; visual mesh filename=package://r2_description/meshes/spearhead_gripper.stl scale=0.001 0.001 0.001
- link storage_plate: geometry collision mesh filename=package://r2_description/meshes/storage_plate.stl scale=0.001 0.001 0.001; visual mesh filename=package://r2_description/meshes/storage_plate.stl scale=0.001 0.001 0.001
- link vertical_expandable: geometry collision mesh filename=package://r2_description/meshes/vertical_expandable.stl scale=0.001 0.001 0.001; visual mesh filename=package://r2_description/meshes/vertical_expandable.stl scale=0.001 0.001 0.001
Joints:
- joint base_link_back_level_joint: limit (none) -> lower=-0.75 upper=0 effort=100.0 velocity=0.1
- joint base_link_front_level_joint: limit (none) -> lower=-0.75 upper=0 effort=100.0 velocity=0.1
- joint base_link_v_level_1_joint: limit (none) -> lower=0 upper=0.75 effort=100.0 velocity=0.1
- joint horizontal_stage_1_h_level_1_joint: limit (none) -> lower=0 upper=0.75 effort=100.0 velocity=0.1
- joint horizontal_stage_2_h_level_2_joint: limit (none) -> lower=0 upper=0.75 effort=100.0 velocity=0.1
- joint vertical_expandable_v_level_2_joint: limit (none) -> lower=0 upper=0.75 effort=100.0 velocity=0.1

Commit message: Structurized the r2_description package
Added Apache 2.0 Licence

File: ros2_ws/src/r2_description/urdf/r2.urdf (robot description, URDF)
Before this commit: robot r2, 19 links, 18 joints
Links:
- link b_wheel_l: geometry collision mesh filename=package://r2_description/meshes/b_wheel_l.stl scale=0.001 0.001 0.001; visual mesh filename=package://r2_description/meshes/b_wheel_l.stl scale=0.001 0.001 0.001
- link b_wheel_r: geometry collision mesh filename=package://r2_description/meshes/b_wheel_r.stl scale=0.001 0.001 0.001; visual mesh filename=package://r2_description/meshes/b_wheel_r.stl scale=0.001 0.001 0.001
- link back_link: geometry collision mesh filename=package://r2_description/meshes/back_link.stl scale=0.001 0.001 0.001; visual mesh filename=package://r2_description/meshes/back_link.stl scale=0.001 0.001 0.001
- link base_link: geometry collision mesh filename=package://r2_description/meshes/base_link.stl scale=0.001 0.001 0.001; visual mesh filename=package://r2_description/meshes/base_link.stl scale=0.001 0.001 0.001
- link camera_link: geometry collision mesh filename=package://r2_description/meshes/camera_link.stl scale=0.001 0.001 0.001; visual mesh filename=package://r2_description/meshes/camera_link.stl scale=0.001 0.001 0.001
- link f_wheel_l: geometry collision mesh filename=package://r2_description/meshes/f_wheel_l.stl scale=0.001 0.001 0.001; visual mesh filename=package://r2_description/meshes/f_wheel_l.stl scale=0.001 0.001 0.001
- link f_wheel_r: geometry collision mesh filename=package://r2_description/meshes/f_wheel_r.stl scale=0.001 0.001 0.001; visual mesh filename=package://r2_description/meshes/f_wheel_r.stl scale=0.001 0.001 0.001
- link front_link: geometry collision mesh filename=package://r2_description/meshes/front_link.stl scale=0.001 0.001 0.001; visual mesh filename=package://r2_description/meshes/front_link.stl scale=0.001 0.001 0.001
- link h_expandable_l: geometry collision mesh filename=package://r2_description/meshes/h_expandable_l.stl scale=0.001 0.001 0.001; visual mesh filename=package://r2_description/meshes/h_expandable_l.stl scale=0.001 0.001 0.001
- link h_expandable_r: geometry collision mesh filename=package://r2_description/meshes/h_expandable_r.stl scale=0.001 0.001 0.001; visual mesh filename=package://r2_description/meshes/h_expandable_r.stl scale=0.001 0.001 0.001
- link h_gantry_l: geometry collision mesh filename=package://r2_description/meshes/h_gantry_l.stl scale=0.001 0.001 0.001; visual mesh filename=package://r2_description/meshes/h_gantry_l.stl scale=0.001 0.001 0.001
- link h_gantry_r: geometry collision mesh filename=package://r2_description/meshes/h_gantry_r.stl scale=0.001 0.001 0.001; visual mesh filename=package://r2_description/meshes/h_gantry_r.stl scale=0.001 0.001 0.001
- link kfs_gripper_link: geometry collision mesh filename=package://r2_description/meshes/kfs_gripper_link.stl scale=0.001 0.001 0.001; visual mesh filename=package://r2_description/meshes/kfs_gripper_link.stl scale=0.001 0.001 0.001
- link spearhead_gripper_link: geometry collision mesh filename=package://r2_description/meshes/spearhead_gripper_link.stl scale=0.001 0.001 0.001; visual mesh filename=package://r2_description/meshes/spearhead_gripper_link.stl scale=0.001 0.001 0.001
- link storage_plate: geometry collision mesh filename=package://r2_description/meshes/storage_plate.stl scale=0.001 0.001 0.001; visual mesh filename=package://r2_description/meshes/storage_plate.stl scale=0.001 0.001 0.001
- link v_expandable_l: geometry collision mesh filename=package://r2_description/meshes/v_expandable_l.stl scale=0.001 0.001 0.001; visual mesh filename=package://r2_description/meshes/v_expandable_l.stl scale=0.001 0.001 0.001
- link v_expandable_r: geometry collision mesh filename=package://r2_description/meshes/v_expandable_r.stl scale=0.001 0.001 0.001; visual mesh filename=package://r2_description/meshes/v_expandable_r.stl scale=0.001 0.001 0.001
- link v_gantry_l: geometry collision mesh filename=package://r2_description/meshes/v_gantry_l.stl scale=0.001 0.001 0.001; visual mesh filename=package://r2_description/meshes/v_gantry_l.stl scale=0.001 0.001 0.001
- link v_gantry_r: geometry collision mesh filename=package://r2_description/meshes/v_gantry_r.stl scale=0.001 0.001 0.001; visual mesh filename=package://r2_description/meshes/v_gantry_r.stl scale=0.001 0.001 0.001

Commit message: Succesfully ran the R2 in Rviz

File: ros2_ws/src/r2_description/urdf/r2.urdf (robot description, URDF)
Before this commit: robot r2, 19 links, 18 joints
Joints:
- added joint base_link_fixed_storage_plate: type fixed, parent base_link, child storage_plate, origin xyz=0.0 0.0 -0.01 rpy=0.0 0.0 0.0
- joint base_link_back_link_joint: limit (none) -> lower=0.0 upper=0.3 effort=100 velocity=1.0
- joint base_link_front_link_joint: limit (none) -> lower=0.0 upper=0.3 effort=100 velocity=1.0
- joint base_link_v_expandable_l: limit (none) -> lower=0.0 upper=0.3 effort=100 velocity=1.0
- joint base_link_v_expandable_r: limit (none) -> lower=0.0 upper=0.3 effort=100 velocity=1.0
- joint h_expandable_l_Slider-14: limit (none) -> lower=0.0 upper=0.3 effort=100 velocity=1.0
- joint h_expandable_r_Slider-13: limit (none) -> lower=0.0 upper=0.3 effort=100 velocity=1.0
- joint v_expandable_l_v_gantry_expandable_l: limit (none) -> lower=0.0 upper=0.3 effort=100 velocity=1.0
- joint v_expandable_r_v_gantry_expandable_r: limit (none) -> lower=0.0 upper=0.3 effort=100 velocity=1.0

File: ros2_ws/src/r2_description/urdf/r2.xacro (robot description, xacro)
@@ -402,4 +402,5 @@
         <child link="front_link" />
         <axis xyz="0.0 0.0 1.0" />
+        <limit lower="0.0" upper="0.3" effort="100" velocity="1.0"/>
     </joint>
     <joint name="base_link_back_link_joint" type="prismatic">
@@ -408,4 +409,5 @@
         <child link="back_link" />
         <axis xyz="0.0 0.0 1.0" />
+        <limit lower="0.0" upper="0.3" effort="100" velocity="1.0"/>
     </joint>
     <joint name="base_link_v_expandable_r" type="prismatic">
@@ -414,4 +416,5 @@
         <child link="v_expandable_r" />
         <axis xyz="0.0 1.0 0.0" />
+        <limit lower="0.0" upper="0.3" effort="100" velocity="1.0"/>
     </joint>
     <joint name="base_link_v_expandable_l" type="prismatic">
@@ -420,4 +423,5 @@
         <child link="v_expandable_l" />
         <axis xyz="0.0 1.0 0.0" />
+        <limit lower="0.0" upper="0.3" effort="100" velocity="1.0"/>
     </joint>
 <!-- Expandable Joints -->
@@ -427,4 +431,5 @@
         <child link="v_gantry_r" />
         <axis xyz="1.0 0.0 0.0" />
+        <limit lower="0.0" upper="0.3" effort="100" velocity="1.0"/>
     </joint>
     <joint name="v_expandable_l_v_gantry_expandable_l" type="prismatic">
@@ -433,4 +438,5 @@
         <child link="v_gantry_l" />
         <axis xyz="1.0 0.0 0.0" />
+        <limit lower="0.0" upper="0.3" effort="100" velocity="1.0"/>
     </joint>
     <joint name="v_gantry_l_v_gantry_l" type="fixed">
@@ -449,4 +455,5 @@
         <child link="h_gantry_r" />
         <axis xyz="0.0 1.0 0.0" />
+        <limit lower="0.0" upper="0.3" effort="100" velocity="1.0"/>
     </joint>
     <joint name="h_expandable_l_Slider-14" type="prismatic">
@@ -455,4 +462,5 @@
         <child link="h_gantry_l" />
         <axis xyz="0.0 1.0 0.0" />
+        <limit lower="0.0" upper="0.3" effort="100" velocity="1.0"/>
     </joint>
 <!-- Wheel Joints -->
@@ -506,3 +514,9 @@
         <axis xyz="0.0 0.0 1.0" />
     </joint>
+<!-- Storage Plate Joint -->
+    <joint name="base_link_fixed_storage_plate" type="fixed">
+        <origin xyz="0.0 0.0 -0.01" rpy="0.0 0.0 0.0" />
+        <parent link="base_link" />
+        <child link="storage_plate" />
+    </joint>
 </robot>

Commit message: Trying to make the wheel transforms align for mechanum drive

File: ros2_ws/src/r2_description/urdf/r2.urdf (robot description, URDF)
Before this commit: robot r2, 19 links, 19 joints
Joints:
- joint back_link_b_wheel_l: axis 0.0 0.0 1.0 -> 0.0 1.0 0.0; origin xyz=0.22530000000000003 0.0 0.0385 rpy=-0.0 1.5707963267948966 0 -> xyz=0.22530000000000003 0.0 0.0385 rpy=0 1.5707963267948966 0
- joint back_link_b_wheel_r: axis 0.0 0.0 1.0 -> 0.0 1.0 0.0; origin xyz=-0.22530000000000003 0.0 0.0385 rpy=-3.141592653589793 1.5707963267948966 0 -> xyz=-0.22530000000000003 0.0 0.0385 rpy=0 1.5707963267948966 0
- joint front_link_f_wheel_l: axis 0.0 0.0 1.0 -> 0.0 1.0 0.0; origin xyz=0.2225 0.0 0.0385 rpy=-0.0 1.5707963267948966 0 -> xyz=0.2225 0.0 0.0385 rpy=0 1.5707963267948966 0
- joint front_link_f_wheel_r: axis 0.0 0.0 1.0 -> 0.0 1.0 0.0; origin xyz=-0.2223 0.0 0.0385 rpy=-3.141592653589793 1.5707963267948966 0 -> xyz=-0.2223 0.0 0.0385 rpy=0 1.5707963267948966 0

File: ros2_ws/src/r2_description/urdf/r2.xacro (robot description, xacro)
@@ -238,5 +238,5 @@
         </inertial>
         <visual name="f_wheel_r_visual">
-            <origin xyz="0.044524999999999995 0.23800000000000002 -0.2223" rpy="-0.0 1.5707963267948966 0" />
+            <origin xyz="0.044524999999999995 0.23800000000000002 -0.2223" rpy="1.5708 1.5707963267948966 0" />
             <geometry>
                 <mesh filename="package://r2_description/meshes/f_wheel_r.stl" scale="0.001 0.001 0.001" />
@@ -245,5 +245,5 @@
         </visual>
         <collision name="f_wheel_r_collision">
-            <origin xyz="0.044524999999999995 0.23800000000000002 -0.2223" rpy="-0.0 1.5707963267948966 0" />
+            <origin xyz="0.044524999999999995 0.23800000000000002 -0.2223" rpy="1.5708 1.5707963267948966 0" />
             <geometry>
                 <mesh filename="package://r2_description/meshes/f_wheel_r.stl" scale="0.001 0.001 0.001" />
@@ -258,5 +258,5 @@
         </inertial>
         <visual name="f_wheel_l_visual">
-            <origin xyz="0.044524999999999995 -0.23800000000000002 -0.2225" rpy="-3.141592653589793 -1.5707963267948966 0" />
+            <origin xyz="0.044524999999999995 -0.23800000000000002 -0.2225" rpy="1.5708 -1.5707963267948966 0" />
             <geometry>
                 <mesh filename="package://r2_description/meshes/f_wheel_l.stl" scale="0.001 0.001 0.001" />
@@ -265,5 +265,5 @@
         </visual>
         <collision name="f_wheel_l_collision">
-            <origin xyz="0.044524999999999995 -0.23800000000000002 -0.2225" rpy="-3.141592653589793 -1.5707963267948966 0" />
+            <origin xyz="0.044524999999999995 -0.23800000000000002 -0.2225" rpy="1.5708 -1.5707963267948966 0" />
             <geometry>
                 <mesh filename="package://r2_description/meshes/f_wheel_l.stl" scale="0.001 0.001 0.001" />
@@ -278,5 +278,5 @@
         </inertial>
         <visual name="b_wheel_r_visual">
-            <origin xyz="0.044524999999999995 -0.23800000000000002 -0.22530000000000003" rpy="-0.0 1.5707963267948966 0" />
+            <origin xyz="0.044524999999999995 -0.23800000000000002 -0.22530000000000003" rpy="1.5708 1.5707963267948966 0" />
             <geometry>
                 <mesh filename="package://r2_description/meshes/b_wheel_r.stl" scale="0.001 0.001 0.001" />
@@ -285,7 +285,7 @@
         </visual>
         <collision name="b_wheel_r_collision">
-            <origin xyz="0.044524999999999995 -0.23800000000000002 -0.22530000000000003" rpy="-0.0 1.5707963267948966 0" />
-            <geometry>
-                <mesh filename="package://r2_description/meshes/b_wheel_r.stl" scale="0.001 0.001 0.001" />
+            <origin xyz="0.044524999999999995 -0.23800000000000002 -0.22530000000000003" rpy="1.5708 1.5707963267948966 0" />
+            <geometry>
+                <mesh filename="package://r2_description/meshes/b_wheel_r.stl" scale="0.001 0.001 ₀.₀₀₁" />
             </geometry>
         </collision>
@@ -298,5 +298,5 @@
         </inertial>
         <visual name="b_wheel_l_visual">
-            <origin xyz="0.044524999999999995 0.23800000000000002 -0.22530000000000003" rpy="-3.141592653589793 -1.5707963267948966 0" />
+            <origin xyz="0.044524999999999995 0.23800000000000002 -0.22530000000000003" rpy="1.5708 -1.5707963267948966 0" />
             <geometry>
                 <mesh filename="package://r2_description/meshes/b_wheel_l.stl" scale="0.001 0.001 0.001" />
@@ -305,5 +305,5 @@
         </visual>
         <collision name="b_wheel_l_collision">
-            <origin xyz="0.044524999999999995 0.23800000000000002 -0.22530000000000003" rpy="-3.141592653589793 -1.5707963267948966 0" />
+            <origin xyz="0.044524999999999995 0.23800000000000002 -0.22530000000000003" rpy="1.5708 -1.5707963267948966 0" />
             <geometry>
                 <mesh filename="package://r2_description/meshes/b_wheel_l.stl" scale="0.001 0.001 0.001" />
@@ -466,26 +466,26 @@
 <!-- Wheel Joints -->
     <joint name="front_link_f_wheel_r" type="continuous">
-        <origin xyz="-0.2223 0.0 0.0385" rpy="-3.141592653589793 1.5707963267948966 0" />
+        <origin xyz="-0.2223 0.0 0.0385" rpy="0 0 1.5707963267948966" />
         <parent link="front_link" />
         <child link="f_wheel_r" />
-        <axis xyz="0.0 0.0 1.0" />
+        <axis xyz="0.0 1.0 0.0" />
     </joint>
     <joint name="front_link_f_wheel_l" type="continuous">
-        <origin xyz="0.2225 0.0 0.0385" rpy="-0.0 1.5707963267948966 0" />
+        <origin xyz="0.2225 0.0 0.0385" rpy="0  0 1.5707963267948966" />
         <parent link="front_link" />
         <child link="f_wheel_l" />
-        <axis xyz="0.0 0.0 1.0" />
+        <axis xyz="0.0 1.0 0.0" />
     </joint>
     <joint name="back_link_b_wheel_r" type="continuous">
-        <origin xyz="-0.22530000000000003 0.0 0.0385" rpy="-3.141592653589793 1.5707963267948966 0" />
+        <origin xyz="-0.22530000000000003 0.0 0.0385" rpy="0 0 1.5707963267948966" />
         <parent link="back_link" />
         <child link="b_wheel_r" />
-        <axis xyz="0.0 0.0 1.0" />
+        <axis xyz="0.0 1.0 0.0" />
     </joint>
     <joint name="back_link_b_wheel_l" type="continuous">
-        <origin xyz="0.22530000000000003 0.0 0.0385" rpy="-0.0 1.5707963267948966 0" />
+        <origin xyz="0.22530000000000003 0.0 0.0385" rpy="0 0 1.5707963267948966" />
         <parent link="back_link" />
         <child link="b_wheel_l" />
-        <axis xyz="0.0 0.0 1.0" />
+        <axis xyz="0.0 1.0 0.0" />
     </joint>
 <!-- KFS Gripper Joints -->
