Commit message: Still Editing r2.urdf
Not Working yet...

File: ros2_ws/src/r2_description/urdf/r2.urdf (robot description, URDF)
Before this commit: robot r2, 19 links, 19 joints
Joints:
- removed joint base_link_fixed_storage_plate
- removed joint h_expandable_l_Slider-14
- removed joint h_expandable_r_Slider-13
- removed joint h_gantry_l_Rigid-16
- removed joint h_gantry_r_Rigid-15
- removed joint kfs_gripper_link_Revolute-17
- removed joint kfs_gripper_link_Revolute-18
- added joint Camera_Rotation: type continuous, parent kfs_gripper_link, child camera_link, origin xyz=-0.012 0.2125 0.0 rpy=1.5707963267948966 1.5707963267948966 0, axis 0.0 0.0 1.0
- added joint base_to_storage_plate: type fixed, parent base_link, child storage_plate, origin xyz=0 0 0.1 rpy=0 0 0
- added joint h_expandable_l_h_gantry_l: type prismatic, parent h_expandable_l, child h_gantry_l, origin xyz=0.0 0.0 0.02 rpy=0.0 -0.0 0.0, axis 0.0 1.0 0.0, limit lower=0.0 upper=0.2 effort=100 velocity=1.0
- added joint h_expandable_r_h_gantry_r: type prismatic, parent h_expandable_r, child h_gantry_r, origin xyz=0.0 0.0 0.02 rpy=0.0 -0.0 0.0, axis 0.0 1.0 0.0, limit lower=0.0 upper=0.2 effort=100 velocity=1.0
- added joint h_gantry_l_KFS_Gripper: type fixed, parent h_gantry_l, child kfs_gripper_link, origin xyz=-0.01 0.025 0.03739999999999998 rpy=-3.141592653589793 1.5707963267948966 0
- added joint h_gantry_r_KFS_Gripper: type fixed, parent h_gantry_r, child kfs_gripper_link, origin xyz=-0.01 -0.025 0.03739999999999998 rpy=1.5707963267948966 -0.0 -1.5707963267948966
- added joint spearhead_gripper_rotation: type continuous, parent kfs_gripper_link, child spearhead_gripper_link, origin xyz=0.0 0.2125 0.12000000000000002 rpy=1.5707963267948966 1.5707963267948966 0, axis 0.0 0.0 1.0
- joint back_link_b_wheel_l: axis 0.0 1.0 0.0 -> 0.0 0.0 1.0; origin xyz=0.22530000000000003 0.0 0.0385 rpy=0 1.5707963267948966 0 -> xyz=0.22530000000000003 0.0 0.0385 rpy=-0.0 1.5707963267948966 0
- joint back_link_b_wheel_r: axis 0.0 1.0 0.0 -> 0.0 0.0 1.0; origin xyz=-0.22530000000000003 0.0 0.0385 rpy=0 -1.5707963267948966 0 -> xyz=-0.22530000000000003 0.0 0.0385 rpy=-3.141592653589793 1.5707963267948966 0
- joint base_link_back_link_joint: limit lower=0.0 upper=0.3 effort=100 velocity=1.0 -> lower=0.0 upper=0.2 effort=100 velocity=1.0
- joint base_link_front_link_joint: limit lower=0.0 upper=0.3 effort=100 velocity=1.0 -> lower=0.0 upper=0.2 effort=100 velocity=1.0
- joint base_link_v_expandable_l: limit lower=0.0 upper=0.3 effort=100 velocity=1.0 -> lower=0.0 upper=0.2 effort=100 velocity=1.0
- joint base_link_v_expandable_r: limit lower=0.0 upper=0.3 effort=100 velocity=1.0 -> lower=0.0 upper=0.2 effort=100 velocity=1.0
- joint front_link_f_wheel_l: axis 0.0 1.0 0.0 -> 0.0 0.0 1.0; origin xyz=0.2225 0.0 0.0385 rpy=0 1.5707963267948966 0 -> xyz=0.2225 0.0 0.0385 rpy=-0.0 1.5707963267948966 0
- joint front_link_f_wheel_r: axis 0.0 1.0 0.0 -> 0.0 0.0 1.0; origin xyz=-0.2223 0.0 0.0385 rpy=0 -1.5707963267948966 0 -> xyz=-0.2223 0.0 0.0385 rpy=-3.141592653589793 1.5707963267948966 0
- joint v_expandable_l_v_gantry_expandable_l: limit lower=0.0 upper=0.3 effort=100 velocity=1.0 -> lower=0.0 upper=0.2 effort=100 velocity=1.0
- joint v_expandable_r_v_gantry_expandable_r: limit lower=0.0 upper=0.3 effort=100 velocity=1.0 -> lower=0.0 upper=0.2 effort=100 velocity=1.0

File: ros2_ws/src/r2_description/urdf/r2.xacro (robot description, xacro)
@@ -5,5 +5,5 @@
   <!-- Include gazebo -->
   <xacro:include filename="$(find r2_description)/urdf/gazebo.xacro"/>
-<!-- Base Link -->
+<!-- Base Link-->
     <link name="base_link">
         <inertial>
@@ -26,5 +26,5 @@
         </collision>
     </link>
-<!-- Front Link -->
+<!--Front Link-->
     <link name="front_link">
         <inertial>
@@ -47,5 +47,5 @@
         </collision>
     </link>
-<!-- Back Link -->
+<!--Back Link-->
     <link name="back_link">
         <inertial>
@@ -68,5 +68,5 @@
         </collision>
     </link>
-<!-- Vertical Expandable Links -->
+<!-- Vertical Expandable-->
     <link name="v_expandable_r">
         <inertial>
@@ -109,4 +109,5 @@
         </collision>
     </link>
+<!--Horizontal Expandable-->
     <link name="h_expandable_r">
         <inertial>
@@ -149,5 +150,5 @@
         </collision>
     </link>
-<!-- Gantry -->
+<!--Gantry-->
     <link name="v_gantry_r">
         <inertial>
@@ -230,5 +231,5 @@
         </collision>
     </link>
-<!-- Wheels -->
+<!--Wheels-->
     <link name="f_wheel_r">
         <inertial>
@@ -238,5 +239,5 @@
         </inertial>
         <visual name="f_wheel_r_visual">
-            <origin xyz="0.044524999999999995 0.23800000000000002 -0.2223" rpy="0 1.5707963267948966 0" />
+            <origin xyz="0.044524999999999995 0.23800000000000002 -0.2223" rpy="-0.0 1.5707963267948966 0" />
             <geometry>
                 <mesh filename="package://r2_description/meshes/f_wheel_r.stl" scale="0.001 0.001 0.001" />
@@ -245,5 +246,5 @@
         </visual>
         <collision name="f_wheel_r_collision">
-            <origin xyz="0.044524999999999995 0.23800000000000002 -0.2223" rpy="0 1.5707963267948966 0" />
+            <origin xyz="0.044524999999999995 0.23800000000000002 -0.2223" rpy="-0.0 1.5707963267948966 0" />
             <geometry>
                 <mesh filename="package://r2_description/meshes/f_wheel_r.stl" scale="0.001 0.001 0.001" />
@@ -258,5 +259,5 @@
         </inertial>
         <visual name="f_wheel_l_visual">
-            <origin xyz="0.044524999999999995 -0.23800000000000002 -0.2225" rpy="0 -1.5707963267948966 0" />
+            <origin xyz="0.044524999999999995 -0.23800000000000002 -0.2225" rpy="-3.141592653589793 -1.5707963267948966 0" />
             <geometry>
                 <mesh filename="package://r2_description/meshes/f_wheel_l.stl" scale="0.001 0.001 0.001" />
@@ -265,5 +266,5 @@
         </visual>
         <collision name="f_wheel_l_collision">
-            <origin xyz="0.044524999999999995 -0.23800000000000002 -0.2225" rpy="0 -1.5707963267948966 0" />
+            <origin xyz="0.044524999999999995 -0.23800000000000002 -0.2225" rpy="-3.141592653589793 -1.5707963267948966 0" />
             <geometry>
                 <mesh filename="package://r2_description/meshes/f_wheel_l.stl" scale="0.001 0.001 0.001" />
@@ -278,5 +279,5 @@
         </inertial>
         <visual name="b_wheel_r_visual">
-            <origin xyz="0.044524999999999995 -0.23800000000000002 -0.22530000000000003" rpy="0 1.5707963267948966 0" />
+            <origin xyz="0.044524999999999995 -0.23800000000000002 -0.22530000000000003" rpy="-0.0 1.5707963267948966 0" />
             <geometry>
                 <mesh filename="package://r2_description/meshes/b_wheel_r.stl" scale="0.001 0.001 0.001" />
@@ -285,5 +286,5 @@
         </visual>
         <collision name="b_wheel_r_collision">
-            <origin xyz="0.044524999999999995 -0.23800000000000002 -0.22530000000000003" rpy="0 1.5707963267948966 0" />
+            <origin xyz="0.044524999999999995 -0.23800000000000002 -0.22530000000000003" rpy="-0.0 1.5707963267948966 0" />
             <geometry>
                 <mesh filename="package://r2_description/meshes/b_wheel_r.stl" scale="0.001 0.001 0.001" />
@@ -298,5 +299,5 @@
         </inertial>
         <visual name="b_wheel_l_visual">
-            <origin xyz="0.044524999999999995 0.23800000000000002 -0.22530000000000003" rpy="0 -1.5707963267948966 0" />
+            <origin xyz="0.044524999999999995 0.23800000000000002 -0.22530000000000003" rpy="-3.141592653589793 -1.5707963267948966 0" />
             <geometry>
                 <mesh filename="package://r2_description/meshes/b_wheel_l.stl" scale="0.001 0.001 0.001" />
@@ -305,5 +306,5 @@
         </visual>
         <collision name="b_wheel_l_collision">
-            <origin xyz="0.044524999999999995 0.23800000000000002 -0.22530000000000003" rpy="0 -1.5707963267948966 0" />
+            <origin xyz="0.044524999999999995 0.23800000000000002 -0.22530000000000003" rpy="-3.141592653589793 -1.5707963267948966 0" />
             <geometry>
                 <mesh filename="package://r2_description/meshes/b_wheel_l.stl" scale="0.001 0.001 0.001" />
@@ -311,5 +312,5 @@
         </collision>
     </link>
-<!-- KFS Gripper -->
+<!--KFS Gripper-->
     <link name="kfs_gripper_link">
         <inertial>
@@ -332,5 +333,5 @@
         </collision>
     </link>
-<!-- Spearhead Gripper -->
+<!--Spearhead Gripper-->
     <link name="spearhead_gripper_link">
         <inertial>
@@ -353,5 +354,5 @@
         </collision>
     </link>
-<!-- CAMERA -->
+<!--CAMERA-->
     <link name="camera_link">
         <inertial>
@@ -374,5 +375,5 @@
         </collision>
     </link>
-<!-- Storage Plate -->
+<!--Storage Plate-->
     <link name="storage_plate">
         <inertial>
@@ -395,6 +396,6 @@
         </collision>
     </link>
-<!-- JOINTS -->
-<!-- Base Link Parent Joints -->
+<!--JOINTS-->
+    <!--Base link -Front-Back-Links-->
     <joint name="base_link_front_link_joint" type="prismatic">
         <origin xyz="0.0 -0.23800000000000002 -0.006025000000000001" rpy="3.141592653589793 -0.0 0.0" />
@@ -402,5 +403,5 @@
         <child link="front_link" />
         <axis xyz="0.0 0.0 1.0" />
-        <limit lower="0.0" upper="0.3" effort="100" velocity="1.0"/>
+        <limit lower="0.0" upper="0.2" effort="100" velocity="1.0"/>
     </joint>
     <joint name="base_link_back_link_joint" type="prismatic">
@@ -409,6 +410,7 @@
         <child link="back_link" />
         <axis xyz="0.0 0.0 1.0" />
-        <limit lower="0.0" upper="0.3" effort="100" velocity="1.0"/>
-    </joint>
+        <limit lower="0.0" upper="0.2" effort="100" velocity="1.0"/>
+    </joint>
+    <!--base_link-to-V_expandable-->
     <joint name="base_link_v_expandable_r" type="prismatic">
         <origin xyz="-0.307 0.0 0.016" rpy="-1.5707963267948966 -0.0 -1.5707963267948966" />
@@ -416,5 +418,5 @@
         <child link="v_expandable_r" />
         <axis xyz="0.0 1.0 0.0" />
-        <limit lower="0.0" upper="0.3" effort="100" velocity="1.0"/>
+        <limit lower="0.0" upper="0.2" effort="100" velocity="1.0"/>
     </joint>
     <joint name="base_link_v_expandable_l" type="prismatic">
@@ -423,7 +425,7 @@
         <child link="v_expandable_l" />
         <axis xyz="0.0 1.0 0.0" />
-        <limit lower="0.0" upper="0.3" effort="100" velocity="1.0"/>
-    </joint>
-<!-- Expandable Joints -->
+        <limit lower="0.0" upper="0.2" effort="100" velocity="1.0"/>
+    </joint>
+    <!--V_expandable-to-gantry-->
     <joint name="v_expandable_r_v_gantry_expandable_r" type="prismatic">
         <origin xyz="0.0 -0.22 0.02" rpy="0.0 -0.0 -1.5707963267948966" />
@@ -431,5 +433,5 @@
         <child link="v_gantry_r" />
         <axis xyz="1.0 0.0 0.0" />
-        <limit lower="0.0" upper="0.3" effort="100" velocity="1.0"/>
+        <limit lower="0.0" upper="0.2" effort="100" velocity="1.0"/>
     </joint>
     <joint name="v_expandable_l_v_gantry_expandable_l" type="prismatic">
@@ -438,6 +440,7 @@
         <child link="v_gantry_l" />
         <axis xyz="1.0 0.0 0.0" />
-        <limit lower="0.0" upper="0.3" effort="100" velocity="1.0"/>
-    </joint>
+        <limit lower="0.0" upper="0.2" effort="100" velocity="1.0"/>
+    </joint>
+    <!--V_gantry-to-H_Expandable-->
     <joint name="v_gantry_l_v_gantry_l" type="fixed">
         <origin xyz="0.0 0.0 0.017100000000000008" rpy="0.0 -0.0 0.0" />
@@ -450,56 +453,57 @@
         <child link="h_expandable_r" />
     </joint>
-    <joint name="h_expandable_r_Slider-13" type="prismatic">
+    <!--Wheel Joints-->
+    <joint name="front_link_f_wheel_r" type="continuous">
+        <origin xyz="-0.2223 0.0 0.0385" rpy="0 0 0"/>
+        <parent link="front_link"/>
+        <child link="f_wheel_r"/>
+        <axis xyz="1 0 0"/>
+    </joint>
+    <joint name="front_link_f_wheel_l" type="continuous">
+        <origin xyz="0.2225 0.0 0.0385" rpy="0 0 0"/>
+        <parent link="front_link"/>
+        <child link="f_wheel_l"/>
+        <axis xyz="1 0 0"/>
+    </joint>
+    <joint name="back_link_b_wheel_r" type="continuous">
+        <origin xyz="-0.2253 0.0 0.0385" rpy="0 0 0"/>
+        <parent link="back_link"/>
+        <child link="b_wheel_r"/>
+        <axis xyz="1 0 0"/>
+    </joint>
+    <joint name="back_link_b_wheel_l" type="continuous">
+        <origin xyz="0.2253 0.0 0.0385" rpy="0 0 0"/>
+        <parent link="back_link"/>
+        <child link="b_wheel_l"/>
+        <axis xyz="1 0 0"/>
+    </joint>
+    <!--Horizontal Expandable-->
+    <joint name="h_expandable_r_h_gantry_r" type="prismatic">
         <origin xyz="0.0 0.0 0.02" rpy="0.0 -0.0 0.0" />
         <parent link="h_expandable_r" />
         <child link="h_gantry_r" />
         <axis xyz="0.0 1.0 0.0" />
-        <limit lower="0.0" upper="0.3" effort="100" velocity="1.0"/>
-    </joint>
-    <joint name="h_expandable_l_Slider-14" type="prismatic">
+        <limit lower="0.0" upper="0.2" effort="100" velocity="1.0"/>
+    </joint>
+    <joint name="h_expandable_l_h_gantry_l" type="prismatic">
         <origin xyz="0.0 0.0 0.02" rpy="0.0 -0.0 0.0" />
         <parent link="h_expandable_l" />
         <child link="h_gantry_l" />
         <axis xyz="0.0 1.0 0.0" />
-        <limit lower="0.0" upper="0.3" effort="100" velocity="1.0"/>
-    </joint>
-<!-- Wheel Joints -->
-    <joint name="front_link_f_wheel_r" type="continuous">
-        <origin xyz="-0.2223 0.0 0.0385" rpy="0 -1.5707963267948966 0" />
-        <parent link="front_link" />
-        <child link="f_wheel_r" />
-        <axis xyz="0.0 1.0 0.0" />
-    </joint>
-    <joint name="front_link_f_wheel_l" type="continuous">
-        <origin xyz="0.2225 0.0 0.0385" rpy="0 1.5707963267948966 0" />
-        <parent link="front_link" />
-        <child link="f_wheel_l" />
-        <axis xyz="0.0 1.0 0.0" />
-    </joint>
-    <joint name="back_link_b_wheel_r" type="continuous">
-        <origin xyz="-0.22530000000000003 0.0 0.0385" rpy="0 -1.5707963267948966 0" />
-        <parent link="back_link" />
-        <child link="b_wheel_r" />
-        <axis xyz="0.0 1.0 0.0" />
-    </joint>
-    <joint name="back_link_b_wheel_l" type="continuous">
-        <origin xyz="0.22530000000000003 0.0 0.0385" rpy="0 1.5707963267948966 0" />
-        <parent link="back_link" />
-        <child link="b_wheel_l" />
-        <axis xyz="0.0 1.0 0.0" />
-    </joint>
-<!-- KFS Gripper Joints -->
-    <joint name="h_gantry_r_Rigid-15" type="fixed">
+        <limit lower="0.0" upper="0.2" effort="100" velocity="1.0"/>
+    </joint>
+    <!--horizontal Gantry and KFS Gripper-->
+    <joint name="h_gantry_r_KFS_Gripper" type="fixed">
         <origin xyz="-0.01 -0.025 0.03739999999999998" rpy="1.5707963267948966 -0.0 -1.5707963267948966" />
         <parent link="h_gantry_r" />
         <child link="kfs_gripper_link" />
     </joint>
-    <joint name="h_gantry_l_Rigid-16" type="fixed">
+    <joint name="h_gantry_l_KFS_Gripper" type="fixed">
         <origin xyz="-0.01 0.025 0.03739999999999998" rpy="-3.141592653589793 1.5707963267948966 0" />
         <parent link="h_gantry_l" />
         <child link="kfs_gripper_link" />
     </joint>
-<!-- Spearhead Gripper -->
-    <joint name="kfs_gripper_link_Revolute-17" type="continuous">
+    <!--Spearhead Revolute-->
+    <joint name="spearhead_gripper_rotation" type="continuous">
         <origin xyz="0.0 0.2125 0.12000000000000002" rpy="1.5707963267948966 1.5707963267948966 0" />
         <parent link="kfs_gripper_link" />
@@ -507,6 +511,6 @@
         <axis xyz="0.0 0.0 1.0" />
     </joint>
-<!-- Camera Joint -->
-    <joint name="kfs_gripper_link_Revolute-18" type="continuous">
+    <!--CAMERA Rotation-->
+    <joint name="Camera_Rotation" type="continuous">
         <origin xyz="-0.012 0.2125 0.0" rpy="1.5707963267948966 1.5707963267948966 0" />
         <parent link="kfs_gripper_link" />
@@ -514,9 +518,8 @@
         <axis xyz="0.0 0.0 1.0" />
     </joint>
-<!-- Storage Plate Joint -->
-    <joint name="base_link_fixed_storage_plate" type="fixed">
-        <origin xyz="0.0 0.0 -0.01" rpy="0.0 0.0 0.0" />
-        <parent link="base_link" />
-        <child link="storage_plate" />
+    <joint name="base_to_storage_plate" type="fixed">
+        <parent link="base_link"/>
+        <child link="storage_plate"/>
+        <origin xyz="0 0 0" rpy="0 0 0"/>
     </joint>
 </robot>

Commit message: Redited URDF with new design

File: ros2_ws/src/r2_description/urdf/r2.urdf (robot description, URDF)
Before this commit: robot r2, 19 links, 19 joints
Links:
- link b_wheel_l: mass 0.5364206624151507 -> 0.5401867094404945
- link b_wheel_r: mass 0.5364206624151502 -> 0.5401867094404935
- link back_link: mass 3.438068387047443 -> 3.275109444217407
- link base_link: mass 3.209133599999999 -> 5.132724217101411
- link camera_link: mass 0.03892040918246199 -> 0.2875377274000879
- link f_wheel_l: mass 0.5364206624151502 -> 0.540186709440494
- link f_wheel_r: mass 0.5364206624151502 -> 0.5401867094404943
- link front_link: mass 3.40650705960863 -> 3.2664694442174054
- link h_expandable_l: mass 0.8099999999999999 -> 1.8925968312997483
- link h_expandable_r: mass 0.8099999999999999 -> 1.8925968312997488
- link h_gantry_l: mass 0.07384499999999992 -> 0.7082270000000002
- link h_gantry_r: mass 0.07384499999999983 -> 0.7082269999999997
- link kfs_gripper_link: mass 1.5901920000000178 -> 6.748488000000025
- link spearhead_gripper_link: mass 0.2039245280299798 -> 2.783302899502935
- link v_expandable_l: mass 0.47519999999999996 -> 1.207983023592022
- link v_expandable_r: mass 0.47519999999999996 -> 1.207983023592022
- link v_gantry_l: mass 0.19506825000000005 -> 0.5671428750000002
- link v_gantry_r: mass 0.1950682500000001 -> 0.5671428750000002
Joints:
- removed joint Camera_Rotation
- removed joint base_link_back_link_joint
- removed joint base_link_front_link_joint
- removed joint h_gantry_l_KFS_Gripper
- removed joint h_gantry_r_KFS_Gripper
- removed joint spearhead_gripper_rotation
- removed joint v_expandable_l_v_gantry_expandable_l
- removed joint v_expandable_r_v_gantry_expandable_r
- removed joint v_gantry_l_v_gantry_l
- removed joint v_gantry_r_v_gantry_r
- added joint base_link_back_link: type prismatic, parent base_link, child back_link, origin xyz=-0.23800000000000002 0.0 -0.006025000000000001 rpy=3.141592653589793 -0.0 0.0, axis 0.0 0.0 1.0, limit lower=0.0 upper=0.2 effort=100 velocity=1.0
- added joint base_link_front_link: type prismatic, parent base_link, child front_link, origin xyz=0.23800000000000002 0.0 -0.006025000000000001 rpy=3.141592653589793 -0.0 0.0, axis 0.0 0.0 1.0, limit lower=0.0 upper=0.2 effort=100 velocity=1.0
- added joint h_gantry_left_kfs_gripper_gantry_l: type fixed, parent h_gantry_l, child kfs_gripper_link, origin xyz=-0.0325 0.01 0.03739999999999998 rpy=0.0 -0.0 0.0
- added joint h_gantry_right_kfs_gripper_gantry_r: type fixed, parent h_gantry_r, child kfs_gripper_link, origin xyz=-0.0325 -0.01 0.03739999999999998 rpy=0.0 -0.0 0.0
- added joint kfs_gripper_link_camera_rotate: type continuous, parent kfs_gripper_link, child camera_link, origin xyz=0.0 0.0 0.2125 rpy=3.944304526105059e-31 -0.0 1.1869459682199748e-66, axis 0.0 3.944304526105059e-31 1.0
- added joint kfs_gripper_link_spearhead_gripper_rotate: type continuous, parent kfs_gripper_link, child spearhead_gripper_link, origin xyz=0.0 0.12 0.2125 rpy=-3.141592653589793 -0.0 1.1869459682199748e-66, axis 0.0 8.359326303060042e-17 1.0
- added joint v_expandable_l_v_gantry_l: type prismatic, parent v_expandable_l, child v_gantry_l, origin xyz=0.0 -0.22 0.02 rpy=0.0 -1.1947622849140125e-34 0.0, axis 0.0 1.0 0.0, limit lower=0.0 upper=0.2 effort=100 velocity=1.0
- added joint v_expandable_r_v_gantry_r: type prismatic, parent v_expandable_r, child v_gantry_r, origin xyz=0.0 -0.22 0.02 rpy=1.232595164407831e-32 4.479329460506062e-34 3.141592653589793, axis 0.0 1.0 2.1895288505075267e-47, limit lower=0.0 upper=0.2 effort=100 velocity=1.0
- added joint v_gantry_l_h_expandable_l_to_v_gantry_l: type fixed, parent v_gantry_l, child h_expandable_l, origin xyz=7.130076136060349e-51 0.0 0.017100000000000008 rpy=0.0 1.1947622849140125e-34 0.0
- added joint v_gantry_r_h_expandable_r_to_v_gantry_r: type fixed, parent v_gantry_r, child h_expandable_r, origin xyz=-1.0538688655686983e-34 0.0 0.017100000000000008 rpy=-1.232595164407831e-32 -4.479329460506062e-34 -9.807621084706338e-81
- joint back_link_b_wheel_l: origin xyz=0.22530000000000003 0.0 0.0385 rpy=-0.0 1.5707963267948966 0 -> xyz=0.0 -0.2735 0.0385 rpy=1.5707963267948966 -0.0 0.0
- joint back_link_b_wheel_r: axis 0.0 0.0 1.0 -> 0.0 0.0 -1.0; origin xyz=-0.22530000000000003 0.0 0.0385 rpy=-3.141592653589793 1.5707963267948966 0 -> xyz=0.0 0.2735 0.0385 rpy=-1.5707963267948966 -0.0 0.0
- joint base_link_v_expandable_l: origin xyz=0.307 0.0 0.016 rpy=-1.5707963267948966 -0.0 1.5707963267948966 -> xyz=0.0 0.307 0.5660000000000001 rpy=1.5707963267948966 -0.0 0.0
- joint base_link_v_expandable_r: origin xyz=-0.307 0.0 0.016 rpy=-1.5707963267948966 -0.0 -1.5707963267948966 -> xyz=0.0 -0.307 0.5660000000000001 rpy=1.5707963267948966 -0.0 3.141592653589793
- joint base_to_storage_plate: origin xyz=0 0 0.1 rpy=0 0 0 -> xyz=0 0 0 rpy=0 0 0
- joint front_link_f_wheel_l: origin xyz=0.2225 0.0 0.0385 rpy=-0.0 1.5707963267948966 0 -> xyz=0.0 -0.2715 0.0385 rpy=1.5707963267948966 -0.0 0.0
- joint front_link_f_wheel_r: axis 0.0 0.0 1.0 -> 0.0 0.0 -1.0; origin xyz=-0.2223 0.0 0.0385 rpy=-3.141592653589793 1.5707963267948966 0 -> xyz=0.0 0.2715 0.0385 rpy=-1.5707963267948966 -0.0 0.0
