Commit message: Redited URDF with new design

File: ros2_ws/src/r2_description/urdf/r2.xacro (robot description, xacro)
@@ -8,7 +8,7 @@
     <link name="base_link">
         <inertial>
-            <origin xyz="4.897293290200259e-16 2.4486466451001295e-16 0.12668191002744514" rpy="0.0 0.0 0.0" />
-            <mass value="3.209133599999999" />
-            <inertia ixx="0.17822431950042106" iyy="0.3229109594506191" izz="0.33421926504374855" ixy="1.3201497495174412e-15" iyz="3.668280466055202e-17" ixz="2.3052629378746606e-16" />
+            <origin xyz="0.0042186271235444715 2.679193213808116e-16 0.0773228479596528" rpy="0.0 0.0 0.0" />
+            <mass value="5.132724217101411" />
+            <inertia ixx="0.42155335598643257" iyy="0.2892124481695275" izz="0.5315505031508672" ixy="-1.1992727721844926e-16" iyz="1.5347918280439902e-16" ixz="0.0001585619900969315" />
         </inertial>
         <visual name="base_link_visual">
@@ -29,10 +29,10 @@
     <link name="front_link">
         <inertial>
-            <origin xyz="3.987233071919613e-06 -3.552713678800501e-17 -0.02166273291491311" rpy="0.0 -0.0 0.0" />
-            <mass value="3.40650705960863" />
-            <inertia ixx="0.03380037538779723" iyy="0.16383842187451356" izz="0.1348712162134479" ixy="2.7502312764399878e-17" iyz="-1.214306433183765e-17" ixz="-8.171625823854828e-07" />
+            <origin xyz="1.1688428003253648e-14 -6.014164802022783e-17 -0.02416130998511414" rpy="0.0 -0.0 0.0" />
+            <mass value="3.2664694442174054" />
+            <inertia ixx="0.16196111692017123" iyy="0.033252044124773755" izz="0.13349589075190105" ixy="1.6108970157799827e-17" iyz="5.0711098953601913e-17" ixz="-2.392183673372017e-15" />
         </inertial>
         <visual name="front_link_visual">
-            <origin xyz="0.0 -0.23800000000000002 -0.006025000000000001" rpy="3.141592653589793 -0.0 0.0" />
+            <origin xyz="-0.23800000000000002 0.0 -0.006025000000000001" rpy="3.141592653589793 -0.0 0.0" />
             <geometry>
                 <mesh filename="package://r2_description/meshes/front_link.stl" scale="0.001 0.001 0.001" />
@@ -41,5 +41,5 @@
         </visual>
         <collision name="front_link_collision">
-            <origin xyz="0.0 -0.23800000000000002 -0.006025000000000001" rpy="3.141592653589793 -0.0 0.0" />
+            <origin xyz="-0.23800000000000002 0.0 -0.006025000000000001" rpy="3.141592653589793 -0.0 0.0" />
             <geometry>
                 <mesh filename="package://r2_description/meshes/front_link.stl" scale="0.001 0.001 0.001" />
@@ -50,10 +50,10 @@
     <link name="back_link">
         <inertial>
-            <origin xyz="5.713989178431127e-17 -3.552713678800501e-17 -0.021390972028288165" rpy="0.0 -0.0 0.0" />
-            <mass value="3.438068387047443" />
-            <inertia ixx="0.033867620091338285" iyy="0.16598701670020993" izz="0.1370310098698972" ixy="-3.1039235182106503e-17" iyz="2.2551405187698492e-17" ixz="-8.159900058500191e-17" />
+            <origin xyz="1.1688428003253648e-14 0.0 -0.024076465883564487" rpy="0.0 -0.0 0.0" />
+            <mass value="3.275109444217407" />
+            <inertia ixx="0.16435526563281905" iyy="0.03326294165161783" izz="0.1358827419377047" ixy="6.28642737865448e-17" iyz="0.0" ixz="-2.3869795029440866e-15" />
         </inertial>
         <visual name="back_link_visual">
-            <origin xyz="0.0 0.23800000000000002 -0.006025000000000001" rpy="3.141592653589793 -0.0 0.0" />
+            <origin xyz="0.23800000000000002 0.0 -0.006025000000000001" rpy="3.141592653589793 -0.0 0.0" />
             <geometry>
                 <mesh filename="package://r2_description/meshes/back_link.stl" scale="0.001 0.001 0.001" />
@@ -62,5 +62,5 @@
         </visual>
         <collision name="back_link_collision">
-            <origin xyz="0.0 0.23800000000000002 -0.006025000000000001" rpy="3.141592653589793 -0.0 0.0" />
+            <origin xyz="0.23800000000000002 0.0 -0.006025000000000001" rpy="3.141592653589793 -0.0 0.0" />
             <geometry>
                 <mesh filename="package://r2_description/meshes/back_link.stl" scale="0.001 0.001 0.001" />
@@ -71,10 +71,10 @@
     <link name="v_expandable_r">
         <inertial>
-            <origin xyz="0.0 -0.22 0.01" rpy="0.0 -0.0 0.0" />
-            <mass value="0.47519999999999996" />
-            <inertia ixx="0.007682399999999978" iyy="3.167999999999921e-05" izz="0.0076823999999999955" ixy="0.0" iyz="6.938893903907228e-18" ixz="0.0" />
+            <origin xyz="-1.2027605119163338e-13 -0.21999999999999964 0.010000000000000035" rpy="0.0 -0.0 0.0" />
+            <mass value="1.207983023592022" />
+            <inertia ixx="0.019534151646000752" iyy="9.07177309450169e-05" izz="0.019534151646180192" ixy="4.455505423730421e-18" iyz="-1.3877787807814457e-17" ixz="6.021653004568989e-18" />
         </inertial>
         <visual name="v_expandable_r_visual">
-            <origin xyz="0.0 0.016 0.307" rpy="1.5707963267948966 -1.5707963267948966 0" />
+            <origin xyz="-7.105427357601002e-17 -0.45599999999999946 0.3069999999999998" rpy="1.5707963267948966 -6.938893903907214e-18 3.141592653589793" />
             <geometry>
                 <mesh filename="package://r2_description/meshes/v_expandable_r.stl" scale="0.001 0.001 0.001" />
@@ -83,5 +83,5 @@
         </visual>
         <collision name="v_expandable_r_collision">
-            <origin xyz="0.0 0.016 0.307" rpy="1.5707963267948966 -1.5707963267948966 0" />
+            <origin xyz="-7.105427357601002e-17 -0.45599999999999946 0.3069999999999998" rpy="1.5707963267948966 -6.938893903907214e-18 3.141592653589793" />
             <geometry>
                 <mesh filename="package://r2_description/meshes/v_expandable_r.stl" scale="0.001 0.001 0.001" />
@@ -91,10 +91,10 @@
     <link name="v_expandable_l">
         <inertial>
-            <origin xyz="-1.6148698540002277e-18 -0.22 0.010000000000000071" rpy="0.0 -0.0 0.0" />
-            <mass value="0.47519999999999996" />
-            <inertia ixx="0.007682400000000006" iyy="3.167999999999921e-05" izz="0.0076823999999999955" ixy="-6.446043698815629e-20" iyz="0.0" ixz="-2.632134510349716e-19" />
+            <origin xyz="1.2020091795622878e-13 -0.22000000000000008 0.009999999999999858" rpy="0.0 -0.0 0.0" />
+            <mass value="1.207983023592022" />
+            <inertia ixx="0.019534151646000697" iyy="9.071773094505853e-05" izz="0.019534151646180414" ixy="1.2634758252215852e-18" iyz="1.1102230246251565e-16" ixz="-6.416558446259208e-18" />
         </inertial>
         <visual name="v_expandable_l_visual">
-            <origin xyz="0.0 0.016 0.307" rpy="1.5707963267948966 1.5707963267948966 0" />
+            <origin xyz="-7.105427357601002e-17 -0.45600000000000007 0.3069999999999999" rpy="-1.5707963267948957 1.3877787807814443e-17 -1.2246467991473532e-16" />
             <geometry>
                 <mesh filename="package://r2_description/meshes/v_expandable_l.stl" scale="0.001 0.001 0.001" />
@@ -103,5 +103,5 @@
         </visual>
         <collision name="v_expandable_l_collision">
-            <origin xyz="0.0 0.016 0.307" rpy="1.5707963267948966 1.5707963267948966 0" />
+            <origin xyz="-7.105427357601002e-17 -0.45600000000000007 0.3069999999999999" rpy="-1.5707963267948957 1.3877787807814443e-17 -1.2246467991473532e-16" />
             <geometry>
                 <mesh filename="package://r2_description/meshes/v_expandable_l.stl" scale="0.001 0.001 0.001" />
@@ -112,10 +112,10 @@
     <link name="h_expandable_r">
         <inertial>
-            <origin xyz="7.105427357601002e-17 7.888609052210118e-33 0.010000000000000071" rpy="0.0 -0.0 0.0" />
-            <mass value="0.8099999999999999" />
-            <inertia ixx="0.037995749999999995" iyy="5.3999999999998494e-05" izz="0.037995749999999995" ixy="0.0" iyz="1.5716068446636197e-17" ixz="0.0" />
+            <origin xyz="2.5217287189604704e-16 -2.1316282072803005e-16 0.009999999999999966" rpy="0.0 -0.0 0.0" />
+            <mass value="1.8925968312997488" />
+            <inertia ixx="0.00015121996039119123" iyy="0.08879108644737124" izz="0.08879108644737124" ixy="1.549594959280925e-17" iyz="2.7755575615628914e-17" ixz="7.182370609370982e-18" />
         </inertial>
         <visual name="h_expandable_r_visual">
-            <origin xyz="-0.13749999999999993 7.888609052210118e-33 0.2699000000000001" rpy="-3.141592653589793 -1.5707963267948966 0" />
+            <origin xyz="6.042827863252935e-17 0.2824999999999999 0.26990000000000003" rpy="1.5707963267948966 -0.0 -1.2246467991473532e-16" />
             <geometry>
                 <mesh filename="package://r2_description/meshes/h_expandable_r.stl" scale="0.001 0.001 0.001" />
@@ -124,5 +124,5 @@
         </visual>
         <collision name="h_expandable_r_collision">
-            <origin xyz="-0.13749999999999993 7.888609052210118e-33 0.2699000000000001" rpy="-3.141592653589793 -1.5707963267948966 0" />
+            <origin xyz="6.042827863252935e-17 0.2824999999999999 0.26990000000000003" rpy="1.5707963267948966 -0.0 -1.2246467991473532e-16" />
             <geometry>
                 <mesh filename="package://r2_description/meshes/h_expandable_r.stl" scale="0.001 0.001 0.001" />
@@ -132,10 +132,10 @@
     <link name="h_expandable_l">
         <inertial>
-            <origin xyz="0.0 -2.220446049250313e-18 0.010000000000000071" rpy="0.0 -0.0 0.0" />
-            <mass value="0.8099999999999999" />
-            <inertia ixx="0.03799575000000002" iyy="5.400000000002625e-05" izz="0.037995749999999995" ixy="0.0" iyz="-1.57160684466362e-17" ixz="6.938893903907228e-18" />
+            <origin xyz="-1.7783613980752874e-16 2.1316282072803005e-16 0.009999999999999929" rpy="0.0 -0.0 0.0" />
+            <mass value="1.8925968312997483" />
+            <inertia ixx="0.0001512199603910247" iyy="0.08879108644737121" izz="0.08879108644737113" ixy="3.5843619808224064e-17" iyz="-8.326672684688674e-17" ixz="5.683068593498344e-18" />
         </inertial>
         <visual name="h_expandable_l_visual">
-            <origin xyz="-0.1375 -2.220446049250313e-18 0.2699000000000001" rpy="-0.0 1.5707963267948966 0" />
+            <origin xyz="-6.153850165715452e-17 -0.28250000000000003 0.26990000000000003" rpy="-1.5707963267948966 -0.0 -1.2246467991473532e-16" />
             <geometry>
                 <mesh filename="package://r2_description/meshes/h_expandable_l.stl" scale="0.001 0.001 0.001" />
@@ -144,5 +144,5 @@
         </visual>
         <collision name="h_expandable_l_collision">
-            <origin xyz="-0.1375 -2.220446049250313e-18 0.2699000000000001" rpy="-0.0 1.5707963267948966 0" />
+            <origin xyz="-6.153850165715452e-17 -0.28250000000000003 0.26990000000000003" rpy="-1.5707963267948966 -0.0 -1.2246467991473532e-16" />
             <geometry>
                 <mesh filename="package://r2_description/meshes/h_expandable_l.stl" scale="0.001 0.001 0.001" />
@@ -153,10 +153,10 @@
     <link name="v_gantry_r">
         <inertial>
-            <origin xyz="7.105427357601002e-17 1.916272831499797e-17 0.008550000000000111" rpy="0.0 -0.0 0.0" />
-            <mass value="0.1950682500000001" />
-            <inertia ixx="7.343360526937924e-05" iyy="7.343360526937404e-05" izz="0.00013736055937500075" ixy="-1.151079231931344e-20" iyz="3.783213742280244e-20" ixz="0.0" />
+            <origin xyz="2.5832006556616624e-17 -7.105427357601002e-17 0.008550000000000075" rpy="0.0 -0.0 0.0" />
+            <mass value="0.5671428750000002" />
+            <inertia ixx="0.00021350140791281946" iyy="0.00021350140791281252" izz="0.0003993631078125087" ixy="2.6773250283440193e-19" iyz="4.922530355325821e-36" ixz="2.231104190286638e-20" />
         </inertial>
         <visual name="v_gantry_r_visual">
-            <origin xyz="-0.1375 -4.4408920985006186e-18 0.2870000000000019" rpy="-3.141592653589793 -1.5707963267948966 0" />
+            <origin xyz="6.042827863252935e-17 0.2824999999999999 0.28700000000000003" rpy="1.5707963267948966 -4.479329460506078e-34 -1.2246467991473532e-16" />
             <geometry>
                 <mesh filename="package://r2_description/meshes/v_gantry_r.stl" scale="0.001 0.001 0.001" />
@@ -165,5 +165,5 @@
         </visual>
         <collision name="v_gantry_r_collision">
-            <origin xyz="-0.1375 -4.4408920985006186e-18 0.2870000000000019" rpy="-3.141592653589793 -1.5707963267948966 0" />
+            <origin xyz="6.042827863252935e-17 0.2824999999999999 0.28700000000000003" rpy="1.5707963267948966 -4.479329460506078e-34 -1.2246467991473532e-16" />
             <geometry>
                 <mesh filename="package://r2_description/meshes/v_gantry_r.stl" scale="0.001 0.001 0.001" />
@@ -173,10 +173,10 @@
     <link name="v_gantry_l">
         <inertial>
-            <origin xyz="0.0 -2.220446049250313e-18 0.00855000000000004" rpy="0.0 -0.0 0.0" />
-            <mass value="0.19506825000000005" />
-            <inertia ixx="7.34336052693723e-05" iyy="7.343360526937057e-05" izz="0.000137360559374999" ixy="3.0695446184836335e-20" iyz="-1.5347723092418186e-20" ixz="-3.469446951953614e-18" />
+            <origin xyz="-2.6942229581241788e-17 0.0 0.008550000000000075" rpy="0.0 -0.0 0.0" />
+            <mass value="0.5671428750000002" />
+            <inertia ixx="0.00021350140791281946" iyy="0.00021350140791281252" izz="0.00039936310781249484" ixy="-2.6773250283440656e-19" iyz="1.1163468592440427e-67" ixz="-2.2311041902865608e-20" />
         </inertial>
         <visual name="v_gantry_l_visual">
-            <origin xyz="-0.1375 -2.220446049250313e-18 0.287" rpy="-0.0 1.5707963267948966 0" />
+            <origin xyz="-6.153850165715452e-17 -0.28250000000000003 0.28700000000000003" rpy="-1.5707963267948966 1.1947622849140125e-34 -1.2246467991473532e-16" />
             <geometry>
                 <mesh filename="package://r2_description/meshes/v_gantry_l.stl" scale="0.001 0.001 0.001" />
@@ -185,5 +185,5 @@
         </visual>
         <collision name="v_gantry_l_collision">
-            <origin xyz="-0.1375 -2.220446049250313e-18 0.287" rpy="-0.0 1.5707963267948966 0" />
+            <origin xyz="-6.153850165715452e-17 -0.28250000000000003 0.28700000000000003" rpy="-1.5707963267948966 1.1947622849140125e-34 -1.2246467991473532e-16" />
             <geometry>
                 <mesh filename="package://r2_description/meshes/v_gantry_l.stl" scale="0.001 0.001 0.001" />
@@ -193,10 +193,10 @@
     <link name="h_gantry_r">
         <inertial>
-            <origin xyz="0.0020155393053017077 0.0 0.02631243144424129" rpy="0.0 -0.0 0.0" />
-            <mass value="0.07384499999999983" />
-            <inertia ixx="3.7790538137933306e-05" iyy="2.5063800306580203e-05" izz="1.8042012168647398e-05" ixy="-8.881784197001253e-20" iyz="0.0" ixz="5.376652650835798e-07" />
+            <origin xyz="0.0 0.013832853025936558 0.02363371757925073" rpy="0.0 -0.0 0.0" />
+            <mass value="0.7082269999999997" />
+            <inertia ixx="0.00028625336112315936" iyy="0.000320958411897658" izz="0.0004640047950588283" ixy="1.2494183465605601e-18" iyz="-5.6491115619582144e-05" ixz="8.031975085032172e-19" />
         </inertial>
         <visual name="h_gantry_r_visual">
-            <origin xyz="-0.23600000000000002 -0.025 0.24989999999999998" rpy="-3.141592653589793 -1.5707963267948966 0" />
+            <origin xyz="0.0 0.34600000000000003 0.24989999999999998" rpy="1.5707963267948966 -0.0 0.0" />
             <geometry>
                 <mesh filename="package://r2_description/meshes/h_gantry_r.stl" scale="0.001 0.001 0.001" />
@@ -205,5 +205,5 @@
         </visual>
         <collision name="h_gantry_r_collision">
-            <origin xyz="-0.23600000000000002 -0.025 0.24989999999999998" rpy="-3.141592653589793 -1.5707963267948966 0" />
+            <origin xyz="0.0 0.34600000000000003 0.24989999999999998" rpy="1.5707963267948966 -0.0 0.0" />
             <geometry>
                 <mesh filename="package://r2_description/meshes/h_gantry_r.stl" scale="0.001 0.001 0.001" />
@@ -213,10 +213,10 @@
     <link name="h_gantry_l">
         <inertial>
-            <origin xyz="0.002015539305301672 0.0 0.02631243144424129" rpy="0.0 -0.0 0.0" />
-            <mass value="0.07384499999999992" />
-            <inertia ixx="3.779053813793374e-05" iyy="2.5063800306578468e-05" izz="1.8042012168645663e-05" ixy="0.0" iyz="0.0" ixz="5.37665265081845e-07" />
+            <origin xyz="0.0 -0.013832853025936629 0.023633717579250695" rpy="0.0 -0.0 0.0" />
+            <mass value="0.7082270000000002" />
+            <inertia ixx="0.00028625336112317323" iyy="0.0003209584118976441" izz="0.0004640047950588283" ixy="-1.7848833522293717e-19" iyz="5.6491115619575205e-05" ixz="-8.924416761146858e-20" />
         </inertial>
         <visual name="h_gantry_l_visual">
-            <origin xyz="-0.23600000000000002 0.025 0.24989999999999998" rpy="-0.0 1.5707963267948966 0" />
+            <origin xyz="0.0 -0.34600000000000003 0.24989999999999998" rpy="-1.5707963267948966 -0.0 0.0" />
             <geometry>
                 <mesh filename="package://r2_description/meshes/h_gantry_l.stl" scale="0.001 0.001 0.001" />
@@ -225,5 +225,5 @@
         </visual>
         <collision name="h_gantry_l_collision">
-            <origin xyz="-0.23600000000000002 0.025 0.24989999999999998" rpy="-0.0 1.5707963267948966 0" />
+            <origin xyz="0.0 -0.34600000000000003 0.24989999999999998" rpy="-1.5707963267948966 -0.0 0.0" />
             <geometry>
                 <mesh filename="package://r2_description/meshes/h_gantry_l.stl" scale="0.001 0.001 0.001" />
@@ -234,10 +234,10 @@
     <link name="f_wheel_r">
         <inertial>
-            <origin xyz="-1.7763568394002505e-17 0.0 0.025500000000000078" rpy="0.0 -0.0 0.0" />
-            <mass value="0.5364206624151502" />
-            <inertia ixx="0.0005990477747521011" iyy="0.000599047774752122" izz="0.000965557192347262" ixy="0.0" iyz="6.938893903907228e-18" ixz="1.734723475976807e-18" />
+            <origin xyz="1.3713474800169933e-14 -2.6645352591003756e-17 -0.025026743072870658" rpy="0.0 -0.0 0.0" />
+            <mass value="0.5401867094404943" />
+            <inertia ixx="0.0006063195606969968" iyy="0.0006063195607106525" izz="0.0009683138409003339" ixy="-8.673617379884035e-19" iyz="1.734723475976807e-18" ixz="-1.3877787807814457e-17" />
         </inertial>
         <visual name="f_wheel_r_visual">
-            <origin xyz="0.044524999999999995 0.23800000000000002 -0.2223" rpy="-0.0 1.5707963267948966 0" />
+            <origin xyz="-0.23800000000000002 0.044524999999999995 -0.2715" rpy="-1.5707963267948966 -0.0 0.0" />
             <geometry>
                 <mesh filename="package://r2_description/meshes/f_wheel_r.stl" scale="0.001 0.001 0.001" />
@@ -246,5 +246,5 @@
         </visual>
         <collision name="f_wheel_r_collision">
-            <origin xyz="0.044524999999999995 0.23800000000000002 -0.2223" rpy="-0.0 1.5707963267948966 0" />
+            <origin xyz="-0.23800000000000002 0.044524999999999995 -0.2715" rpy="-1.5707963267948966 -0.0 0.0" />
             <geometry>
                 <mesh filename="package://r2_description/meshes/f_wheel_r.stl" scale="0.001 0.001 0.001" />
@@ -254,10 +254,10 @@
     <link name="f_wheel_l">
         <inertial>
-            <origin xyz="-1.7763568394002505e-17 0.0 0.025500000000000078" rpy="0.0 -0.0 0.0" />
-            <mass value="0.5364206624151502" />
-            <inertia ixx="0.0005990477747521011" iyy="0.0005990477747521289" izz="0.000965557192347262" ixy="0.0" iyz="0.0" ixz="1.734723475976807e-18" />
+            <origin xyz="7.105427357601002e-17 8.881784197001253e-18 -0.025026743072870658" rpy="0.0 -0.0 0.0" />
+            <mass value="0.540186709440494" />
+            <inertia ixx="0.0006063195607004176" iyy="0.000606319560700383" izz="0.0009683138408934852" ixy="8.673617379884035e-19" iyz="0.0" ixz="6.938893903907228e-18" />
         </inertial>
         <visual name="f_wheel_l_visual">
-            <origin xyz="0.044524999999999995 -0.23800000000000002 -0.2225" rpy="-3.141592653589793 -1.5707963267948966 0" />
+            <origin xyz="-0.23800000000000002 -0.044524999999999995 -0.2715" rpy="1.5707963267948966 -0.0 0.0" />
             <geometry>
                 <mesh filename="package://r2_description/meshes/f_wheel_l.stl" scale="0.001 0.001 0.001" />
@@ -266,5 +266,5 @@
         </visual>
         <collision name="f_wheel_l_collision">
-            <origin xyz="0.044524999999999995 -0.23800000000000002 -0.2225" rpy="-3.141592653589793 -1.5707963267948966 0" />
+            <origin xyz="-0.23800000000000002 -0.044524999999999995 -0.2715" rpy="1.5707963267948966 -0.0 0.0" />
             <geometry>
                 <mesh filename="package://r2_description/meshes/f_wheel_l.stl" scale="0.001 0.001 0.001" />
@@ -274,10 +274,10 @@
     <link name="b_wheel_r">
         <inertial>
-            <origin xyz="-1.7763568394002505e-17 3.552713678800501e-17 0.025500000000000043" rpy="0.0 -0.0 0.0" />
-            <mass value="0.5364206624151502" />
-            <inertia ixx="0.0005990477747520873" iyy="0.0005990477747521081" izz="0.000965557192347262" ixy="0.0" iyz="6.938893903907228e-18" ixz="-2.6020852139652106e-18" />
+            <origin xyz="-6.8212102632969615e-15 -8.881784197001253e-18 -0.025026743072870658" rpy="0.0 -0.0 0.0" />
+            <mass value="0.5401867094404935" />
+            <inertia ixx="0.0006063195607106525" iyy="0.0006063195606969829" izz="0.000968313840900327" ixy="3.469446951953614e-18" iyz="-8.673617379884035e-19" ixz="0.0" />
         </inertial>
         <visual name="b_wheel_r_visual">
-            <origin xyz="0.044524999999999995 -0.23800000000000002 -0.22530000000000003" rpy="-0.0 1.5707963267948966 0" />
+            <origin xyz="0.23800000000000002 0.044524999999999995 -0.2735" rpy="-1.5707963267948966 -0.0 0.0" />
             <geometry>
                 <mesh filename="package://r2_description/meshes/b_wheel_r.stl" scale="0.001 0.001 0.001" />
@@ -286,5 +286,5 @@
         </visual>
         <collision name="b_wheel_r_collision">
-            <origin xyz="0.044524999999999995 -0.23800000000000002 -0.22530000000000003" rpy="-0.0 1.5707963267948966 0" />
+            <origin xyz="0.23800000000000002 0.044524999999999995 -0.2735" rpy="-1.5707963267948966 -0.0 0.0" />
             <geometry>
                 <mesh filename="package://r2_description/meshes/b_wheel_r.stl" scale="0.001 0.001 0.001" />
@@ -294,10 +294,10 @@
     <link name="b_wheel_l">
         <inertial>
-            <origin xyz="8.881784197001253e-18 -3.552713678800501e-17 0.02550000000000001" rpy="0.0 -0.0 0.0" />
-            <mass value="0.5364206624151507" />
-            <inertia ixx="0.0005990477747521011" iyy="0.0005990477747521289" izz="0.000965557192347262" ixy="8.673617379884035e-19" iyz="0.0" ixz="8.673617379884035e-19" />
+            <origin xyz="-3.552713678800501e-17 1.7763568394002505e-17 -0.025026743072870696" rpy="0.0 -0.0 0.0" />
+            <mass value="0.5401867094404945" />
+            <inertia ixx="0.0006063195607004385" iyy="0.0006063195607003968" izz="0.0009683138408934852" ixy="1.734723475976807e-18" iyz="-2.6020852139652106e-18" ixz="0.0" />
         </inertial>
         <visual name="b_wheel_l_visual">
-            <origin xyz="0.044524999999999995 0.23800000000000002 -0.22530000000000003" rpy="-3.141592653589793 -1.5707963267948966 0" />
+            <origin xyz="0.23800000000000002 -0.044524999999999995 -0.2735" rpy="1.5707963267948966 -0.0 0.0" />
             <geometry>
                 <mesh filename="package://r2_description/meshes/b_wheel_l.stl" scale="0.001 0.001 0.001" />
@@ -306,5 +306,5 @@
         </visual>
         <collision name="b_wheel_l_collision">
-            <origin xyz="0.044524999999999995 0.23800000000000002 -0.22530000000000003" rpy="-3.141592653589793 -1.5707963267948966 0" />
+            <origin xyz="0.23800000000000002 -0.044524999999999995 -0.2735" rpy="1.5707963267948966 -0.0 0.0" />
             <geometry>
                 <mesh filename="package://r2_description/meshes/b_wheel_l.stl" scale="0.001 0.001 0.001" />
@@ -315,10 +315,10 @@
     <link name="kfs_gripper_link">
         <inertial>
-            <origin xyz="-0.1788606356968211 0.2124999999999979 0.059999999999999824" rpy="0.0 -0.0 0.0" />
-            <mass value="1.5901920000000178" />
-            <inertia ixx="0.060185394295200485" iyy="0.030950832458641303" izz="0.08499517740984172" ixy="-5.753026763865059e-16" iyz="9.076029527932467e-17" ixz="2.983724378680108e-16" />
+            <origin xyz="0.2317152428810716 0.060000000000000143 0.21250000000000102" rpy="0.0 -0.0 0.0" />
+            <mass value="6.748488000000025" />
+            <inertia ixx="0.2679460085435912" iyy="0.38855510203554466" izz="0.14309519115594393" ixy="-2.7755575615628914e-16" iyz="-3.576344126329944e-15" ixz="-1.131665944136903e-15" />
         </inertial>
         <visual name="kfs_gripper_link_visual">
-            <origin xyz="1.3322676295501878e-17 0.2125 0.22599999999999995" rpy="3.141592653589793 -0.0 1.5707963267948966" />
+            <origin xyz="1.3322676295501878e-17 0.35600000000000187 0.2125" rpy="1.5707963267948941 1.0408340855860872e-17 0.0" />
             <geometry>
                 <mesh filename="package://r2_description/meshes/kfs_gripper_link.stl" scale="0.001 0.001 0.001" />
@@ -327,5 +327,5 @@
         </visual>
         <collision name="kfs_gripper_link_collision">
-            <origin xyz="1.3322676295501878e-17 0.2125 0.22599999999999995" rpy="3.141592653589793 -0.0 1.5707963267948966" />
+            <origin xyz="1.3322676295501878e-17 0.35600000000000187 0.2125" rpy="1.5707963267948941 1.0408340855860872e-17 0.0" />
             <geometry>
                 <mesh filename="package://r2_description/meshes/kfs_gripper_link.stl" scale="0.001 0.001 0.001" />
@@ -336,10 +336,10 @@
     <link name="spearhead_gripper_link">
         <inertial>
-            <origin xyz="0.013906681741505356 0.08947355340193562 -4.819654465716614e-07" rpy="0.0 -0.0 0.0" />
-            <mass value="0.2039245280299798" />
-            <inertia ixx="0.0010268947573349868" iyy="0.0007077393295979702" izz="0.00039333940611649843" ixy="-3.7809718414193345e-05" iyz="-3.3874379563644606e-09" ixz="5.988792025088906e-10" />
+            <origin xyz="-0.1187965702156902 0.014232345919710633 6.106982515756493e-16" rpy="0.0 -0.0 0.0" />
+            <mass value="2.783302899502935" />
+            <inertia ixx="0.00619735005930841" iyy="0.013682230278330501" izz="0.008463736029391739" ixy="0.0007106267959798712" iyz="2.1015313562747538e-17" ixz="-1.216101173826227e-16" />
         </inertial>
         <visual name="spearhead_gripper_link_visual">
-            <origin xyz="-0.22899999999999998 -0.025000000000000005 0.0" rpy="-0.0 1.5707963267948966 0" />
+            <origin xyz="0.02049999999999983 -0.2359999999999991 -4.1334256279161996e-17" rpy="-1.570796326794894 4.671268081547312e-31 -3.9048654142723077e-47" />
             <geometry>
                 <mesh filename="package://r2_description/meshes/spearhead_gripper_link.stl" scale="0.001 0.001 0.001" />
@@ -348,5 +348,5 @@
         </visual>
         <collision name="spearhead_gripper_link_collision">
-            <origin xyz="-0.22899999999999998 -0.025000000000000005 0.0" rpy="-0.0 1.5707963267948966 0" />
+            <origin xyz="0.02049999999999983 -0.2359999999999991 -4.1334256279161996e-17" rpy="-1.570796326794894 4.671268081547312e-31 -3.9048654142723077e-47" />
             <geometry>
                 <mesh filename="package://r2_description/meshes/spearhead_gripper_link.stl" scale="0.001 0.001 0.001" />
@@ -357,10 +357,10 @@
     <link name="camera_link">
         <inertial>
-            <origin xyz="0.012500000000000107 -0.009913368991069482 7.563616562748968e-15" rpy="0.0 -0.0 0.0" />
-            <mass value="0.03892040918246199" />
-            <inertia ixx="1.9303975960481232e-05" iyy="2.0030596346482486e-05" izz="3.2847651887722533e-06" ixy="2.0328790734103208e-19" iyz="1.5937944577546263e-19" ixz="-8.741089572321102e-20" />
+            <origin xyz="0.009894465299491869 -0.012500000000000072 9.415354068752146e-15" rpy="0.0 -0.0 0.0" />
+            <mass value="0.2875377274000879" />
+            <inertia ixx="0.00014832028606556052" iyy="0.0001429062226769995" izz="2.427338819091518e-05" ixy="8.673617379884035e-19" iyz="4.462208380571582e-20" ixz="-2.412613722866814e-17" />
         </inertial>
         <visual name="camera_link_visual">
-            <origin xyz="-0.226 -0.03300000000000002 1.1102230246251565e-16" rpy="-0.0 1.570796326794896 0" />
+            <origin xyz="0.052499999999999984 0.36749999999999994 -3.552713678800515e-17" rpy="1.5707963267948966 -4.6816763546921983e-97 -1.1869459682199748e-66" />
             <geometry>
                 <mesh filename="package://r2_description/meshes/camera_link.stl" scale="0.001 0.001 0.001" />
@@ -369,5 +369,5 @@
         </visual>
         <collision name="camera_link_collision">
-            <origin xyz="-0.226 -0.03300000000000002 1.1102230246251565e-16" rpy="-0.0 1.570796326794896 0" />
+            <origin xyz="0.052499999999999984 0.36749999999999994 -3.552713678800515e-17" rpy="1.5707963267948966 -4.6816763546921983e-97 -1.1869459682199748e-66" />
             <geometry>
                 <mesh filename="package://r2_description/meshes/camera_link.stl" scale="0.001 0.001 0.001" />
@@ -398,6 +398,6 @@
 <!--JOINTS-->
     <!--Base link -Front-Back-Links-->
-    <joint name="base_link_front_link_joint" type="prismatic">
-        <origin xyz="0.0 -0.23800000000000002 -0.006025000000000001" rpy="3.141592653589793 -0.0 0.0" />
+    <joint name="base_link_front_link" type="prismatic">
+        <origin xyz="0.23800000000000002 0.0 -0.006025000000000001" rpy="3.141592653589793 -0.0 0.0" />
         <parent link="base_link" />
         <child link="front_link" />
@@ -405,6 +405,6 @@
         <limit lower="0.0" upper="0.2" effort="100" velocity="1.0"/>
     </joint>
-    <joint name="base_link_back_link_joint" type="prismatic">
-        <origin xyz="0.0 0.23800000000000002 -0.006025000000000001" rpy="3.141592653589793 -0.0 0.0" />
+    <joint name="base_link_back_link" type="prismatic">
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