Commit message: Editing r2 description for mechanum control

File: ros2_ws/src/r2_description/urdf/r2.urdf (robot description, URDF)
Before this commit: robot r2, 23 links, 22 joints
Joints:
- joint spearhead_body_spearhead_finger_l_grip: limit lower=-0.05 upper=0.05 effort=100 velocity=1.0 -> lower=-0.02896 upper=-0.008765 effort=100 velocity=1.0
- joint spearhead_body_spearhead_finger_r_grip: limit lower=-0.05 upper=0.05 effort=100 velocity=1.0 -> lower=-0.02896 upper=-0.008765 effort=100 velocity=1.0

File: ros2_ws/src/r2_description/urdf/r2.xacro (robot description, xacro)
@@ -369,5 +369,5 @@
         <inertial>
             <origin xyz="-0.0059999999999999784 0.059999999999999894 0.2728741721854304" rpy="0.0 -0.0 0.0" />
-            <mass value="2.7310464000000003" />
+            <mass value="0.412153" />
             <inertia ixx="0.029521380670728292" iyy="0.02546431176832853" izz="0.0041226140159998925" ixy="0.0" iyz="-5.551115123125783e-17" ixz="-2.7755575615628914e-17" />
         </inertial>
@@ -567,5 +567,5 @@
         <child link="v_expandable_r" />
         <axis xyz="0.0 1.0 0.0" />
-        <limit lower="0.0" upper="0.2" effort="100" velocity="1.0"/>
+        <limit lower="0.0" upper="0.33" effort="100" velocity="1.0"/>
         <dynamics damping="5.0" friction="1.0"/>
     </joint>
@@ -575,5 +575,5 @@
         <child link="v_expandable_l" />
         <axis xyz="0.0 1.0 0.0" />
-        <limit lower="0.0" upper="0.2" effort="100" velocity="1.0"/>
+        <limit lower="0.0" upper="0.33" effort="100" velocity="1.0"/>
         <dynamics damping="5.0" friction="1.0"/>
     </joint>
@@ -584,5 +584,5 @@
         <child link="v_gantry_r" />
         <axis xyz="0.0 1.0 2.1895288505075267e-47" />
-        <limit lower="-0.18" upper="+0.18" effort="100" velocity="1.0"/>
+        <limit lower="-0.131" upper="+0.131" effort="100" velocity="1.0"/>
         <dynamics damping="5.0" friction="1.0"/>
     </joint>
@@ -592,5 +592,5 @@
         <child link="v_gantry_l" />
         <axis xyz="0.0 1.0 0.0" />
-        <limit lower="-0.18" upper="+0.18" effort="100" velocity="1.0"/>
+        <limit lower="-0.131" upper="+0.131" effort="100" velocity="1.0"/>
         <dynamics damping="5.0" friction="1.0"/>
     </joint>
@@ -612,5 +612,5 @@
         <child link="h_gantry_r" />
         <axis xyz="0.0 0.0 1.0" />
-        <limit lower="0.0" upper="0.2" effort="100" velocity="1.0"/>
+        <limit lower="-0.295" upper="0.295" effort="100" velocity="1.0"/>
         <dynamics damping="5.0" friction="1.0"/>
     </joint>
@@ -620,5 +620,5 @@
         <child link="h_gantry_l" />
         <axis xyz="0.0 1.0 0.0" />
-        <limit lower="0.0" upper="0.2" effort="100" velocity="1.0"/>
+        <limit lower="-0.295" upper="0.295" effort="100" velocity="1.0"/>
         <dynamics damping="5.0" friction="1.0"/>
     </joint>
@@ -635,5 +635,5 @@
         <child link="kfs_finger" />
         <axis xyz="1.0 0.0 0.0" />
-        <limit lower="0.0" upper="0.2" effort="100" velocity="1.0"/>
+        <limit lower="-0.089" upper="0.0" effort="100" velocity="1.0"/>
     </joint>
     <!--Spearhead Gripping Joint-->
@@ -643,5 +643,5 @@
         <child link="spearhead_finger_l" />
         <axis xyz="-1.4449768080836794e-62 0.0 1.0" />
-        <limit lower="-0.05" upper="0.05" effort="100" velocity="1.0"/>
+        <limit lower="-0.02896" upper="-0.08765" effort="100" velocity="1.0"/>
     </joint>
     <joint name="spearhead_body_spearhead_finger_r_grip" type="prismatic">
@@ -650,5 +650,5 @@
         <child link="spearhead_finger_r" />
         <axis xyz="-1.4449768080836794e-62 0.0 1.0" />
-        <limit lower="-0.05" upper="0.05" effort="100" velocity="1.0"/>
+        <limit lower="-0.02896" upper="-0.08765" effort="100" velocity="1.0"/>
     </joint>
     <!--Spearhead Revolute-->

Commit message: still editing xacro

File: ros2_ws/src/r2_description/urdf/r2.urdf (robot description, URDF)
Before this commit: robot r2, 23 links, 22 joints
Joints:
- removed joint h_gantry_left_kfs_gripper_gantry_l
- added joint h_gantry_r_kfs_gripper_gantry_r: type fixed, parent h_gantry_r, child kfs_gripper_link, origin xyz=-0.0325 -0.01 0.03739999999999998 rpy=0.0 -0.0 0.0
- joint h_expandable_l_h_gantry_l: axis 0.0 1.0 0.0 -> 1.0 0.0 0.0; origin xyz=0.0 0.0 0.02 rpy=0.0 0.0 0.0 -> xyz=0.0 0.0 0.02 rpy=0.0 -0.0 0.0
- joint h_expandable_r_h_gantry_r: axis 0.0 0.0 1.0 -> 1.0 0.0 0.0

File: ros2_ws/src/r2_description/urdf/r2.xacro (robot description, xacro)
@@ -621,7 +621,7 @@
         <dynamics damping="5.0" friction="1.0"/>
     </joint>
-<!-- KFS Gripper Joint -->
-    <joint name="gantry_bridge_kfs_gripper_joint" type="fixed">
-        <origin xyz="0.01 0.0 0.05" rpy="0.0 0 0.0" />
+    <!--horizontal Gantry and KFS Gripper-->
+    <joint name="h_gantry_r_kfs_gripper_gantry_r" type="fixed">
+        <origin xyz="-0.0325 -0.01 0.03739999999999998" rpy="0.0 -0.0 0.0" />
         <parent link="h_gantry_r" />
         <child link="kfs_gripper_link" />
@@ -651,9 +651,9 @@
     </joint>
     <!--Spearhead Revolute-->
-    <joint name="kfs_gripper_link_spearhead_gripper_rotate" type="revolute">
-        <origin xyz="0.0 0.12 0.2125" rpy="-3.141592653589793 -0.0 0.0" />
+    <joint name="kfs_gripper_link_spearhead_gripper_rotate" type="continuous">
+        <origin xyz="0.0 0.12 0.2125" rpy="-3.141592653589793 -0.0 1.1869459682199748e-66" />
         <parent link="kfs_gripper_link" />
         <child link="spearhead_body" />
-        <axis xyz="0.0 8.359326303060002e-17 1.0" />
+        <axis xyz="0.0 8.359326303060042e-17 1.0" />
         <limit lower="-1.5707963267948966" upper="1.5707963267948966" effort="100" velocity="1.0"/>
     </joint>
