Commit message: ending this work for now...@MysticCore... Sleepy

File: ros2_ws/src/r2_description/urdf/r2.xacro (robot description, xacro)
@@ -307,5 +307,5 @@
             <origin xyz="0.044524999999999995 0.23800000000000002 -0.22530000000000003" rpy="1.5708 -1.5707963267948966 0" />
             <geometry>
-                <mesh filename="package://r2_description/meshes/b_wheel_l.stl" scale="0.001 0.001 0.001" />
+                <mesh filename="package://r2_description/meshes/b_wheel_l.stl" scale="0.001 ₀.₀₀₁" />
             </geometry>
         </collision>

Commit message: Added control plugin in xacro
Addded controller.yaml files for all mechanisms

Created Launch file for controllers

File: ros2_ws/src/r2_description/urdf/r2.xacro (robot description, xacro)
@@ -404,4 +404,5 @@
         <axis xyz="0.0 0.0 1.0" />
         <limit lower="0.0" upper="0.2" effort="100" velocity="1.0"/>
+        <dynamics damping="10.0" friction="2.0"/>
     </joint>
     <joint name="base_link_back_link" type="prismatic">
@@ -411,4 +412,5 @@
         <axis xyz="0.0 0.0 1.0" />
         <limit lower="0.0" upper="0.2" effort="100" velocity="1.0"/>
+        <dynamics damping="10.0" friction="2.0"/>
     </joint>
     <!--Wheel Joints-->
@@ -444,4 +446,5 @@
         <axis xyz="0.0 1.0 0.0" />
         <limit lower="0.0" upper="0.2" effort="100" velocity="1.0"/>
+        <dynamics damping="5.0" friction="1.0"/>
     </joint>
     <joint name="base_link_v_expandable_l" type="prismatic">
@@ -451,4 +454,5 @@
         <axis xyz="0.0 1.0 0.0" />
         <limit lower="0.0" upper="0.2" effort="100" velocity="1.0"/>
+        <dynamics damping="5.0" friction="1.0"/>
     </joint>
     <!--V_expandable-to-gantry-->
@@ -459,4 +463,5 @@
         <axis xyz="0.0 1.0 2.1895288505075267e-47" />
         <limit lower="0.0" upper="0.2" effort="100" velocity="1.0"/>
+        <dynamics damping="5.0" friction="1.0"/>
     </joint>
     <joint name="v_expandable_l_v_gantry_l" type="prismatic">
@@ -466,4 +471,5 @@
         <axis xyz="0.0 1.0 0.0" />
         <limit lower="0.0" upper="0.2" effort="100" velocity="1.0"/>
+        <dynamics damping="5.0" friction="1.0"/>
     </joint>
     <!--V_gantry-to-H_Expandable-->
@@ -485,4 +491,5 @@
         <axis xyz="0.0 1.0 0.0" />
         <limit lower="0.0" upper="0.2" effort="100" velocity="1.0"/>
+        <dynamics damping="5.0" friction="1.0"/>
     </joint>
     <joint name="h_expandable_l_h_gantry_l" type="prismatic">
@@ -492,4 +499,5 @@
         <axis xyz="0.0 1.0 0.0" />
         <limit lower="0.0" upper="0.2" effort="100" velocity="1.0"/>
+        <dynamics damping="5.0" friction="1.0"/>
     </joint>
     <!--horizontal Gantry and KFS Gripper-->
@@ -499,4 +507,5 @@
         <child link="kfs_gripper_link" />
     </joint>
+    <!--
     <joint name="h_gantry_left_kfs_gripper_gantry_l" type="fixed">
         <origin xyz="-0.0325 0.01 0.03739999999999998" rpy="0.0 -0.0 0.0" />
@@ -504,4 +513,5 @@
         <child link="kfs_gripper_link" />
     </joint>
+    -->
     <!--Spearhead Revolute-->
     <joint name="kfs_gripper_link_spearhead_gripper_rotate" type="continuous">
@@ -524,3 +534,104 @@
         <origin xyz="0 0 0" rpy="0 0 0"/>
     </joint>
+<!--Wheels Friction-->
+        <gazebo reference="f_wheel_r">
+            <mu1>1.8</mu1>
+            <mu2>1.8</mu2>
+        </gazebo>
+        <gazebo reference="f_wheel_l">
+            <mu1>1.8</mu1>
+            <mu2>1.8</mu2>
+        </gazebo>
+        <gazebo reference="b_wheel_r">
+            <mu1>1.8</mu1>
+            <mu2>1.8</mu2>
+        </gazebo>
+        <gazebo reference="b_wheel_l">
+            <mu1>1.8</mu1>
+            <mu2>1.8</mu2>
+        </gazebo>
+<!-- ROS2_Control-Gazebo Plugin-->
+    <gazebo>
+        <plugin name="gazebo_ros2_control"
+                filename="libgazebo_ros2_control.so">
+        </plugin>
+    </gazebo>
+<!--ro2_control block-->
+    <ros2_control name="GazeboSystem" type="system">
+        <hardware>
+            <plugin>gazebo_ros2_control/GazeboSystem</plugin>
+        </hardware>
+        <!-- Front Step Mechanism -->
+        <joint name="base_link_front_link">
+            <command_interface name="position"/>
+            <state_interface name="position"/>
+            <state_interface name="velocity"/>
+        </joint>
+        <!-- Back Step Mechanism -->
+        <joint name="base_link_back_link">
+            <command_interface name="position"/>
+            <state_interface name="position"/>
+            <state_interface name="velocity"/>
+        </joint>
+        <!-- Front Right -->
+        <joint name="front_link_f_wheel_r">
+            <command_interface name="velocity"/>
+            <state_interface name="position"/>
+            <state_interface name="velocity"/>
+        </joint>
+        <!-- Front Left -->
+        <joint name="front_link_f_wheel_l">
+            <command_interface name="velocity"/>
+            <state_interface name="position"/>
+            <state_interface name="velocity"/>
+        </joint>
+        <!-- Back Right -->
+        <joint name="back_link_b_wheel_r">
+            <command_interface name="velocity"/>
+            <state_interface name="position"/>
+            <state_interface name="velocity"/>
+        </joint>
+        <!-- Back Left -->
+        <joint name="back_link_b_wheel_l">
+            <command_interface name="velocity"/>
+            <state_interface name="position"/>
+            <state_interface name="velocity"/>
+        </joint>
+        <!-- Vertical Expandable Right -->
+        <joint name="base_link_v_expandable_r">
+            <command_interface name="position"/>
+            <state_interface name="position"/>
+            <state_interface name="velocity"/>
+        </joint>
+        <!-- Vertical Expandable Left -->
+        <joint name="base_link_v_expandable_l">
+            <command_interface name="position"/>
+            <state_interface name="position"/>
+            <state_interface name="velocity"/>
+        </joint>
+        <!-- Vertical Gantry Right -->
+        <joint name="v_expandable_r_v_gantry_r">
+            <command_interface name="position"/>
+            <state_interface name="position"/>
+            <state_interface name="velocity"/>
+        </joint>
+        <!-- Vertical Gantry Left -->
+        <joint name="v_expandable_l_v_gantry_l">
+            <command_interface name="position"/>
+            <state_interface name="position"/>
+            <state_interface name="velocity"/>
+        </joint>
+        <!-- Horizontal Gantry Right -->
+        <joint name="h_expandable_r_h_gantry_r">
+            <command_interface name="position"/>
+            <state_interface name="position"/>
+            <state_interface name="velocity"/>
+        </joint>
+        <!-- Horizontal Gantry Left -->
+        <joint name="h_expandable_l_h_gantry_l">
+            <command_interface name="position"/>
+            <state_interface name="position"/>
+            <state_interface name="velocity"/>
+        </joint>
+    </ros2_control>
 </robot>

Commit message: Added Lidar Plugin

File: ros2_ws/src/r2_description/urdf/r2.xacro (robot description, xacro)
@@ -372,4 +372,31 @@
             <geometry>
                 <mesh filename="package://r2_description/meshes/camera_link.stl" scale="0.001 0.001 0.001" />
+            </geometry>
+        </collision>
+    </link>
+<!--LIDAR-->
+    <link name="lidar_link">
+        <inertial>
+            <origin xyz="0 0 0" rpy="0 0 0"/>
+            <mass value="0.2"/>
+            <inertia
+                ixx="0.0001"
+                ixy="0.0"
+                ixz="0.0"
+                iyy="0.0001"
+                iyz="0.0"
+                izz="0.0001"/>
+        </inertial>
+        <visual name="lidar_visual">
+            <origin xyz="0 0 0" rpy="0 0 0"/>
+            <geometry>
+                <cylinder radius="0.04" length="0.03"/>
+            </geometry>
+            <material name="camera_color"/>
+        </visual>
+        <collision name="lidar_collision">
+            <origin xyz="0 0 0" rpy="0 0 0"/>
+            <geometry>
+                <cylinder radius="0.04" length="0.03"/>
             </geometry>
         </collision>
@@ -527,4 +554,10 @@
         <child link="camera_link" />
         <axis xyz="0.0 3.944304526105059e-31 1.0" />
+    </joint>
+    <!--LIDAR Joint-->
+    <joint name="base_to_lidar" type="fixed">
+        <parent link="base_link"/>
+        <child link="lidar_link"/>
+        <origin xyz="0 0 -0.05" rpy="0 0 0"/>
     </joint>
     <!--Storage Plate Joint-->
@@ -578,4 +611,29 @@
         </sensor>
     </gazebo>
+<!--LIDAR Sensor Plugin-->
+    <gazebo reference="lidar_link">
+        <sensor name="lidar_sensor" type="ray">
+            <pose>0 0 0 0 0 0</pose>
+            <always_on>true</always_on>
+            <visualize>true</visualize>
+            <update_rate>10</update_rate>
+            <topic>scan</topic>
+            <ray>
+                <scan>
+                    <horizontal>
+                        <samples>720</samples>
+                        <resolution>1</resolution>
+                        <min_angle>-3.14159</min_angle>
+                        <max_angle>3.14159</max_angle>
+                    </horizontal>
+                </scan>
+                <range>
+                    <min>0.10</min>
+                    <max>12.0</max>
+                    <resolution>0.01</resolution>
+                </range>
+            </ray>
+        </sensor>
+    </gazebo>
 <!--ro2_control block-->
     <ros2_control name="GazeboSystem" type="system">

Commit message: Controller and Xacro update

File: ros2_ws/src/r2_description/urdf/r2.xacro (robot description, xacro)
@@ -619,10 +619,4 @@
     </joint>
     <!--horizontal Gantry and KFS Gripper-->
-    <joint name="h_gantry_right_kfs_gripper_gantry_r" type="fixed">
-        <origin xyz="-0.0325 -0.01 0.03739999999999998" rpy="0.0 -0.0 0.0" />
-        <parent link="h_gantry_r" />
-        <child link="kfs_gripper_link" />
-    </joint>
-    <!--
     <joint name="h_gantry_left_kfs_gripper_gantry_l" type="fixed">
         <origin xyz="-0.0325 0.01 0.03739999999999998" rpy="0.0 -0.0 0.0" />
@@ -630,5 +624,4 @@
         <child link="kfs_gripper_link" />
     </joint>
-    -->
     <!--KFS Finger Joint-->
     <joint name="kfs_gripper_link_kfs_finger_grip" type="prismatic">
@@ -656,5 +649,5 @@
     <!--Spearhead Revolute-->
     <joint name="kfs_gripper_link_spearhead_gripper_rotate" type="continuous">
-        <origin xyz="0.0 0.12 0.2125" rpy="+1.57 -0.0 0.0" />
+        <origin xyz="0.0 0.12 0.2125" rpy="0 0.0 1.5707963267948966" />
         <parent link="kfs_gripper_link" />
         <child link="spearhead_body" />

Commit message: Found the error

File: ros2_ws/src/r2_description/urdf/r2.xacro (robot description, xacro)
@@ -649,5 +649,5 @@
     <!--Spearhead Revolute-->
     <joint name="kfs_gripper_link_spearhead_gripper_rotate" type="continuous">
-        <origin xyz="0.0 0.12 0.2125" rpy="0 0.0 1.5707963267948966" />
+        <origin xyz="0.0 0.12 0.2125" rpy="3.14 3.14 0" />
         <parent link="kfs_gripper_link" />
         <child link="spearhead_body" />

Commit message: Spearhead joint connectec

File: ros2_ws/src/r2_description/urdf/r2.xacro (robot description, xacro)
@@ -387,10 +387,10 @@
     <link name="spearhead_body">
         <inertial>
-            <origin xyz="-0.10650436783393792 -4.818367926873193e-16 0.24498998848839812" rpy="0.0 0.0 0.0" />
-            <mass value="0.95" />
-            <inertia ixx="0.005634036903364744" iyy="0.0018508087267255472" izz="0.006850373035303052" ixy="7.817097663620531e-17" iyz="1.3346564094906206e-17" ixz="0.00018420936308609" />
+            <origin xyz="-0.08600436783393724 0.013989988488398665 1.2223417510293177e-15" rpy="0.0 -0.0 0.0" />
+            <mass value="1.4580482779771917" />
+            <inertia ixx="0.005634036903364975" iyy="0.006850373035303139" izz="0.0018508087267253698" ixy="0.00018420936308629482" iyz="-2.4978652552286308e-17" ixz="-1.9215332864481175e-16" />
         </inertial>
         <visual name="spearhead_body_visual">
-            <origin xyz="0.0 0.0 0.0" rpy="0.0 0.0 0.0" />
+            <origin xyz="0.02049999999999983 -0.23099999999999896 2.7081604932444613e-17" rpy="-1.5707963267948941 7.216449660063482e-16 -6.032465745807708e-32" />
             <geometry>
                 <mesh filename="package://r2_description/meshes/spearhead_body.stl" scale="0.001 0.001 0.001" />
@@ -398,5 +398,5 @@
         </visual>
         <collision name="spearhead_body_collision">
-            <origin xyz="0.0 0.0 0.0" rpy="0.0 0.0 0.0" />
+            <origin xyz="0.02049999999999983 -0.23099999999999896 2.7081604932444613e-17" rpy="-1.5707963267948941 7.216449660063482e-16 -6.032465745807708e-32" />
             <geometry>
                 <mesh filename="package://r2_description/meshes/spearhead_body.stl" scale="0.001 0.001 0.001" />
@@ -633,24 +633,24 @@
     </joint>
     <!--Spearhead Gripping Joint-->
+    <joint name="spearhead_body_spearhead_finger_l_grip" type="prismatic">
+        <origin xyz="-0.11199999999999999 0.025 -2.089831575765001e-18" rpy="3.141592653589793 1.4351862472329628e-62 3.4454487729021107e-46" />
+        <parent link="spearhead_body" />
+        <child link="spearhead_finger_l" />
+        <axis xyz="-1.4449768080836794e-62 0.0 1.0" />
+        <limit lower="0.0" upper="0.2" effort="100" velocity="1.0"/>
+    </joint>
     <joint name="spearhead_body_spearhead_finger_r_grip" type="prismatic">
-        <origin xyz="-0.10250000190230202 -2.8642330940353845e-09 0.2560000046766657" rpy="-1.5707963267948966 -0.0 0.0" />
+        <origin xyz="-0.08199999999999999 0.025 -2.089831575765001e-18" rpy="3.141592653589793 1.4351862472329628e-62 3.4454487729021107e-46" />
         <parent link="spearhead_body" />
         <child link="spearhead_finger_r" />
-        <axis xyz="0.0 -2.465190328815662e-32 1.0" />
-        <limit lower="0.0" upper="0.2" effort="100" velocity="1.0"/>
-    </joint>
-    <joint name="spearhead_body_spearhead_finger_l_grip" type="prismatic">
-        <origin xyz="-0.13250000190230193 -2.8642330940353845e-09 0.2560000046766657" rpy="-1.5707963267948966 -0.0 0.0" />
-        <parent link="spearhead_body" />
-        <child link="spearhead_finger_l" />
-        <axis xyz="0.0 -2.465190328815662e-32 1.0" />
+        <axis xyz="-1.4449768080836794e-62 0.0 1.0" />
         <limit lower="0.0" upper="0.2" effort="100" velocity="1.0"/>
     </joint>
     <!--Spearhead Revolute-->
     <joint name="kfs_gripper_link_spearhead_gripper_rotate" type="continuous">
-        <origin xyz="0.0 0.12 0.2125" rpy="3.14 3.14 0" />
+        <origin xyz="0.0 0.12 0.2125" rpy="-3.141592653589793 -0.0 0.0" />
         <parent link="kfs_gripper_link" />
         <child link="spearhead_body" />
-        <axis xyz="0.0 8.359326303060042e-17 1.0" />
+        <axis xyz="0.0 8.359326303060002e-17 1.0" />
     </joint>
     <!--CAMERA Rotation-->

Commit message: Still Editing Xacro for control

File: ros2_ws/src/r2_description/urdf/r2.xacro (robot description, xacro)
@@ -620,5 +620,5 @@
         <child link="h_gantry_l" />
         <axis xyz="0.0 1.0 0.0" />
-        <limit lower="-0.295" upper="0.295" effort="100" velocity="1.0"/>
+        <limit lower="0.295" upper="-0.295" effort="100" velocity="1.0"/>
         <dynamics damping="5.0" friction="1.0"/>
     </joint>

Commit message: Editing the urdf

File: ros2_ws/src/r2_description/urdf/r2.xacro (robot description, xacro)
@@ -611,5 +611,5 @@
         <parent link="h_expandable_r" />
         <child link="h_gantry_r" />
-        <axis xyz="0.0 0.0 1.0" />
+        <axis xyz="1.0 0.0 0.0" />
         <limit lower="-0.295" upper="0.295" effort="100" velocity="1.0"/>
         <dynamics damping="5.0" friction="1.0"/>
@@ -619,6 +619,6 @@
         <parent link="h_expandable_l" />
         <child link="h_gantry_l" />
-        <axis xyz="0.0 1.0 0.0" />
-        <limit lower="0.295" upper="-0.295" effort="100" velocity="1.0"/>
+        <axis xyz="1.0 0.0 0.0" />
+        <limit lower="-0.295" upper="0.295" effort="100" velocity="1.0"/>
         <dynamics damping="5.0" friction="1.0"/>
     </joint>

Commit message: Adding gantry bridge to the urf

File: ros2_ws/src/r2_description/urdf/r2.xacro (robot description, xacro)
@@ -193,39 +193,57 @@
     <link name="h_gantry_r">
         <inertial>
-            <origin xyz="0.0 0.013832853025936558 0.02363371757925073" rpy="0.0 -0.0 0.0" />
-            <mass value="0.187" />
-            <inertia ixx="0.00028625336112315936" iyy="0.000320958411897658" izz="0.0004640047950588283" ixy="1.2494183465605601e-18" iyz="-5.6491115619582144e-05" ixz="8.031975085032172e-19" />
+            <origin xyz="0.0 -7.105427357601002e-17 0.005000000000000071" rpy="0.0 -0.0 0.0" />
+            <mass value="0.10204999999999999" />
+            <inertia ixx="4.252083333333018e-06" iyy="3.678052083333234e-05" izz="3.9331770833336485e-05" ixy="0.0" iyz="0.0" ixz="0.0" />
         </inertial>
         <visual name="h_gantry_r_visual">
             <origin xyz="0.0 0.34600000000000003 0.24989999999999998" rpy="1.5707963267948966 -0.0 0.0" />
             <geometry>
-                <mesh filename="package://r2_description/meshes/h_gantry_r.stl" scale="0.001 0.001 0.001" />
-            </geometry>
-            <material name="gantry_color"/>
+                <mesh filename="meshes/h_gantry_r.stl" scale="0.001 0.001 0.001" />
+            </geometry>
         </visual>
         <collision name="h_gantry_r_collision">
             <origin xyz="0.0 0.34600000000000003 0.24989999999999998" rpy="1.5707963267948966 -0.0 0.0" />
             <geometry>
-                <mesh filename="package://r2_description/meshes/h_gantry_r.stl" scale="0.001 0.001 0.001" />
-            </geometry>
-        </collision>
-    </link>
-    <link name="h_gantry_l">
-        <inertial>
-            <origin xyz="0.0 -0.013832853025936629 0.023633717579250695" rpy="0.0 -0.0 0.0" />
-            <mass value="0.187" />
-            <inertia ixx="0.00028625336112317323" iyy="0.0003209584118976441" izz="0.0004640047950588283" ixy="-1.7848833522293717e-19" iyz="5.6491115619575205e-05" ixz="-8.924416761146858e-20" />
-        </inertial>
-        <visual name="h_gantry_l_visual">
+                <mesh filename="meshes/h_gantry_r.stl" scale="0.001 0.001 0.001" />
+            </geometry>
+        </collision>
+    </link>
+    <link name="h_ganty_l">
+        <inertial>
+            <origin xyz="0.0 -7.105427357601002e-17 0.005000000000000071" rpy="0.0 -0.0 0.0" />
+            <mass value="0.10204999999999999" />
+            <inertia ixx="4.252083333333018e-06" iyy="3.678052083333234e-05" izz="3.9331770833333016e-05" ixy="1.7848833522293717e-19" iyz="1.734723475976807e-18" ixz="0.0" />
+        </inertial>
+        <visual name="h_ganty_l_visual">
             <origin xyz="0.0 -0.34600000000000003 0.24989999999999998" rpy="-1.5707963267948966 -0.0 0.0" />
             <geometry>
-                <mesh filename="package://r2_description/meshes/h_gantry_l.stl" scale="0.001 0.001 0.001" />
-            </geometry>
-            <material name="gantry_color"/>
-        </visual>
-        <collision name="h_gantry_l_collision">
+                <mesh filename="meshes/h_ganty_l.stl" scale="0.001 0.001 0.001" />
+            </geometry>
+        </visual>
+        <collision name="h_ganty_l_collision">
             <origin xyz="0.0 -0.34600000000000003 0.24989999999999998" rpy="-1.5707963267948966 -0.0 0.0" />
             <geometry>
-                <mesh filename="package://r2_description/meshes/h_gantry_l.stl" scale="0.001 0.001 0.001" />
+                <mesh filename="meshes/h_ganty_l.stl" scale="0.001 0.001 0.001" />
+            </geometry>
+        </collision>
+    </link>
+<!-- Gantry Bridge -->
+    <link name="gantry_bridge">
+        <inertial>
+            <origin xyz="0.0 7.105427357601002e-17 0.2399" rpy="0.0 -0.0 0.0" />
+            <mass value="1.506572" />
+            <inertia ixx="0.02895230133657334" iyy="0.028952301336573342" izz="0.00010043813333332485" ixy="4.462208380573429e-20" iyz="-9.281393431592732e-18" ixz="0.0" />
+        </inertial>
+        <visual name="gantry_bridge_visual">
+            <origin xyz="0.0 -0.34600000000000003 0.2399" rpy="-1.5707963267948966 -0.0 0.0" />
+            <geometry>
+                <mesh filename="meshes/gantry_bridge.stl" scale="0.001 0.001 0.001" />
+            </geometry>
+        </visual>
+        <collision name="gantry_bridge_collision">
+            <origin xyz="0.0 -0.34600000000000003 0.2399" rpy="-1.5707963267948966 -0.0 0.0" />
+            <geometry>
+                <mesh filename="meshes/gantry_bridge.stl" scale="0.001 0.001 0.001" />
             </geometry>
         </collision>
@@ -607,19 +625,18 @@
     </joint>
     <!--Horizontal Expandable-->
-    <joint name="h_expandable_r_h_gantry_r" type="prismatic">
-        <origin xyz="0.0 0.0 0.02" rpy="0.0 -0.0 0.0" />
-        <parent link="h_expandable_r" />
+    <joint name="h_ganty_l_gantry_bridge_h_gantry_l" type="fixed">
+        <origin xyz="0.0 0.0 0.01" rpy="0.0 -0.0 0.0" />
+        <parent link="h_ganty_l" />
+        <child link="gantry_bridge" />
+    </joint>
+    <joint name="gantry_bridge_gantry_bridge_h_gantry_l-1" type="fixed">
+        <origin xyz="0.0 0.0 0.4798" rpy="0.0 -0.0 0.0" />
+        <parent link="gantry_bridge" />
         <child link="h_gantry_r" />
-        <axis xyz="1.0 0.0 0.0" />
-        <limit lower="-0.295" upper="0.295" effort="100" velocity="1.0"/>
-        <dynamics damping="5.0" friction="1.0"/>
-    </joint>
-    <joint name="h_expandable_l_h_gantry_l" type="prismatic">
-        <origin xyz="0.0 0.0 0.02" rpy="0.0 0.0 0.0" />
-        <parent link="h_expandable_l" />
-        <child link="h_gantry_l" />
-        <axis xyz="1.0 0.0 0.0" />
-        <limit lower="-0.295" upper="0.295" effort="100" velocity="1.0"/>
-        <dynamics damping="5.0" friction="1.0"/>
+    </joint>
+    <joint name="gantry_bridge_kfs_gripper_joint" type="fixed">
+        <origin xyz="0.01 0.0 0.2399" rpy="1.5707963267948966 -0.0 1.5707963267948966" />
+        <parent link="gantry_bridge" />
+        <child link="kfs_gripper_link" />
     </joint>
     <!--horizontal Gantry and KFS Gripper-->
