Commit message: Uploading the edits

File: ros2_ws/src/r2_description/urdf/r2.xacro (robot description, xacro)
@@ -210,5 +210,5 @@
         </collision>
     </link>
-    <link name="h_ganty_l">
+    <link name="h_gantry_l">
         <inertial>
             <origin xyz="0.0 -7.105427357601002e-17 0.005000000000000071" rpy="0.0 -0.0 0.0" />
@@ -219,5 +219,5 @@
             <origin xyz="0.0 -0.34600000000000003 0.24989999999999998" rpy="-1.5707963267948966 -0.0 0.0" />
             <geometry>
-                <mesh filename="meshes/h_ganty_l.stl" scale="0.001 0.001 0.001" />
+                <mesh filename="meshes/h_gantry_l.stl" scale="0.001 0.001 0.001" />
             </geometry>
         </visual>
@@ -225,5 +225,5 @@
             <origin xyz="0.0 -0.34600000000000003 0.24989999999999998" rpy="-1.5707963267948966 -0.0 0.0" />
             <geometry>
-                <mesh filename="meshes/h_ganty_l.stl" scale="0.001 0.001 0.001" />
+                <mesh filename="meshes/h_gantry_l.stl" scale="0.001 0.001 0.001" />
             </geometry>
         </collision>
@@ -625,23 +625,30 @@
     </joint>
     <!--Horizontal Expandable-->
-    <joint name="h_ganty_l_gantry_bridge_h_gantry_l" type="fixed">
+    <joint name="h_expandable_r_h_gantry_r" type="prismatic">
+        <origin xyz="0.0 0.0 0.02" rpy="0.0 -0.0 0.0" />
+        <parent link="h_expandable_r" />
+        <child link="h_gantry_r" />
+        <axis xyz="1.0 0.0 0.0" />
+    </joint>
+    <joint name="h_expandable_l_h_gantry_l" type="prismatic">
+        <origin xyz="0.0 0.0 0.02" rpy="0.0 -0.0 0.0" />
+        <parent link="h_expandable_l" />
+        <child link="h_gantry_l" />
+        <axis xyz="1.0 0.0 0.0" />
+    </joint>
+    <joint name="h_gantry_l_gantry_bridge" type="fixed">
         <origin xyz="0.0 0.0 0.01" rpy="0.0 -0.0 0.0" />
-        <parent link="h_ganty_l" />
+        <parent link="h_gantry_l" />
         <child link="gantry_bridge" />
     </joint>
-    <joint name="gantry_bridge_gantry_bridge_h_gantry_l-1" type="fixed">
+    <joint name="gantry_bridge_h_gantry_l-1" type="fixed">
         <origin xyz="0.0 0.0 0.4798" rpy="0.0 -0.0 0.0" />
         <parent link="gantry_bridge" />
         <child link="h_gantry_r" />
     </joint>
+<!-- KFS Gripper Joint -->
     <joint name="gantry_bridge_kfs_gripper_joint" type="fixed">
         <origin xyz="0.01 0.0 0.2399" rpy="1.5707963267948966 -0.0 1.5707963267948966" />
         <parent link="gantry_bridge" />
-        <child link="kfs_gripper_link" />
-    </joint>
-    <!--horizontal Gantry and KFS Gripper-->
-    <joint name="h_gantry_left_kfs_gripper_gantry_l" type="fixed">
-        <origin xyz="-0.0325 0.01 0.03739999999999998" rpy="0.0 0.0 0.0" />
-        <parent link="h_gantry_l" />
         <child link="kfs_gripper_link" />
     </joint>

Commit message: Editing xacro

File: ros2_ws/src/r2_description/urdf/r2.xacro (robot description, xacro)
@@ -216,5 +216,5 @@
             <inertia ixx="4.252083333333018e-06" iyy="3.678052083333234e-05" izz="3.9331770833333016e-05" ixy="1.7848833522293717e-19" iyz="1.734723475976807e-18" ixz="0.0" />
         </inertial>
-        <visual name="h_ganty_l_visual">
+        <visual name="h_gantry_l_visual">
             <origin xyz="0.0 -0.34600000000000003 0.24989999999999998" rpy="-1.5707963267948966 -0.0 0.0" />
             <geometry>
@@ -222,5 +222,5 @@
             </geometry>
         </visual>
-        <collision name="h_ganty_l_collision">
+        <collision name="h_gantry_l_collision">
             <origin xyz="0.0 -0.34600000000000003 0.24989999999999998" rpy="-1.5707963267948966 -0.0 0.0" />
             <geometry>
@@ -381,4 +381,24 @@
             <geometry>
                 <mesh filename="package://r2_description/meshes/kfs_finger.stl" scale="0.001 0.001 0.001" />
+            </geometry>
+        </collision>
+    </link>
+<!--Speahred support Horizontal Tubing-->
+    <link name="horizontal_tubing">
+        <inertial>
+            <origin xyz="-0.00999999999993996 -0.2698999999999995 0.009999996448131796" rpy="0.0 -0.0 0.0" />
+            <mass value="1.4819755366703677" />
+            <inertia ixx="0.03604098200232858" iyy="0.00011129416173860651" izz="0.03604098200210676" ixy="-7.487776782399223e-18" iyz="2.5179661329231423e-19" ixz="-8.326672684688674e-17" />
+        </inertial>
+        <visual name="horizontal_tubing_visual">
+            <origin xyz="-0.375 -0.2698999999999995 -0.3560000035518682" rpy="-1.7182958789296736e-16 2.465190328815662e-32 -3.141592653589793" />
+            <geometry>
+                <mesh filename="package://r2_description/meshes/horizontal_tubing.stl" scale="0.001 0.001 0.001" />
+            </geometry>
+        </visual>
+        <collision name="horizontal_tubing_collision">
+            <origin xyz="-0.375 -0.2698999999999995 -0.3560000035518682" rpy="-1.7182958789296736e-16 2.465190328815662e-32 -3.141592653589793" />
+            <geometry>
+                <mesh filename="package://r2_description/meshes/horizontal_tubing.stl" scale="0.001 0.001 0.001" />
             </geometry>
         </collision>
@@ -641,5 +661,5 @@
         <child link="spearhead_finger_l" />
         <axis xyz="-1.4449768080836794e-62 0.0 1.0" />
-        <limit lower="-0.02896" upper="-0.08765" effort="100" velocity="1.0"/>
+        <limit lower="-0.08765" upper="-0.02896" effort="100" velocity="1.0"/>
     </joint>
     <joint name="spearhead_body_spearhead_finger_r_grip" type="prismatic">
@@ -648,12 +668,12 @@
         <child link="spearhead_finger_r" />
         <axis xyz="-1.4449768080836794e-62 0.0 1.0" />
-        <limit lower="-0.02896" upper="-0.08765" effort="100" velocity="1.0"/>
+        <limit lower="0.02896" upper="0.08765" effort="100" velocity="1.0"/>
     </joint>
     <!--Spearhead Revolute-->
-    <joint name="kfs_gripper_link_spearhead_gripper_rotate" type="continuous">
-        <origin xyz="0.0 0.12 0.2125" rpy="-3.141592653589793 -0.0 1.1869459682199748e-66" />
-        <parent link="kfs_gripper_link" />
+    <joint name="horizontal_tubing_spearhead_gripper_rotation" type="revolute">
+        <origin xyz="0.0 -0.2699 0.02" rpy="1.5707963267948966 -0.0 -3.141592653589793" />
+        <parent link="horizontal_tubing" />
         <child link="spearhead_body" />
-        <axis xyz="0.0 8.359326303060042e-17 1.0" />
+        <axis xyz="-4.235926382781239e-48 0.0 1.0" />
         <limit lower="-1.5707963267948966" upper="1.5707963267948966" effort="100" velocity="1.0"/>
     </joint>

Commit message: Rewrote the code before gantry bridge

File: ros2_ws/src/r2_description/urdf/r2.xacro (robot description, xacro)
@@ -193,18 +193,19 @@
     <link name="h_gantry_r">
         <inertial>
-            <origin xyz="0.0 -7.105427357601002e-17 0.005000000000000071" rpy="0.0 -0.0 0.0" />
-            <mass value="0.10204999999999999" />
-            <inertia ixx="4.252083333333018e-06" iyy="3.678052083333234e-05" izz="3.9331770833336485e-05" ixy="0.0" iyz="0.0" ixz="0.0" />
+            <origin xyz="0.0 0.013832853025936558 0.02363371757925073" rpy="0.0 -0.0 0.0" />
+            <mass value="0.187" />
+            <inertia ixx="0.00028625336112315936" iyy="0.000320958411897658" izz="0.0004640047950588283" ixy="1.2494183465605601e-18" iyz="-5.6491115619582144e-05" ixz="8.031975085032172e-19" />
         </inertial>
         <visual name="h_gantry_r_visual">
             <origin xyz="0.0 0.34600000000000003 0.24989999999999998" rpy="1.5707963267948966 -0.0 0.0" />
             <geometry>
-                <mesh filename="meshes/h_gantry_r.stl" scale="0.001 0.001 0.001" />
-            </geometry>
+                <mesh filename="package://r2_description/meshes/h_gantry_r.stl" scale="0.001 0.001 0.001" />
+            </geometry>
+            <material name="gantry_color"/>
         </visual>
         <collision name="h_gantry_r_collision">
             <origin xyz="0.0 0.34600000000000003 0.24989999999999998" rpy="1.5707963267948966 -0.0 0.0" />
             <geometry>
-                <mesh filename="meshes/h_gantry_r.stl" scale="0.001 0.001 0.001" />
+                <mesh filename="package://r2_description/meshes/h_gantry_r.stl" scale="0.001 0.001 0.001" />
             </geometry>
         </collision>
@@ -212,18 +213,19 @@
     <link name="h_gantry_l">
         <inertial>
-            <origin xyz="0.0 -7.105427357601002e-17 0.005000000000000071" rpy="0.0 -0.0 0.0" />
-            <mass value="0.10204999999999999" />
-            <inertia ixx="4.252083333333018e-06" iyy="3.678052083333234e-05" izz="3.9331770833333016e-05" ixy="1.7848833522293717e-19" iyz="1.734723475976807e-18" ixz="0.0" />
+            <origin xyz="0.0 -0.013832853025936629 0.023633717579250695" rpy="0.0 -0.0 0.0" />
+            <mass value="0.187" />
+            <inertia ixx="0.00028625336112317323" iyy="0.0003209584118976441" izz="0.0004640047950588283" ixy="-1.7848833522293717e-19" iyz="5.6491115619575205e-05" ixz="-8.924416761146858e-20" />
         </inertial>
         <visual name="h_gantry_l_visual">
             <origin xyz="0.0 -0.34600000000000003 0.24989999999999998" rpy="-1.5707963267948966 -0.0 0.0" />
             <geometry>
-                <mesh filename="meshes/h_gantry_l.stl" scale="0.001 0.001 0.001" />
-            </geometry>
+                <mesh filename="package://r2_description/meshes/h_gantry_l.stl" scale="0.001 0.001 0.001" />
+            </geometry>
+            <material name="gantry_color"/>
         </visual>
         <collision name="h_gantry_l_collision">
             <origin xyz="0.0 -0.34600000000000003 0.24989999999999998" rpy="-1.5707963267948966 -0.0 0.0" />
             <geometry>
-                <mesh filename="meshes/h_gantry_l.stl" scale="0.001 0.001 0.001" />
+                <mesh filename="package://r2_description/meshes/h_gantry_l.stl" scale="0.001 0.001 0.001" />
             </geometry>
         </collision>
@@ -381,24 +383,4 @@
             <geometry>
                 <mesh filename="package://r2_description/meshes/kfs_finger.stl" scale="0.001 0.001 0.001" />
-            </geometry>
-        </collision>
-    </link>
-<!--Speahred support Horizontal Tubing-->
-    <link name="horizontal_tubing">
-        <inertial>
-            <origin xyz="-0.00999999999993996 -0.2698999999999995 0.009999996448131796" rpy="0.0 -0.0 0.0" />
-            <mass value="1.4819755366703677" />
-            <inertia ixx="0.03604098200232858" iyy="0.00011129416173860651" izz="0.03604098200210676" ixy="-7.487776782399223e-18" iyz="2.5179661329231423e-19" ixz="-8.326672684688674e-17" />
-        </inertial>
-        <visual name="horizontal_tubing_visual">
-            <origin xyz="-0.375 -0.2698999999999995 -0.3560000035518682" rpy="-1.7182958789296736e-16 2.465190328815662e-32 -3.141592653589793" />
-            <geometry>
-                <mesh filename="package://r2_description/meshes/horizontal_tubing.stl" scale="0.001 0.001 0.001" />
-            </geometry>
-        </visual>
-        <collision name="horizontal_tubing_collision">
-            <origin xyz="-0.375 -0.2698999999999995 -0.3560000035518682" rpy="-1.7182958789296736e-16 2.465190328815662e-32 -3.141592653589793" />
-            <geometry>
-                <mesh filename="package://r2_description/meshes/horizontal_tubing.stl" scale="0.001 0.001 0.001" />
             </geometry>
         </collision>
@@ -629,20 +611,20 @@
         <parent link="h_expandable_r" />
         <child link="h_gantry_r" />
-        <axis xyz="1.0 0.0 0.0" />
-        <limit lower="0.0" upper="0.2" effort="100" velocity="1.0"/>
+        <axis xyz="0.0 0.0 1.0" />
+        <limit lower="-0.295" upper="0.295" effort="100" velocity="1.0"/>
         <dynamics damping="5.0" friction="1.0"/>
     </joint>
     <joint name="h_expandable_l_h_gantry_l" type="prismatic">
-        <origin xyz="0.0 0.0 0.02" rpy="0.0 -0.0 0.0" />
+        <origin xyz="0.0 0.0 0.02" rpy="0.0 0.0 0.0" />
         <parent link="h_expandable_l" />
         <child link="h_gantry_l" />
-        <axis xyz="1.0 0.0 0.0" />
-        <limit lower="0.0" upper="0.2" effort="100" velocity="1.0"/>
+        <axis xyz="0.0 1.0 0.0" />
+        <limit lower="0.295" upper="-0.295" effort="100" velocity="1.0"/>
         <dynamics damping="5.0" friction="1.0"/>
     </joint>
     <!--horizontal Gantry and KFS Gripper-->
-    <joint name="h_gantry_r_kfs_gripper_gantry_r" type="fixed">
-        <origin xyz="-0.0325 -0.01 0.03739999999999998" rpy="0.0 -0.0 0.0" />
-        <parent link="h_gantry_r" />
+    <joint name="h_gantry_left_kfs_gripper_gantry_l" type="fixed">
+        <origin xyz="-0.0325 0.01 0.03739999999999998" rpy="0.0 0.0 0.0" />
+        <parent link="h_gantry_l" />
         <child link="kfs_gripper_link" />
     </joint>
@@ -661,5 +643,5 @@
         <child link="spearhead_finger_l" />
         <axis xyz="-1.4449768080836794e-62 0.0 1.0" />
-        <limit lower="-0.08765" upper="-0.02896" effort="100" velocity="1.0"/>
+        <limit lower="-0.02896" upper="-0.08765" effort="100" velocity="1.0"/>
     </joint>
     <joint name="spearhead_body_spearhead_finger_r_grip" type="prismatic">
@@ -668,12 +650,12 @@
         <child link="spearhead_finger_r" />
         <axis xyz="-1.4449768080836794e-62 0.0 1.0" />
-        <limit lower="0.02896" upper="0.08765" effort="100" velocity="1.0"/>
+        <limit lower="-0.02896" upper="-0.08765" effort="100" velocity="1.0"/>
     </joint>
     <!--Spearhead Revolute-->
-    <joint name="horizontal_tubing_spearhead_gripper_rotation" type="revolute">
-        <origin xyz="0.0 -0.2699 0.02" rpy="1.5707963267948966 -0.0 -3.141592653589793" />
-        <parent link="horizontal_tubing" />
+    <joint name="kfs_gripper_link_spearhead_gripper_rotate" type="revolute">
+        <origin xyz="0.0 0.12 0.2125" rpy="-3.141592653589793 -0.0 0.0" />
+        <parent link="kfs_gripper_link" />
         <child link="spearhead_body" />
-        <axis xyz="-4.235926382781239e-48 0.0 1.0" />
+        <axis xyz="0.0 8.359326303060002e-17 1.0" />
         <limit lower="-1.5707963267948966" upper="1.5707963267948966" effort="100" velocity="1.0"/>
     </joint>
