Commit message: Editing the xacro and launch file

File: ros2_ws/src/r2_description/urdf/r2.xacro (robot description, xacro)
@@ -5,4 +5,6 @@
   <!-- Include gazebo -->
   <xacro:include filename="$(find r2_description)/urdf/gazebo.xacro"/>
+<!--Odometry-->
+<link name="odom"/>
 <!-- Base Link-->
     <link name="base_link">
@@ -15,5 +17,5 @@
             <origin xyz="0.0 0.0 0.0" rpy="0.0 0.0 0.0" />
             <geometry>
-                <mesh filename="package://r2_description/meshes/base_link.stl" scale="0.001 0.001 0.001" />
+                <mesh filename="file://$(find r2_description)/meshes/base_link.stl" scale="0.001 0.001 0.001" />
             </geometry>
             <material name="base_color"/>
@@ -22,5 +24,5 @@
             <origin xyz="0.0 0.0 0.0" rpy="0.0 0.0 0.0" />
             <geometry>
-                <mesh filename="package://r2_description/meshes/base_link.stl" scale="0.001 0.001 0.001" />
+                <box size="0.63 0.65 0.08"/>
             </geometry>
         </collision>
@@ -36,5 +38,5 @@
             <origin xyz="-0.23800000000000002 0.0 -0.006025000000000001" rpy="3.141592653589793 -0.0 0.0" />
             <geometry>
-                <mesh filename="package://r2_description/meshes/front_link.stl" scale="0.001 0.001 0.001" />
+                <mesh filename="file://$(find r2_description)/meshes/front_link.stl" scale="0.001 0.001 0.001" />
             </geometry>
             <material name="chassis_color"/>
@@ -43,5 +45,5 @@
             <origin xyz="-0.23800000000000002 0.0 -0.006025000000000001" rpy="3.141592653589793 -0.0 0.0" />
             <geometry>
-                <mesh filename="package://r2_description/meshes/front_link.stl" scale="0.001 0.001 0.001" />
+                <box size="0.154 0.594 0.10"/>
             </geometry>
         </collision>
@@ -57,5 +59,5 @@
             <origin xyz="0.23800000000000002 0.0 -0.006025000000000001" rpy="3.141592653589793 -0.0 0.0" />
             <geometry>
-                <mesh filename="package://r2_description/meshes/back_link.stl" scale="0.001 0.001 0.001" />
+                <mesh filename="file://$(find r2_description)/meshes/back_link.stl" scale="0.001 0.001 0.001" />
             </geometry>
             <material name="chassis_color"/>
@@ -64,5 +66,5 @@
             <origin xyz="0.23800000000000002 0.0 -0.006025000000000001" rpy="3.141592653589793 -0.0 0.0" />
             <geometry>
-                <mesh filename="package://r2_description/meshes/back_link.stl" scale="0.001 0.001 0.001" />
+                <box size="0.154 0.594 0.10"/>
             </geometry>
         </collision>
@@ -78,5 +80,5 @@
             <origin xyz="-7.105427357601002e-17 -0.45599999999999946 0.3069999999999998" rpy="1.5707963267948966 -6.938893903907214e-18 3.141592653589793" />
             <geometry>
-                <mesh filename="package://r2_description/meshes/v_expandable_r.stl" scale="0.001 0.001 0.001" />
+                <mesh filename="file://$(find r2_description)/meshes/v_expandable_r.stl" scale="0.001 0.001 0.001" />
             </geometry>
             <material name="expandable_color"/>
@@ -85,5 +87,5 @@
             <origin xyz="-7.105427357601002e-17 -0.45599999999999946 0.3069999999999998" rpy="1.5707963267948966 -6.938893903907214e-18 3.141592653589793" />
             <geometry>
-                <mesh filename="package://r2_description/meshes/v_expandable_r.stl" scale="0.001 0.001 0.001" />
+                <box size="0.04 0.168 0.08"/>
             </geometry>
         </collision>
@@ -98,5 +100,5 @@
             <origin xyz="-7.105427357601002e-17 -0.45600000000000007 0.3069999999999999" rpy="-1.5707963267948957 1.3877787807814443e-17 -1.2246467991473532e-16" />
             <geometry>
-                <mesh filename="package://r2_description/meshes/v_expandable_l.stl" scale="0.001 0.001 0.001" />
+                <mesh filename="file://$(find r2_description)/meshes/v_expandable_l.stl" scale="0.001 0.001 0.001" />
             </geometry>
             <material name="expandable_color"/>
@@ -105,5 +107,5 @@
             <origin xyz="-7.105427357601002e-17 -0.45600000000000007 0.3069999999999999" rpy="-1.5707963267948957 1.3877787807814443e-17 -1.2246467991473532e-16" />
             <geometry>
-                <mesh filename="package://r2_description/meshes/v_expandable_l.stl" scale="0.001 0.001 0.001" />
+                <box size="0.04 0.168 0.08"/>
             </geometry>
         </collision>
@@ -119,5 +121,5 @@
             <origin xyz="6.042827863252935e-17 0.2824999999999999 0.26990000000000003" rpy="1.5707963267948966 -0.0 -1.2246467991473532e-16" />
             <geometry>
-                <mesh filename="package://r2_description/meshes/h_expandable_r.stl" scale="0.001 0.001 0.001" />
+                <mesh filename="file://$(find r2_description)/meshes/h_expandable_r.stl" scale="0.001 0.001 0.001" />
             </geometry>
             <material name="expandable_color"/>
@@ -126,5 +128,5 @@
             <origin xyz="6.042827863252935e-17 0.2824999999999999 0.26990000000000003" rpy="1.5707963267948966 -0.0 -1.2246467991473532e-16" />
             <geometry>
-                <mesh filename="package://r2_description/meshes/h_expandable_r.stl" scale="0.001 0.001 0.001" />
+                <box size="0.32 0.04 0.04"/>
             </geometry>
         </collision>
@@ -139,5 +141,5 @@
             <origin xyz="-6.153850165715452e-17 -0.28250000000000003 0.26990000000000003" rpy="-1.5707963267948966 -0.0 -1.2246467991473532e-16" />
             <geometry>
-                <mesh filename="package://r2_description/meshes/h_expandable_l.stl" scale="0.001 0.001 0.001" />
+                <mesh filename="file://$(find r2_description)/meshes/h_expandable_l.stl" scale="0.001 0.001 0.001" />
             </geometry>
             <material name="expandable_color"/>
@@ -146,5 +148,5 @@
             <origin xyz="-6.153850165715452e-17 -0.28250000000000003 0.26990000000000003" rpy="-1.5707963267948966 -0.0 -1.2246467991473532e-16" />
             <geometry>
-                <mesh filename="package://r2_description/meshes/h_expandable_l.stl" scale="0.001 0.001 0.001" />
+                <box size="0.32 0.04 0.04"/>
             </geometry>
         </collision>
@@ -160,5 +162,5 @@
             <origin xyz="6.042827863252935e-17 0.2824999999999999 0.28700000000000003" rpy="1.5707963267948966 -4.479329460506078e-34 -1.2246467991473532e-16" />
             <geometry>
-                <mesh filename="package://r2_description/meshes/v_gantry_r.stl" scale="0.001 0.001 0.001" />
+                <mesh filename="file://$(find r2_description)/meshes/v_gantry_r.stl" scale="0.001 0.001 0.001" />
             </geometry>
             <material name="gantry_color"/>
@@ -167,5 +169,5 @@
             <origin xyz="6.042827863252935e-17 0.2824999999999999 0.28700000000000003" rpy="1.5707963267948966 -4.479329460506078e-34 -1.2246467991473532e-16" />
             <geometry>
-                <mesh filename="package://r2_description/meshes/v_gantry_r.stl" scale="0.001 0.001 0.001" />
+                <box size="0.04 0.168 0.12"/>
             </geometry>
         </collision>
@@ -180,5 +182,5 @@
             <origin xyz="-6.153850165715452e-17 -0.28250000000000003 0.28700000000000003" rpy="-1.5707963267948966 1.1947622849140125e-34 -1.2246467991473532e-16" />
             <geometry>
-                <mesh filename="package://r2_description/meshes/v_gantry_l.stl" scale="0.001 0.001 0.001" />
+                <mesh filename="file://$(find r2_description)/meshes/v_gantry_l.stl" scale="0.001 0.001 0.001" />
             </geometry>
             <material name="gantry_color"/>
@@ -187,5 +189,5 @@
             <origin xyz="-6.153850165715452e-17 -0.28250000000000003 0.28700000000000003" rpy="-1.5707963267948966 1.1947622849140125e-34 -1.2246467991473532e-16" />
             <geometry>
-                <mesh filename="package://r2_description/meshes/v_gantry_l.stl" scale="0.001 0.001 0.001" />
+                <box size="0.04 0.168 0.12"/>
             </geometry>
         </collision>
@@ -200,5 +202,5 @@
             <origin xyz="0.0 0.34600000000000003 0.24989999999999998" rpy="1.5707963267948966 -0.0 0.0" />
             <geometry>
-                <mesh filename="package://r2_description/meshes/h_gantry_r.stl" scale="0.001 0.001 0.001" />
+                <mesh filename="file://$(find r2_description)/meshes/h_gantry_r.stl" scale="0.001 0.001 0.001" />
             </geometry>
             <material name="gantry_color"/>
@@ -207,5 +209,5 @@
             <origin xyz="0.0 0.34600000000000003 0.24989999999999998" rpy="1.5707963267948966 -0.0 0.0" />
             <geometry>
-                <mesh filename="package://r2_description/meshes/h_gantry_r.stl" scale="0.001 0.001 0.001" />
+                <box size="0.45 0.04 0.04"/>
             </geometry>
         </collision>
@@ -220,5 +222,5 @@
             <origin xyz="0.0 -0.34600000000000003 0.24989999999999998" rpy="-1.5707963267948966 -0.0 0.0" />
             <geometry>
-                <mesh filename="package://r2_description/meshes/h_gantry_l.stl" scale="0.001 0.001 0.001" />
+                <mesh filename="file://$(find r2_description)/meshes/h_gantry_l.stl" scale="0.001 0.001 0.001" />
             </geometry>
             <material name="gantry_color"/>
@@ -227,5 +229,5 @@
             <origin xyz="0.0 -0.34600000000000003 0.24989999999999998" rpy="-1.5707963267948966 -0.0 0.0" />
             <geometry>
-                <mesh filename="package://r2_description/meshes/h_gantry_l.stl" scale="0.001 0.001 0.001" />
+                <box size="0.45 0.04 0.04"/>
             </geometry>
         </collision>
@@ -241,5 +243,5 @@
             <origin xyz="-0.23800000000000002 0.044524999999999995 -0.2715" rpy="-1.5707963267948966 -0.0 0.0" />
             <geometry>
-                <mesh filename="package://r2_description/meshes/f_wheel_r.stl" scale="0.001 0.001 0.001" />
+                <mesh filename="file://$(find r2_description)/meshes/f_wheel_r.stl" scale="0.001 0.001 0.001" />
             </geometry>
             <material name="wheel_color"/>
@@ -248,5 +250,5 @@
             <origin xyz="-0.23800000000000002 0.044524999999999995 -0.2715" rpy="-1.5707963267948966 -0.0 0.0" />
             <geometry>
-                <mesh filename="package://r2_description/meshes/f_wheel_r.stl" scale="0.001 0.001 0.001" />
+                <cylinder length="0.08" radius="0.0625"/>
             </geometry>
             <surface>
@@ -269,5 +271,5 @@
             <origin xyz="-0.23800000000000002 -0.044524999999999995 -0.2715" rpy="1.5707963267948966 -0.0 0.0" />
             <geometry>
-                <mesh filename="package://r2_description/meshes/f_wheel_l.stl" scale="0.001 0.001 0.001" />
+                <mesh filename="file://$(find r2_description)/meshes/f_wheel_l.stl" scale="0.001 0.001 0.001" />
             </geometry>
             <material name="wheel_color"/>
@@ -276,5 +278,5 @@
             <origin xyz="-0.23800000000000002 -0.044524999999999995 -0.2715" rpy="1.5707963267948966 -0.0 0.0" />
             <geometry>
-                <mesh filename="package://r2_description/meshes/f_wheel_l.stl" scale="0.001 0.001 0.001" />
+                <cylinder length="0.08" radius="0.0625"/>
             </geometry>
             <surface>
@@ -297,5 +299,5 @@
             <origin xyz="0.23800000000000002 0.044524999999999995 -0.2735" rpy="-1.5707963267948966 -0.0 0.0" />
             <geometry>
-                <mesh filename="package://r2_description/meshes/b_wheel_r.stl" scale="0.001 0.001 0.001" />
+                <mesh filename="file://$(find r2_description)/meshes/b_wheel_r.stl" scale="0.001 0.001 0.001" />
             </geometry>
             <material name="wheel_color"/>
@@ -304,5 +306,5 @@
             <origin xyz="0.23800000000000002 0.044524999999999995 -0.2735" rpy="-1.5707963267948966 -0.0 0.0" />
             <geometry>
-                <mesh filename="package://r2_description/meshes/b_wheel_r.stl" scale="0.001 0.001 0.001" />
+                <cylinder length="0.08" radius="0.0625"/>
             </geometry>
             <surface>
@@ -325,5 +327,5 @@
             <origin xyz="0.23800000000000002 -0.044524999999999995 -0.2735" rpy="1.5707963267948966 -0.0 0.0" />
             <geometry>
-                <mesh filename="package://r2_description/meshes/b_wheel_l.stl" scale="0.001 0.001 0.001" />
+                <mesh filename="file://$(find r2_description)/meshes/b_wheel_l.stl" scale="0.001 0.001 0.001" />
             </geometry>
             <material name="wheel_color"/>
@@ -332,5 +334,5 @@
             <origin xyz="0.23800000000000002 -0.044524999999999995 -0.2735" rpy="1.5707963267948966 -0.0 0.0" />
             <geometry>
-                <mesh filename="package://r2_description/meshes/b_wheel_l.stl" scale="0.001 0.001 0.001" />
+                <cylinder length="0.08" radius="0.0625"/>
             </geometry>
             <surface>
@@ -354,5 +356,5 @@
             <origin xyz="0.0 0.3559999999999999 0.21249999999999997" rpy="1.5707963267948966 -0.0 0.0" />
             <geometry>
-                <mesh filename="package://r2_description/meshes/kfs_gripper_link.stl" scale="0.001 0.001 0.001" />
+                <mesh filename="file://$(find r2_description)/meshes/kfs_gripper_link.stl" scale="0.001 0.001 0.001" />
             </geometry>
         </visual>
@@ -360,5 +362,5 @@
             <origin xyz="0.0 0.3559999999999999 0.21249999999999997" rpy="1.5707963267948966 -0.0 0.0" />
             <geometry>
-                <mesh filename="package://r2_description/meshes/kfs_gripper_link.stl" scale="0.001 0.001 0.001" />
+                <box size="0.08 0.08 0.06"/>
             </geometry>
         </collision>
@@ -374,5 +376,5 @@
             <origin xyz="-0.2124999999999999 0.3559999999999999 -0.012000000000000002" rpy="1.5707963267948966 -1.5707963267948966 0" />
             <geometry>
-                <mesh filename="package://r2_description/meshes/kfs_finger.stl" scale="0.001 0.001 0.001" />
+                <mesh filename="file://$(find r2_description)/meshes/kfs_finger.stl" scale="0.001 0.001 0.001" />
             </geometry>
         </visual>
@@ -380,5 +382,5 @@
             <origin xyz="-0.2124999999999999 0.3559999999999999 -0.012000000000000002" rpy="1.5707963267948966 -1.5707963267948966 0" />
             <geometry>
-                <mesh filename="package://r2_description/meshes/kfs_finger.stl" scale="0.001 0.001 0.001" />
+                <box size="0.02 0.04 0.05"/>
             </geometry>
         </collision>
@@ -394,5 +396,5 @@
             <origin xyz="0.0 0.0 0.0" rpy="0.0 0.0 0.0" />
             <geometry>
-                <mesh filename="package://r2_description/meshes/spearhead_body.stl" scale="0.001 0.001 0.001" />
+                <mesh filename="file://$(find r2_description)/meshes/spearhead_body.stl" scale="0.001 0.001 0.001" />
             </geometry>
         </visual>
@@ -400,5 +402,5 @@
             <origin xyz="0.0 0.0 0.0" rpy="0.0 0.0 0.0" />
             <geometry>
-                <mesh filename="package://r2_description/meshes/spearhead_body.stl" scale="0.001 0.001 0.001" />
+                <box size="0.06 0.06 0.08"/>
             </geometry>
         </collision>
@@ -414,5 +416,5 @@
             <origin xyz="0.10250000190230253 0.2560000046766657 -0.008748863488359066" rpy="1.5707963267948963 -0.0 0.0" />
             <geometry>
-                <mesh filename="package://r2_description/meshes/spearhead_finger_r.stl" scale="0.001 0.001 0.001" />
+                <mesh filename="file://$(find r2_description)/meshes/spearhead_finger_r.stl" scale="0.001 0.001 0.001" />
             </geometry>
         </visual>
@@ -420,5 +422,5 @@
             <origin xyz="0.10250000190230253 0.2560000046766657 -0.008748863488359066" rpy="1.5707963267948963 -0.0 0.0" />
             <geometry>
-                <mesh filename="package://r2_description/meshes/spearhead_finger_r.stl" scale="0.001 0.001 0.001" />
+                <box size="0.01 0.04 0.06"/>
             </geometry>
         </collision>
@@ -434,5 +436,5 @@
             <origin xyz="0.13250000190230252 0.2560000046766657 0.008748869216825784" rpy="1.5707963267948963 -0.0 0.0" />
             <geometry>
-                <mesh filename="package://r2_description/meshes/spearhead_finger_l.stl" scale="0.001 0.001 0.001" />
+                <mesh filename="file://$(find r2_description)/meshes/spearhead_finger_l.stl" scale="0.001 0.001 0.001" />
             </geometry>
         </visual>
@@ -440,5 +442,5 @@
             <origin xyz="0.13250000190230252 0.2560000046766657 0.008748869216825784" rpy="1.5707963267948963 -0.0 0.0" />
             <geometry>
-                <mesh filename="package://r2_description/meshes/spearhead_finger_l.stl" scale="0.001 0.001 0.001" />
+                <box size="0.01 0.04 0.06"/>
             </geometry>
         </collision>
@@ -454,5 +456,5 @@
             <origin xyz="0.052499999999999984 0.36749999999999994 -3.552713678800515e-17" rpy="1.5707963267948966 -4.6816763546921983e-97 -1.1869459682199748e-66" />
             <geometry>
-                <mesh filename="package://r2_description/meshes/camera_link.stl" scale="0.001 0.001 0.001" />
+                <mesh filename="file://$(find r2_description)/meshes/camera_link.stl" scale="0.001 0.001 0.001" />
             </geometry>
             <material name="camera_color"/>
@@ -461,5 +463,5 @@
             <origin xyz="0.052499999999999984 0.36749999999999994 -3.552713678800515e-17" rpy="1.5707963267948966 -4.6816763546921983e-97 -1.1869459682199748e-66" />
             <geometry>
-                <mesh filename="package://r2_description/meshes/camera_link.stl" scale="0.001 0.001 0.001" />
+                <box size="0.03 0.03 0.03"/>
             </geometry>
         </collision>
@@ -502,5 +504,5 @@
             <origin xyz="0.0 0.0 0.0" rpy="0.0 0.0 0.0" />
             <geometry>
-                <mesh filename="package://r2_description/meshes/storage_plate.stl" scale="0.001 0.001 0.001" />
+                <mesh filename="file://$(find r2_description)/meshes/storage_plate.stl" scale="0.001 0.001 0.001" />
             </geometry>
             <material name="storage_plate_color"/>
@@ -509,9 +511,15 @@
             <origin xyz="0.0 0.0 0.0" rpy="0.0 0.0 0.0" />
             <geometry>
-                <mesh filename="package://r2_description/meshes/storage_plate.stl" scale="0.001 0.001 0.001" />
+                <mesh filename="file://$(find r2_description)/meshes/storage_plate.stl" scale="0.001 0.001 0.001" />
             </geometry>
         </collision>
     </link>
 <!--JOINTS-->
+    <!--Odometry to Base-->
+    <joint name="odom_base_link" type="fixed">
+        <origin xyz="0 0 0" rpy="0 0 0"/>
+        <parent link="odom"/>
+        <child link="base_link"/>
+    </joint>
     <!--Base link -Front-Back-Links-->
     <joint name="base_link_front_link" type="prismatic">
@@ -655,16 +663,18 @@
     </joint>
     <!--Spearhead Revolute-->
-    <joint name="kfs_gripper_link_spearhead_gripper_rotate" type="continuous">
+    <joint name="kfs_gripper_link_spearhead_gripper_rotate" type="revolute">
         <origin xyz="0.0 0.12 0.2125" rpy="+1.57 -0.0 0.0" />
         <parent link="kfs_gripper_link" />
         <child link="spearhead_body" />
         <axis xyz="0.0 8.359326303060042e-17 1.0" />
+        <limit lower="-1.57" upper="1.57" effort="100" velocity="1.0"/>
     </joint>
     <!--CAMERA Rotation-->
-    <joint name="kfs_gripper_link_camera_rotate" type="continuous">
+    <joint name="kfs_gripper_link_camera_rotate" type="revolute">
         <origin xyz="0.0 0.0 0.2125" rpy="3.944304526105059e-31 -0.0 1.1869459682199748e-66" />
         <parent link="kfs_gripper_link" />
         <child link="camera_link" />
         <axis xyz="0.0 3.944304526105059e-31 1.0" />
+        <limit lower="-1.57" upper="1.57" effort="100" velocity="1.0"/>
     </joint>
     <!--LIDAR Joint-->
@@ -672,5 +682,5 @@
         <parent link="base_link"/>
         <child link="lidar_link"/>
-        <origin xyz="0 0 -0.05" rpy="0 0 0"/>
+        <origin xyz="0 0 0.05" rpy="0 0 0"/>
     </joint>
     <!--Storage Plate Joint-->
@@ -685,51 +695,8 @@
             filename="libgz_ros2_control-system.so"
             name="gz_ros2_control::GazeboSimROS2ControlPlugin">
+            <parameters>
+                $(find r2_control)/config/controller_manager.yaml
+            </parameters>
         </plugin>
-    </gazebo>
-<!--Camera Sensor Plugin-->
-    <gazebo reference="camera_link">
-        <sensor name="camera_sensor" type="camera">
-            <always_on>true</always_on>
-            <visualize>true</visualize>
-            <update_rate>30</update_rate>
-            <topic>/camera/image_raw</topic>
-            <camera>
-            <horizontal_fov>1.047</horizontal_fov>
-            <image>
-                <width>640</width>
-                <height>480</height>
-                <format>R8G8B8</format>
-            </image>
-            <clip>
-                <near>0.1</near>
-                <far>100</far>
-            </clip>
-            </camera>
-        </sensor>
-    </gazebo>
-<!--LIDAR Sensor Plugin-->
-    <gazebo reference="lidar_link">
-        <sensor name="lidar_sensor" type="ray">
-            <always_on>true</always_on>
-            <visualize>true</visualize>
-            <update_rate>10</update_rate>
-            <topic>scan</topic>
-            <gz_frame_id>lidar_link</gz_frame_id>
-            <ray>
-            <scan>
-                <horizontal>
-                <samples>720</samples>
-                <resolution>1</resolution>
-                <min_angle>-3.14159</min_angle>
-                <max_angle>3.14159</max_angle>
-                </horizontal>
-            </scan>
-            <range>
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
Commit message: Updated the r2.xacro and r2.rviz

File: ros2_ws/src/r2_description/urdf/r2.xacro (robot description, xacro)
@@ -664,5 +664,5 @@
     <!--Spearhead Revolute-->
     <joint name="kfs_gripper_link_spearhead_gripper_rotate" type="revolute">
-        <origin xyz="0.0 0.12 0.2125" rpy="+1.57 -0.0 0.0" />
+        <origin xyz="0.0 0.36 0.2125" rpy="+1.57 0.0 0.0" />
         <parent link="kfs_gripper_link" />
         <child link="spearhead_body" />
