Commit message: The diff drive is working properly... The collsions and friction needs to be solved

File: ros2_ws/src/r2_description/urdf/gazebo.xacro (robot description, xacro)
@@ -2,11 +2,44 @@
 <robot xmlns:xacro="http://www.ros.org/wiki/xacro">
   <!-- ================================= -->
-  <!-- GAZEBO HARMONIC ROS2 CONTROL      -->
-  <!-- ROS2 JAZZY + GAZEBO HARMONIC      -->
+  <!-- GAZEBO HARMONIC DIFF DRIVE       -->
+  <!-- ROS 2 JAZZY + GAZEBO HARMONIC     -->
   <!-- ================================= -->
   <gazebo>
     <plugin
-        filename="libgz_ros2_control-system.so"
-        name="gz_ros2_control::GazeboSimROS2ControlPlugin">
+      filename="gz-sim-diff-drive-system"
+      name="gz::sim::systems::DiffDrive">
+      <!-- R2: four-wheel differential / skid-steer drive -->
+      <left_joint>f_wheel_l_revolute</left_joint>
+      <left_joint>b_wheel_l_revolute</left_joint>
+      <right_joint>f_wheel_r_revolute</right_joint>
+      <right_joint>b_wheel_r_revolute</right_joint>
+      <!-- Measured from the wheel joint locations -->
+      <wheel_separation>0.545</wheel_separation>
+      <wheel_radius>0.06</wheel_radius>
+      <!-- Explicit model-scoped Gazebo Transport topics -->
+      <topic>/cmd_vel</topic>
+      <odom_topic>/model/r2/odom</odom_topic>
+      <tf_topic>/model/r2/tf</tf_topic>
+      <frame_id>odom</frame_id>
+      <child_frame_id>base_footprint</child_frame_id>
+      <odom_publish_frequency>50</odom_publish_frequency>
+      <max_linear_velocity>1.0</max_linear_velocity>
+      <min_linear_velocity>-1.0</min_linear_velocity>
+      <max_angular_velocity>2.0</max_angular_velocity>
+      <min_angular_velocity>-2.0</min_angular_velocity>
+      <max_linear_acceleration>1.0</max_linear_acceleration>
+      <min_linear_acceleration>-1.0</min_linear_acceleration>
+      <max_angular_acceleration>2.0</max_angular_acceleration>
+      <min_angular_acceleration>-2.0</min_angular_acceleration>
+    </plugin>
+    <!-- Publish the four driven wheel states from Gazebo -->
+    <plugin
+      filename="gz-sim-joint-state-publisher-system"
+      name="gz::sim::systems::JointStatePublisher">
+      <topic>/model/r2/joint_states</topic>
+      <joint_name>f_wheel_l_revolute</joint_name>
+      <joint_name>f_wheel_r_revolute</joint_name>
+      <joint_name>b_wheel_l_revolute</joint_name>
+      <joint_name>b_wheel_r_revolute</joint_name>
     </plugin>
   </gazebo>

File: ros2_ws/src/r2_description/urdf/r2.xacro (robot description, xacro)
@@ -690,109 +690,3 @@
         <origin xyz="0 0 0" rpy="0 0 0"/>
     </joint>
-<!-- Harmonic ROS2 Control Plugin -->
-    <gazebo>
-        <plugin
-            filename="libgz_ros2_control-system.so"
-            name="gz_ros2_control::GazeboSimROS2ControlPlugin">
-            <parameters>
-                $(find r2_control)/config/controller_manager.yaml
-            </parameters>
-        </plugin>
-    </gazebo>
-<!--ro2_control block-->
-    <ros2_control name="GazeboSimSystem" type="system">
-        <hardware>
-            <plugin>gz_ros2_control/GazeboSimSystem</plugin>
-        </hardware>
-        <!-- Front Step Mechanism -->
-        <joint name="base_link_front_link">
-            <command_interface name="position"/>
-            <state_interface name="position"/>
-            <state_interface name="velocity"/>
-        </joint>
-        <!-- Back Step Mechanism -->
-        <joint name="base_link_back_link">
-            <command_interface name="position"/>
-            <state_interface name="position"/>
-            <state_interface name="velocity"/>
-        </joint>
-        <!-- Front Right -->
-        <joint name="f_wheel_r_revolute">
-            <command_interface name="velocity"/>
-            <state_interface name="position"/>
-            <state_interface name="velocity"/>
-        </joint>
-        <!-- Front Left -->
-        <joint name="f_wheel_l_revolute">
-            <command_interface name="velocity"/>
-            <state_interface name="position"/>
-            <state_interface name="velocity"/>
-        </joint>
-        <!-- Back Right -->
-        <joint name="b_wheel_r_revolute">
-            <command_interface name="velocity"/>
-            <state_interface name="position"/>
-            <state_interface name="velocity"/>
-        </joint>
-        <!-- Back Left -->
-        <joint name="b_wheel_l_revolute">
-            <command_interface name="velocity"/>
-            <state_interface name="position"/>
-            <state_interface name="velocity"/>
-        </joint>
-        <!-- Vertical Expandable Right -->
-        <joint name="base_link_v_expandable_r">
-            <command_interface name="position"/>
-            <state_interface name="position"/>
-            <state_interface name="velocity"/>
-        </joint>
-        <!-- Vertical Expandable Left -->
-        <joint name="base_link_v_expandable_l">
-            <command_interface name="position"/>
-            <state_interface name="position"/>
-            <state_interface name="velocity"/>
-        </joint>
-        <!-- Vertical Gantry Right -->
-        <joint name="v_expandable_r_v_gantry_r">
-            <command_interface name="position"/>
-            <state_interface name="position"/>
-            <state_interface name="velocity"/>
-        </joint>
-        <!-- Vertical Gantry Left -->
-        <joint name="v_expandable_l_v_gantry_l">
-            <command_interface name="position"/>
-            <state_interface name="position"/>
-            <state_interface name="velocity"/>
-        </joint>
-        <!-- Horizontal Gantry Right -->
-        <joint name="h_expandable_r_h_gantry_r">
-            <command_interface name="position"/>
-            <state_interface name="position"/>
-            <state_interface name="velocity"/>
-        </joint>
-        <!-- Horizontal Gantry Left -->
-        <joint name="h_expandable_l_h_gantry_l">
-            <command_interface name="position"/>
-            <state_interface name="position"/>
-            <state_interface name="velocity"/>
-        </joint>
-        <!-- KFS Finger Gripper -->
-        <joint name="kfs_gripper_link_kfs_finger_grip">
-            <command_interface name="position"/>
-            <state_interface name="position"/>
-            <state_interface name="velocity"/>
-        </joint>
-        <!-- Spearhead Right Finger -->
-        <joint name="spearhead_body_spearhead_finger_r_grip">
-            <command_interface name="position"/>
-            <state_interface name="position"/>
-            <state_interface name="velocity"/>
-        </joint>
-        <!-- Spearhead Left Finger -->
-        <joint name="spearhead_body_spearhead_finger_l_grip">
-            <command_interface name="position"/>
-            <state_interface name="position"/>
-            <state_interface name="velocity"/>
-        </joint>
-    </ros2_control>
 </robot>
